Commit message: minor corrections on the robot spawn

File: UR5/ur_e_description/urdf/moving_base.gazebo.xacro (robot description, xacro)
@@ -2,4 +2,20 @@
 <robot name="moving_base" xmlns:xacro="http://ros.org/wiki/xacro">
     <xacro:arg name="imu_visual" default="false" />
+    <xacro:arg name="laser_visual" default="false" />
+    <xacro:arg name="camera_visual" default="false" />
+    <!--    bumper sensor-->
+    <gazebo reference="base_link_mb">
+        <sensor name="base_link_mb" type="contact">
+            <update_rate>1000.0</update_rate>
+            <always_on>true</always_on>
+            <contact>
+                <collision>base_footprint_fixed_joint_lump__base_link_collision</collision>
+            </contact>
+            <plugin name="base_link_contact_sensor_plugin" filename="libgazebo_ros_bumper.so">
+                <bumperTopicName>contact</bumperTopicName>
+                <frameName>world</frameName>
+            </plugin>
+        </sensor>
+    </gazebo>
     <gazebo reference="base_link_mb">
         <material>Gazebo/DarkGrey</material>
@@ -162,3 +178,38 @@
     </xacro:macro> -->
     <!-- add sensor part -->
+    <!-- lidar sensor -->
+    <!-- <gazebo reference="base_scan">
+        <material>Gazebo/DarkGrey</material>
+        <sensor type="ray" name="lds_lfcd_sensor">
+            <pose>0 0 0 0 0 0</pose>
+            <visualize>$(arg laser_visual)</visualize>
+            <update_rate>5</update_rate>
+            <ray>
+                <scan>
+                    <horizontal> -->
+                        <!--                        number of lidar points per rotation, here = 360-->
+                        <!-- <samples>360</samples>
+                        <resolution>1</resolution>
+                        <min_angle>0.0</min_angle>
+                        <max_angle>6.28319</max_angle>
+                    </horizontal>
+                </scan>
+                <range>
+                    <min>0.120</min>
+                    <max>3.5</max>
+                    <resolution>0.015</resolution>
+                </range>
+                <noise>
+                    <type>gaussian</type>
+                    <mean>0.0</mean>
+                    <stddev>0.01</stddev>
+                </noise>
+            </ray>
+            <plugin name="gazebo_ros_lds_lfcd_controller" filename="libgazebo_ros_laser.so">
+                <topicName>scan</topicName>
+                <frameName>base_scan</frameName>
+            </plugin>
+        </sensor>
+    </gazebo> -->
+    <!-- lidar sensor -->
 </robot>

File: UR5/ur_e_description/urdf/moving_base.urdf.xacro (robot description, xacro)
@@ -3,5 +3,5 @@
     <xacro:include filename="$(find ur_e_description)/urdf/properties.xacro" />
     <xacro:include filename="$(find ur_e_description)/urdf/moving_base.gazebo.xacro" />
-     <xacro:property name="M_PI" value="3.1415926535897931" />
+    <xacro:property name="M_PI" value="3.1415926535897931" />
     <!-- testing adding a velodyne laser  -->
     <!-- VLP-16 -->
@@ -230,3 +230,30 @@
     </joint>
     <link name="imu_link" />
+    <!-- lidar sensor -->
+    <!-- <joint name="scan_joint" type="fixed">
+        <parent link="base_link" />
+        <child link="base_scan" />
+        <origin xyz="-0.064 0 0.122" rpy="0 0 0" />
+    </joint> -->
+    <!-- <link name="base_scan">
+        <visual>
+            <origin xyz="0 0 0.0" rpy="0 0 0" />
+            <geometry>
+                <mesh filename="package://turtlebot3_description/meshes/sensors/lds.stl" scale="0.001 0.001 0.001" />
+            </geometry>
+            <material name="dark" />
+        </visual>
+        <collision>
+            <origin xyz="0.015 0 -0.0065" rpy="0 0 0" />
+            <geometry>
+                <cylinder length="0.0315" radius="0.055" />
+            </geometry>
+        </collision>
+        <inertial>
+            <mass value="0.114" />
+            <origin xyz="0 0 0" />
+            <inertia ixx="0.001" ixy="0.0" ixz="0.0" iyy="0.001" iyz="0.0" izz="0.001" />
+        </inertial>
+    </link> -->
+    <!-- lidar sensor -->
 </robot>

File: UR5/ur_e_description/urdf/ur5e.urdf.xacro (robot description, xacro)
@@ -3,4 +3,13 @@
   <xacro:include filename="$(find ur_e_description)/urdf/ur.transmission.xacro" />
   <xacro:include filename="$(find ur_e_description)/urdf/ur.gazebo.xacro" />
+  <!-- place robot on moving base -->
+  <xacro:include filename="$(find ur_e_description)/urdf/moving_base.urdf.xacro" />
+  <joint name="moving_base_to_ur5e" type="fixed">
+    <parent link="base_link_mb" />
+    <child link="base_link" />
+    <!-- <origin xyz="0.0 0.0 0.771" rpy="0.0 0.0 0.0" /> -->
+    <origin xyz="-0.296 -0.1688 0.826" rpy="0.0 0.0 0.0" />
+  </joint>
+  <!-- place robot on moving base -->
   <xacro:macro name="cylinder_inertial" params="radius length mass *origin">
     <inertial>

File: UR5/ur_e_description/urdf/ur5e_joint_limited_robot.urdf.xacro (robot description, xacro)
@@ -15,12 +15,13 @@
     wrist_3_lower_limit="${-pi}" wrist_3_upper_limit="${pi}"
   />
+  <!-- THIS PART WAS MOVED TO UR5E.URDF.XACRO  -->
   <!-- place robot on moving base -->
-  <xacro:include filename="$(find ur_e_description)/urdf/moving_base.urdf.xacro" />
+  <!-- <xacro:include filename="$(find ur_e_description)/urdf/moving_base.urdf.xacro" />
   <joint name="moving_base_to_ur5e" type="fixed">
     <parent link="base_link_mb" />
     <child link="base_link" />
-    <!-- <origin xyz="0.0 0.0 0.771" rpy="0.0 0.0 0.0" /> -->
     <origin xyz="-0.296 -0.1688 0.826" rpy="0.0 0.0 0.0"/>
-  </joint>
+  </joint> -->
+  <!-- THIS PART WAS MOVED TO UR5E.URDF.XACRO  -->
   <!-- sensor -->
   <!-- <xacro:include filename="$(find ur_e_description)/urdf/astra.urdf.xacro" />

Commit message: add front and back laser w/ imgs

File: UR5/ur_e_description/urdf/moving_base.gazebo.xacro (robot description, xacro)
@@ -3,5 +3,4 @@
     <xacro:arg name="imu_visual" default="false" />
     <xacro:arg name="laser_visual" default="false" />
-    <xacro:arg name="camera_visual" default="false" />
     <!--    bumper sensor-->
     <gazebo reference="base_link_mb">
@@ -177,9 +176,9 @@
         </gazebo>
     </xacro:macro> -->
-    <!-- add sensor part -->
-    <!-- lidar sensor -->
-    <!-- <gazebo reference="base_scan">
+    <!-- add sensor camera part -->
+    <!-- lidar sensor front -->
+    <gazebo reference="base_scan_front">
         <material>Gazebo/DarkGrey</material>
-        <sensor type="ray" name="lds_lfcd_sensor">
+        <sensor type="ray" name="lds_lfcd_sensor_front">
             <pose>0 0 0 0 0 0</pose>
             <visualize>$(arg laser_visual)</visualize>
@@ -187,10 +186,9 @@
             <ray>
                 <scan>
-                    <horizontal> -->
-                        <!--                        number of lidar points per rotation, here = 360-->
-                        <!-- <samples>360</samples>
+                    <horizontal>
+                        <samples>360</samples>
                         <resolution>1</resolution>
                         <min_angle>0.0</min_angle>
-                        <max_angle>6.28319</max_angle>
+                        <max_angle>3.14</max_angle>
                     </horizontal>
                 </scan>
@@ -207,9 +205,43 @@
             </ray>
             <plugin name="gazebo_ros_lds_lfcd_controller" filename="libgazebo_ros_laser.so">
-                <topicName>scan</topicName>
-                <frameName>base_scan</frameName>
+                <topicName>laser/scan_front</topicName>
+                <frameName>base_scan_front</frameName>
             </plugin>
         </sensor>
-    </gazebo> -->
-    <!-- lidar sensor -->
+    </gazebo>
+    <!-- lidar sensor front -->
+    <!-- lidar sensor back -->
+    <gazebo reference="base_scan_back">
+        <material>Gazebo/DarkGrey</material>
+        <sensor type="ray" name="lds_lfcd_sensor_back">
+            <pose>0 0 0 0 0 0</pose>
+            <visualize>$(arg laser_visual)</visualize>
+            <update_rate>5</update_rate>
+            <ray>
+                <scan>
+                    <horizontal>
+                        <samples>360</samples>
+                        <resolution>1</resolution>
+                        <min_angle>0.0</min_angle>
+                        <max_angle>3.14</max_angle>
+                    </horizontal>
+                </scan>
+                <range>
+                    <min>0.120</min>
+                    <max>3.5</max>
+                    <resolution>0.015</resolution>
+                </range>
+                <noise>
+                    <type>gaussian</type>
+                    <mean>0.0</mean>
+                    <stddev>0.01</stddev>
+                </noise>
+            </ray>
+            <plugin name="gazebo_ros_lds_lfcd_controller" filename="libgazebo_ros_laser.so">
+                <topicName>laser/scan_back</topicName>
+                <frameName>base_scan_back</frameName>
+            </plugin>
+        </sensor>
+    </gazebo>
+    <!-- lidar sensor back -->
 </robot>

File: UR5/ur_e_description/urdf/moving_base.urdf.xacro (robot description, xacro)
@@ -230,18 +230,11 @@
     </joint>
     <link name="imu_link" />
-    <!-- lidar sensor -->
-    <!-- <joint name="scan_joint" type="fixed">
-        <parent link="base_link" />
-        <child link="base_scan" />
-        <origin xyz="-0.064 0 0.122" rpy="0 0 0" />
-    </joint> -->
-    <!-- <link name="base_scan">
-        <visual>
-            <origin xyz="0 0 0.0" rpy="0 0 0" />
-            <geometry>
-                <mesh filename="package://turtlebot3_description/meshes/sensors/lds.stl" scale="0.001 0.001 0.001" />
-            </geometry>
-            <material name="dark" />
-        </visual>
+    <!-- lidar sensor front -->
+    <joint name="scan_joint_front" type="fixed">
+        <parent link="base_link_mb" />
+        <child link="base_scan_front" />
+        <origin xyz="-0.450 0 0.180" rpy="0 0 ${M_PI/2}" />
+    </joint>
+    <link name="base_scan_front">
         <collision>
             <origin xyz="0.015 0 -0.0065" rpy="0 0 0" />
@@ -255,5 +248,25 @@
             <inertia ixx="0.001" ixy="0.0" ixz="0.0" iyy="0.001" iyz="0.0" izz="0.001" />
         </inertial>
-    </link> -->
-    <!-- lidar sensor -->
+    </link>
+    <!-- lidar sensor front -->
+    <!-- lidar sensor back -->
+    <joint name="scan_joint_back" type="fixed">
+        <parent link="base_link_mb" />
+        <child link="base_scan_back" />
+        <origin xyz="0.450 0 0.180" rpy="0 0 -${M_PI/2}" />
+    </joint>
+    <link name="base_scan_back">
+        <collision>
+            <origin xyz="0.015 0 -0.0065" rpy="0 0 0" />
+            <geometry>
+                <cylinder length="0.0315" radius="0.055" />
+            </geometry>
+        </collision>
+        <inertial>
+            <mass value="0.114" />
+            <origin xyz="0 0 0" />
+            <inertia ixx="0.001" ixy="0.0" ixz="0.0" iyy="0.001" iyz="0.0" izz="0.001" />
+        </inertial>
+    </link>
+    <!-- lidar sensor back -->
 </robot>

Commit message: update lidar pose

File: UR5/ur_e_description/urdf/moving_base.gazebo.xacro (robot description, xacro)
@@ -189,6 +189,6 @@
                         <samples>360</samples>
                         <resolution>1</resolution>
-                        <min_angle>0.0</min_angle>
-                        <max_angle>3.14</max_angle>
+                        <min_angle>0</min_angle>
+                        <max_angle>4.71</max_angle>
                     </horizontal>
                 </scan>
@@ -223,6 +223,6 @@
                         <samples>360</samples>
                         <resolution>1</resolution>
-                        <min_angle>0.0</min_angle>
-                        <max_angle>3.14</max_angle>
+                        <min_angle>0</min_angle>
+                        <max_angle>4.71</max_angle>
                     </horizontal>
                 </scan>

File: UR5/ur_e_description/urdf/moving_base.urdf.xacro (robot description, xacro)
@@ -235,5 +235,5 @@
         <parent link="base_link_mb" />
         <child link="base_scan_front" />
-        <origin xyz="-0.450 0 0.180" rpy="0 0 ${M_PI/2}" />
+        <origin xyz="-0.700 0 0.180" rpy="0 0 ${M_PI/4}" />
     </joint>
     <link name="base_scan_front">
@@ -255,5 +255,5 @@
         <parent link="base_link_mb" />
         <child link="base_scan_back" />
-        <origin xyz="0.450 0 0.180" rpy="0 0 -${M_PI/2}" />
+        <origin xyz="0.700 0 0.180" rpy="0 0 -${3*M_PI/4}" />
     </joint>
     <link name="base_scan_back">
