Commit message: AGV world

File: UR5/ur_e_description/urdf/moving_base.urdf.xacro (robot description, xacro)
@@ -24,4 +24,10 @@
             rpy="0 0 3.14" />
     </xacro:sensor_astra> -->
+    <link name="world" />
+    <joint name="world_joint" type="fixed">
+      <parent link="world" />
+      <child link="base_link_mb" />
+      <origin xyz="0.0 0.0 0.0" rpy="0.0 0.0 0.0" />
+    </joint>
     <link name="base_link_mb">
         <visual>
