Commit message: add cameras realsense d415 to manipulator

File: UR5/ur_e_description/urdf/ur.gazebo.xacro (robot description, xacro)
@@ -28,5 +28,5 @@
   ur.gazebo.xacro
   ur5e.urdf.xacro -->
-  <xacro:macro name="sim_3dsensor" params="prefix">
+  <!-- <xacro:macro name="sim_3dsensor" params="prefix">
     <gazebo reference="${prefix}_depth_frame">
       <sensor type="depth" name="camera">
@@ -65,5 +65,5 @@
       </sensor>
     </gazebo>
-  </xacro:macro>
+  </xacro:macro> -->
   <!-- add sensor part -->
 </robot>

File: UR5/ur_e_description/urdf/ur5e.urdf.xacro (robot description, xacro)
@@ -12,5 +12,5 @@
     <parent link="base_link_mb" />
     <child link="base_link" />
-    <origin xyz="-0.296 -0.1688 0.826" rpy="0.0 0.0 0.0" />
+    <origin xyz="-0.295 0.0 0.780" rpy="0.0 0.0 0.0" />
   </joint>
   <!-- place robot on moving base -->
@@ -487,9 +487,31 @@
     ur.gazebo.xacro
     ur5e.urdf.xacro -->
-    <xacro:include filename="$(find ur_e_description)/urdf/astra.urdf.xacro" />
+    <!-- <xacro:include filename="$(find ur_e_description)/urdf/astra.urdf.xacro" />
     <xacro:sensor_astra parent="ee_link" prefix="camera">
       <origin xyz="0.06 -0.05 0.05"
         rpy="${-pi} -0.0 0.0" />
-    </xacro:sensor_astra>
+    </xacro:sensor_astra> -->
+    <!-- add intel realsense camera d415 sensor -->
+    <xacro:arg name="realsense_EE_enabled" default="$(optenv REALSENSE_EE_ENABLED 1)" />
+    <xacro:arg name="realsense_EE_topic" default="$(optenv REALSENSE_EE_TOPIC EE_realsense)" />
+    <xacro:arg name="realsense_EE_prefix" default="$(optenv REALSENSE_EE_PREFIX EE_camera_realsense)" />
+    <xacro:arg name="realsense_EE_parent" default="$(optenv REALSENSE_EE_PARENT ee_link)" />
+    <xacro:arg name="realsense_EE_xyz" default="$(optenv REALSENSE_EE_XYZ 0.095 0.000 -0.075)" />
+    <xacro:arg name="realsense_EE_rpy" default="$(optenv REALSENSE_EE_RPY -3.14 0.0 1.57)" />
+    <!-- <material name="white">
+      <color rgba="1.0 1.0 1.0 1.0" />
+    </material> -->
+    <xacro:include filename="$(find ur_e_description)/urdf/realsense/intel_realsense.urdf.xacro" />
+    <xacro:if value="$(arg realsense_EE_enabled)">
+      <link name="$(arg realsense_EE_prefix)_realsense_mountpoint" />
+      <joint name="$(arg realsense_EE_prefix)_realsense_mountpoint_joint" type="fixed">
+        <origin xyz="$(arg realsense_EE_xyz)" rpy="$(arg realsense_EE_rpy)" />
+        <parent link="$(arg realsense_EE_parent)" />
+        <child link="$(arg realsense_EE_prefix)_realsense_mountpoint" />
+      </joint>
+      <xacro:intel_realsense_mount prefix="$(arg realsense_EE_prefix)" topic="$(arg realsense_EE_topic)"
+        parent_link="$(arg realsense_EE_prefix)_realsense_mountpoint" />
+    </xacro:if>
+    <!-- add intel realsense d415 sensor -->
     <!-- SENSOR CAMERA ON END EFFECTOR -->
     <xacro:ur_arm_transmission prefix="${prefix}" />
@@ -498,9 +520,9 @@
     <!-- <link name="${prefix}base" />
     <joint name="${prefix}base_link-base_fixed_joint" type="fixed"> -->
-      <!-- NOTE: this rotation is only needed as long as base_link itself is
+    <!-- NOTE: this rotation is only needed as long as base_link itself is
                  not corrected wrt the real robot (ie: rotated over 180
                  degrees)
       -->
-      <!-- <origin xyz="0 0 0" rpy="0 0 ${-pi}" />
+    <!-- <origin xyz="0 0 0" rpy="0 0 ${-pi}" />
       <parent link="${prefix}base_link" />
       <child link="${prefix}base" />
