Commit message: add e0 eye on hand calibration

File: UR5/ur_e_description/urdf/astra.urdf.xacro (robot description, xacro)
@@ -3,28 +3,28 @@
   <xacro:include filename="$(find ur_e_description)/urdf/ur.gazebo.xacro" />
   <!-- Xacro properties -->
-  <xacro:property name="astra_cam_py" value="-0.0125"/>
+  <xacro:property name="astra_cam_py" value="-0.0125" />
   <xacro:property name="astra_depth_rel_rgb_py" value="0.0250" />
-  <xacro:property name="astra_cam_rel_rgb_py"   value="-0.0125" />
-  <xacro:property name="astra_dae_display_scale"   value="0.1" />
+  <xacro:property name="astra_cam_rel_rgb_py" value="-0.0125" />
+  <xacro:property name="astra_dae_display_scale" value="0.1" />
   <!-- Parameterised in part by the values in turtlebot_properties.urdf.xacro -->
   <xacro:macro name="sensor_astra" params="parent prefix *origin">
     <joint name="${prefix}_joint" type="fixed">
       <xacro:insert_block name="origin" />
-      <parent link="${parent}"/>
-      <child link="${prefix}_link"/>
+      <parent link="${parent}" />
+      <child link="${prefix}_link" />
     </joint>
     <link name="${prefix}_link">
-      <visual>
+      <!-- <visual>
         <origin xyz="-0.03 -0.06 0" rpy="${pi} 0 ${pi/2}"/>
         <geometry>
           <mesh filename="package://ur_e_description/meshes/sensors/astra2.dae" scale="1 1 1"/>
         </geometry>
-      </visual>
+      </visual> -->
       <collision>
         <!-- <origin xyz="0.0 0.0 0.0" rpy="0 0 0" /> -->
-        <origin xyz="-0.01 -0.06 0" rpy="0 0 0"/>
+        <origin xyz="-0.01 -0.06 0" rpy="0 0 0" />
         <geometry>
-        <box size="0.0400 0.1650 0.0300"/>
-      </geometry>
+          <box size="0.0400 0.1650 0.0300" />
+        </geometry>
       </collision>
       <inertial>
@@ -32,14 +32,18 @@
         <origin xyz="0 0 0" />
         <inertia ixx="0.003881243" ixy="0.0" ixz="0.0"
-                 iyy="0.000498940" iyz="0.0"
-                 izz="0.003879257" />
+          iyy="0.000498940" iyz="0.0"
+          izz="0.003879257" />
       </inertial>
     </link>
+    <!-- add to improve set initial pose on atom -->
+    <gazebo reference="${prefix}_link">
+      <selfCollide>false</selfCollide>
+    </gazebo>
     <joint name="${prefix}_rgb_joint" type="fixed">
       <origin xyz="0 -0.045 0" rpy="0 0 0" />
-      <parent link="${prefix}_link"/>
+      <parent link="${prefix}_link" />
       <child link="${prefix}_rgb_frame" />
     </joint>
-    <link name="${prefix}_rgb_frame"/>
+    <link name="${prefix}_rgb_frame" />
     <joint name="${prefix}_rgb_optical_joint" type="fixed">
       <origin xyz="0 0 0" rpy="${-pi/2} 0 ${-pi/2}" />
@@ -47,17 +51,34 @@
       <child link="${prefix}_rgb_optical_frame" />
     </joint>
-    <link name="${prefix}_rgb_optical_frame"/>
+    <!-- add to improve set initial pose on atom -->
+    <link name="${prefix}_rgb_optical_frame">
+      <visual>
+        <origin xyz="0.0 0.0 -0.03" rpy="${pi/2} 0 0" />
+        <geometry>
+          <mesh filename="package://t2rgb_description/meshes/sensors/astra2.dae" scale="1 1 1" />
+        </geometry>
+      </visual>
+    </link>
     <joint name="${prefix}_depth_joint" type="fixed">
-        <origin xyz="0 -0.02 0" rpy="0 0 0" />
-        <parent link="${prefix}_link" />
-        <child link="${prefix}_depth_frame" />
+      <origin xyz="0 -0.02 0" rpy="0 0 0" />
+      <parent link="${prefix}_link" />
+      <child link="${prefix}_depth_frame" />
     </joint>
-    <link name="${prefix}_depth_frame"/>
+    <link name="${prefix}_depth_frame" />
     <joint name="${prefix}_depth_optical_joint" type="fixed">
-        <origin xyz="0 0 0" rpy="${-pi/2} 0 ${-pi/2}" />
-        <parent link="${prefix}_depth_frame" />
-        <child link="${prefix}_depth_optical_frame" />
+      <origin xyz="0 0 0" rpy="${-pi/2} 0 ${-pi/2}" />
+      <parent link="${prefix}_depth_frame" />
+      <child link="${prefix}_depth_optical_frame" />
     </joint>
-    <link name="${prefix}_depth_optical_frame"/>
+       <!-- add to improve set initial pose on atom -->
+       <link name="${prefix}_depth_optical_frame">
+        <!-- <visual>
+          <origin xyz="0.0 0.0 0.0" rpy="0 0 0" />
+          <geometry> -->
+            <!-- Use a slightly smaller scale than 1, so that when both models overlap its the rgb that appears.-->
+            <!-- <mesh filename="package://t2rgb_description/meshes/sensors/astra2.dae" scale="0.98 0.98 0.98" />
+          </geometry>
+        </visual> -->
+      </link>
     <xacro:sim_3dsensor prefix="${prefix}" />
   </xacro:macro>

File: UR5/ur_e_description/urdf/moving_base.gazebo.xacro (robot description, xacro)
@@ -13,4 +13,6 @@
             <plugin name="base_link_contact_sensor_plugin" filename="libgazebo_ros_bumper.so">
                 <bumperTopicName>contact</bumperTopicName>
+                <!-- toogle this part to move the AGV in odom -->
+                <!-- <frameName>base_footprint</frameName> -->
                 <frameName>world</frameName>
             </plugin>
@@ -92,7 +94,11 @@
             <odometryTopic>odom</odometryTopic>
             <odometryFrame>odom</odometryFrame>
+            <!-- toogle this part to move the AGV in odom -->
+            <!-- <odometrySource>base_footprint</odometrySource> -->
             <odometrySource>world</odometrySource>
             <publishOdomTF>true</publishOdomTF>
-            <robotBaseFrame>base_footprint</robotBaseFrame>
+            <!-- toogle this part to move the AGV in odom -->
+            <!-- <robotBaseFrame>base_footprint</robotBaseFrame> -->
+            <robotBaseFrame>world</robotBaseFrame>
             <publishWheelTF>false</publishWheelTF>
             <publishTf>true</publishTf>
@@ -178,5 +184,5 @@
     <!-- add sensor camera part -->
     <!-- lidar sensor front -->
-    <gazebo reference="base_scan_front">
+    <!-- <gazebo reference="base_scan_front">
         <material>Gazebo/DarkGrey</material>
         <sensor type="ray" name="lds_lfcd_sensor_front">
@@ -209,8 +215,8 @@
             </plugin>
         </sensor>
-    </gazebo>
+    </gazebo> -->
     <!-- lidar sensor front -->
     <!-- lidar sensor back -->
-    <gazebo reference="base_scan_back">
+    <!-- <gazebo reference="base_scan_back">
         <material>Gazebo/DarkGrey</material>
         <sensor type="ray" name="lds_lfcd_sensor_back">
@@ -243,5 +249,5 @@
             </plugin>
         </sensor>
-    </gazebo>
+    </gazebo> -->
     <!-- lidar sensor back -->
 </robot>

File: UR5/ur_e_description/urdf/moving_base.urdf.xacro (robot description, xacro)
@@ -1,4 +1,5 @@
 <?xml version="1.0"?>
 <robot name="moving_base" xmlns:xacro="http://ros.org/wiki/xacro">
+    <!-- 2D LIDARS CODE AT THE END -->
     <xacro:include filename="$(find ur_e_description)/urdf/properties.xacro" />
     <xacro:include filename="$(find ur_e_description)/urdf/moving_base.gazebo.xacro" />
@@ -12,5 +13,6 @@
     <xacro:property name="organize_cloud" value="$(arg organize_cloud)" />
     <xacro:include filename="$(find velodyne_description)/urdf/VLP-16.urdf.xacro" />
-    <xacro:VLP-16 parent="base_link_mb" name="velodyne" topic="/velodyne_points" organize_cloud="${organize_cloud}" hz="10" samples="440" gpu="${gpu}">
+    <xacro:VLP-16 parent="base_link_mb" name="velodyne" topic="/velodyne_points"
+    organize_cloud="${organize_cloud}" hz="10" samples="440" gpu="${gpu}">
         <origin xyz="-0.350 -0.250 0.850" rpy="0 0 0" />
     </xacro:VLP-16> -->
@@ -22,35 +24,63 @@
             rpy="0 0 3.14" />
     </xacro:sensor_astra> -->
-    <link name="base_footprint" />
-    <joint name="base_joint" type="fixed">
+    <link name="base_link_mb">
+        <visual>
+            <origin xyz="-0.43 -0.33 0.03" rpy="${M_PI/2} 0 ${M_PI/2}" />
+            <geometry>
+                <!-- <box size="0.900 0.600 0.770" /> -->
+                <!-- <box size="0.900 0.650 0.770" /> -->
+                <mesh filename="package://ur_e_description/meshes/moving_base/moving_base.STL"
+                    scale="0.001 0.001 0.001" />
+            </geometry>
+            <material name="light_black" />
+        </visual>
+        <collision>
+            <origin xyz="0 0 0.459" rpy="0 0 0" />
+            <geometry>
+                <box size="0.900 0.600 0.770" />
+            </geometry>
+        </collision>
+        <!-- <inertial> -->
+            <!-- <origin xyz="0 0 0" rpy="0 0 0" /> -->
+            <!-- <mass value="46" /> -->
+            <!-- <inertia ixx="8.7002718e-03" ixy="-4.7576583e-05" ixz="1.1160499e-04"
+                iyy="8.6195418e-03" iyz="-3.5422299e-06"
+                izz="1.4612727e-02" /> -->
+            <!-- <inertia ixx="0.6022" ixy="-0.02364" ixz="-0.1197" iyy="1.7386" iyz="-0.001544" -->
+                <!-- izz="2.0296" /> -->
+        <!-- </inertial> -->
+    </link>
+    <!-- toogle this part to move the AGV in odom -->
+    <!-- <link name="base_footprint">
+        <collision>
+            <origin xyz="0 0 0" />
+            <geometry>
+                <sphere radius="0.00000001" />
+            </geometry>
+        </collision>
+    </link> -->
+    <!-- Colour -->
+    <!-- <gazebo reference="base_footprint">
+        <material>Gazebo/Purple</material>
+    </gazebo>
+    <joint name="base_footprint_joint" type="fixed">
         <parent link="base_footprint" />
         <child link="base_link_mb" />
         <origin xyz="0 0 0.010" rpy="0 0 0" />
-    </joint>
-    <link name="base_link_mb">
-        <visual>
-            <origin xyz="-0.43 -0.33 0.03" rpy="${M_PI/2} 0 ${M_PI/2}" />
-            <geometry>
-                <!-- <box size="0.900 0.600 0.770" /> -->
-                <!-- <box size="0.900 0.650 0.770" /> -->
-                <mesh filename="package://ur_e_description/meshes/moving_base/moving_base.STL" scale="0.001 0.001 0.001" />
-            </geometry>
-            <material name="light_black" />
-        </visual>
-        <collision>
-            <origin xyz="0 0 0.459" rpy="0 0 0" />
-            <geometry>
-                <box size="0.900 0.600 0.770" />
-            </geometry>
-        </collision>
-        <inertial>
-            <origin xyz="0 0 0" rpy="0 0 0" />
-            <mass value="46" />
-            <!-- <inertia ixx="8.7002718e-03" ixy="-4.7576583e-05" ixz="1.1160499e-04"
-                iyy="8.6195418e-03" iyz="-3.5422299e-06"
-                izz="1.4612727e-02" /> -->
-            <inertia ixx="0.6022" ixy="-0.02364" ixz="-0.1197" iyy="1.7386" iyz="-0.001544" izz="2.0296" />
-        </inertial>
-    </link>
+    </joint> -->
+    <!-- Inertial link stores the robot's inertial information FROM HUSKY GROUNG ROBOT -->
+    <link name="inertial_link">
+        <inertial>
+            <mass value="46.034" />
+            <origin xyz="-0.00065 -0.085 0.062" />
+            <inertia ixx="0.6022" ixy="-0.02364" ixz="-0.1197" iyy="1.7386" iyz="-0.001544"
+                izz="2.0296" />
+        </inertial>
+    </link>
+    <joint name="inertial_joint" type="fixed">
+        <origin xyz="0 0 0" rpy="0 0 0" />
+        <parent link="base_link_mb" />
+        <child link="inertial_link" />
+    </joint>
     <joint name="wheel_left_joint" type="continuous">
         <parent link="base_link_mb" />
@@ -63,5 +93,6 @@
             <origin xyz="0 0 -0.055" rpy="-1.57 0 0" />
             <geometry>
-                <mesh filename="package://ur_e_description/meshes/wheels/left_tire.stl" scale="0.0025 0.0025 0.0025" />
+                <mesh filename="package://ur_e_description/meshes/wheels/left_tire.stl"
+                    scale="0.0025 0.0025 0.0025" />
             </geometry>
             <material name="dark" />
@@ -91,5 +122,6 @@
             <origin xyz="0 0 0.055" rpy="1.57 0 0" />
             <geometry>
-                <mesh filename="package://ur_e_description/meshes/wheels/left_tire.stl" scale="0.0025 0.0025 0.0025" />
+                <mesh filename="package://ur_e_description/meshes/wheels/left_tire.stl"
+                    scale="0.0025 0.0025 0.0025" />
             </geometry>
             <material name="dark" />
@@ -119,5 +151,6 @@
             <origin xyz="0.027 -0.06 0" rpy="1.57 0 0" />
             <geometry>
-                <mesh filename="package://ur_e_description/meshes/wheels/left_tire.stl" scale="0.0020 0.0020 0.0020" />
+                <mesh filename="package://ur_e_description/meshes/wheels/left_tire.stl"
+                    scale="0.0020 0.0020 0.0020" />
                 <!-- <cylinder length="0.024" radius="0.084" /> -->
             </geometry>
@@ -147,5 +180,6 @@
             <origin xyz="0.027 -0.06 0" rpy="-1.57 0 0" />
             <geometry>
-                <mesh filename="package://ur_e_description/meshes/wheels/left_tire.stl" scale="0.0020 0.0020 0.0020" />
+                <mesh filename="package://ur_e_description/meshes/wheels/left_tire.stl"
+                    scale="0.0020 0.0020 0.0020" />
                 <!-- <cylinder length="0.024" radius="0.084" /> -->
             </geometry>
@@ -177,5 +211,6 @@
             <origin xyz="0 -0.06 0" rpy="1.57 0 0" />
             <geometry>
-                <mesh filename="package://ur_e_description/meshes/wheels/left_tire.stl" scale="0.0020 0.0020 0.0020" />
+                <mesh filename="package://ur_e_description/meshes/wheels/left_tire.stl"
+                    scale="0.0020 0.0020 0.0020" />
                 <!-- <cylinder length="0.024" radius="0.084" /> -->
             </geometry>
@@ -205,5 +240,6 @@
             <origin xyz="0 -0.06 0" rpy="-1.57 0 0" />
             <geometry>
-                <mesh filename="package://ur_e_description/meshes/wheels/left_tire.stl" scale="0.0020 0.0020 0.0020" />
+                <mesh filename="package://ur_e_description/meshes/wheels/left_tire.stl"
+                    scale="0.0020 0.0020 0.0020" />
                 <!-- <cylinder length="0.024" radius="0.084" /> -->
             </geometry>
@@ -231,6 +267,7 @@
     </joint>
     <link name="imu_link" />
+    <!-- ROMEVED FOR NOW - JORGE FEB 2023 -->
     <!-- lidar sensor front -->
-    <joint name="scan_joint_front" type="fixed">
+    <!-- <joint name="scan_joint_front" type="fixed">
         <parent link="base_link_mb" />
         <child link="base_scan_front" />
@@ -249,8 +286,8 @@
             <inertia ixx="0.001" ixy="0.0" ixz="0.0" iyy="0.001" iyz="0.0" izz="0.001" />
         </inertial>
-    </link>
+    </link> -->
     <!-- lidar sensor front -->
     <!-- lidar sensor back -->
-    <joint name="scan_joint_back" type="fixed">
+    <!-- <joint name="scan_joint_back" type="fixed">
         <parent link="base_link_mb" />
         <child link="base_scan_back" />
@@ -269,5 +306,6 @@
             <inertia ixx="0.001" ixy="0.0" ixz="0.0" iyy="0.001" iyz="0.0" izz="0.001" />
         </inertial>
-    </link>
+    </link> -->
     <!-- lidar sensor back -->
+    <!-- ROMEVED FOR NOW - JORGE FEB 2023 -->
 </robot>

File: UR5/ur_e_description/urdf/ur.gazebo.xacro (robot description, xacro)
@@ -25,5 +25,8 @@
   </xacro:macro>
   <!-- add sensor camera part -->
-  <!-- <xacro:macro name="sim_3dsensor" params="prefix">
+  <!-- Files to add sensor camera on end-effector:
+  ur.gazebo.xacro
+  ur5e.urdf.xacro -->
+  <xacro:macro name="sim_3dsensor" params="prefix">
     <gazebo reference="${prefix}_depth_frame">
       <sensor type="depth" name="camera">
@@ -62,5 +65,5 @@
       </sensor>
     </gazebo>
-  </xacro:macro> -->
+  </xacro:macro>
   <!-- add sensor part -->
 </robot>

File: UR5/ur_e_description/urdf/ur.transmission.xacro (robot description, xacro)
@@ -56,6 +56,12 @@
       </actuator>
     </transmission>
-    <!-- add gripper part -->
-    <!-- <transmission name="${prefix}left_finger_trans">
+    <!-- add gripper part start
+    FOR THE GRIPPER (toogle gripper parts in):
+    ur_e_description/urdf/ur.transmission.xacro
+    ur_e_description/urdf/ur5e.urdf.xacro
+    ur_e_gazebo/launch/ur5.launch
+    ur5_e_moveit_config/config/ur5e.srdf
+    -->
+    <transmission name="${prefix}left_finger_trans">
       <type>transmission_interface/SimpleTransmission</type>
       <joint name="${prefix}left_finger_joint">
@@ -76,6 +82,6 @@
         <mechanicalReduction>1</mechanicalReduction>
       </actuator>
-    </transmission> -->
-    <!-- add gripper part -->
+    </transmission>
+    <!-- add gripper part end -->
   </xacro:macro>
 </robot>
