Commit message: add e0 eye on hand calibration

File: UR5/ur_e_description/urdf/ur5e.urdf.xacro (robot description, xacro)
@@ -5,4 +5,5 @@
   <!-- place robot on moving base -->
   <xacro:include filename="$(find ur_e_description)/urdf/moving_base.urdf.xacro" />
+  <!-- *************THIS IS THE TRANSFORMATION TO BE CALIBRATED************* -->
   <joint name="moving_base_to_ur5e" type="fixed">
     <parent link="base_link_mb" />
@@ -16,8 +17,11 @@
       <mass value="${mass}" />
       <xacro:insert_block name="origin" />
-      <inertia ixx="${0.0833333 * mass * (3 * radius * radius + length * length)}" ixy="0.0" ixz="0.0" iyy="${0.0833333 * mass * (3 * radius * radius + length * length)}" iyz="0.0" izz="${0.5 * mass * radius * radius}" />
+      <inertia ixx="${0.0833333 * mass * (3 * radius * radius + length * length)}" ixy="0.0"
+        ixz="0.0" iyy="${0.0833333 * mass * (3 * radius * radius + length * length)}" iyz="0.0"
+        izz="${0.5 * mass * radius * radius}" />
     </inertial>
   </xacro:macro>
-  <xacro:macro name="ur5e_robot" params="prefix joint_limited
+  <xacro:macro name="ur5e_robot"
+    params="prefix joint_limited
     shoulder_pan_lower_limit:=${-pi}    shoulder_pan_upper_limit:=${pi}
     shoulder_lift_lower_limit:=${-pi}    shoulder_lift_upper_limit:=${pi}
@@ -53,5 +57,6 @@
       joint_direction = [-1, -1, 1, 1, 1, 1]
       mass = [3.7000, 8.3930, 2.2750, 1.2190, 1.2190, 0.1879]
-      center_of_mass = [ [0, -0.02561, 0.00193], [0.2125, 0, 0.11336], [0.11993, 0.0, 0.0265], [0, -0.0018, 0.01634], [0, 0.0018,0.01634], [0, 0, -0.001159] ]
+      center_of_mass = [ [0, -0.02561, 0.00193], [0.2125, 0, 0.11336], [0.11993, 0.0, 0.0265], [0,
+    -0.0018, 0.01634], [0, 0.0018,0.01634], [0, 0, -0.001159] ]
     -->
     <xacro:property name="d1" value="0.163" />
@@ -71,16 +76,24 @@
     <xacro:property name="wrist_2_length" value="${d5}" />
     <xacro:property name="wrist_3_length" value="${d6}" />
-    <!--property name="shoulder_height" value="0.089159" /-->
-    <!--property name="shoulder_offset" value="0.13585" /-->
+    <!--property
+    name="shoulder_height" value="0.089159" /-->
+    <!--property
+    name="shoulder_offset" value="0.13585" /-->
     <!-- shoulder_offset - elbow_offset + wrist_1_length = 0.10915 -->
-    <!--property name="upper_arm_length" value="0.42500" /-->
-    <!--property name="elbow_offset" value="0.1197" /-->
+    <!--property
+    name="upper_arm_length" value="0.42500" /-->
+    <!--property
+    name="elbow_offset" value="0.1197" /-->
     <!-- CAD measured -->
-    <!--property name="forearm_length" value="0.39225" /-->
-    <!--property name="wrist_1_length" value="0.093" /-->
+    <!--property
+    name="forearm_length" value="0.39225" /-->
+    <!--property
+    name="wrist_1_length" value="0.093" /-->
     <!-- CAD measured -->
-    <!--property name="wrist_2_length" value="0.09465" /-->
+    <!--property
+    name="wrist_2_length" value="0.09465" /-->
     <!-- In CAD this distance is 0.930, but in the spec it is 0.09465 -->
-    <!--property name="wrist_3_length" value="0.0823" /-->
+    <!--property
+    name="wrist_3_length" value="0.0823" /-->
     <xacro:property name="shoulder_radius" value="0.060" /> <!-- manually measured -->
     <xacro:property name="upper_arm_radius" value="0.054" /> <!-- manually measured -->
@@ -114,11 +127,16 @@
         <limit lower="${-2.0 * pi}" upper="${2.0 * pi}" effort="150.0" velocity="3.14" />
         <xacro:if value="${safety_limits}">
-          <safety_controller soft_lower_limit="${-2.0 * pi + safety_pos_margin}" soft_upper_limit="${2.0 * pi - safety_pos_margin}" k_position="${safety_k_position}" k_velocity="0.0" />
+          <safety_controller soft_lower_limit="${-2.0 * pi + safety_pos_margin}"
+            soft_upper_limit="${2.0 * pi - safety_pos_margin}" k_position="${safety_k_position}"
+            k_velocity="0.0" />
         </xacro:if>
       </xacro:unless>
       <xacro:if value="${joint_limited}">
-        <limit lower="${shoulder_pan_lower_limit}" upper="${shoulder_pan_upper_limit}" effort="150.0" velocity="3.14" />
-        <xacro:if value="${safety_limits}">
-          <safety_controller soft_lower_limit="${shoulder_pan_lower_limit + safety_pos_margin}" soft_upper_limit="${shoulder_pan_upper_limit - safety_pos_margin}" k_position="${safety_k_position}" k_velocity="0.0" />
+        <limit lower="${shoulder_pan_lower_limit}" upper="${shoulder_pan_upper_limit}"
+          effort="150.0" velocity="3.14" />
+        <xacro:if value="${safety_limits}">
+          <safety_controller soft_lower_limit="${shoulder_pan_lower_limit + safety_pos_margin}"
+            soft_upper_limit="${shoulder_pan_upper_limit - safety_pos_margin}"
+            k_position="${safety_k_position}" k_velocity="0.0" />
         </xacro:if>
       </xacro:if>
@@ -151,11 +169,16 @@
         <limit lower="${-2.0 * pi}" upper="${2.0 * pi}" effort="150.0" velocity="3.14" />
         <xacro:if value="${safety_limits}">
-          <safety_controller soft_lower_limit="${-2.0 * pi + safety_pos_margin}" soft_upper_limit="${2.0 * pi - safety_pos_margin}" k_position="${safety_k_position}" k_velocity="0.0" />
+          <safety_controller soft_lower_limit="${-2.0 * pi + safety_pos_margin}"
+            soft_upper_limit="${2.0 * pi - safety_pos_margin}" k_position="${safety_k_position}"
+            k_velocity="0.0" />
         </xacro:if>
       </xacro:unless>
       <xacro:if value="${joint_limited}">
-        <limit lower="${shoulder_lift_lower_limit}" upper="${shoulder_lift_upper_limit}" effort="150.0" velocity="3.14" />
-        <xacro:if value="${safety_limits}">
-          <safety_controller soft_lower_limit="${shoulder_lift_lower_limit + safety_pos_margin}" soft_upper_limit="${shoulder_lift_upper_limit - safety_pos_margin}" k_position="${safety_k_position}" k_velocity="0.0" />
+        <limit lower="${shoulder_lift_lower_limit}" upper="${shoulder_lift_upper_limit}"
+          effort="150.0" velocity="3.14" />
+        <xacro:if value="${safety_limits}">
+          <safety_controller soft_lower_limit="${shoulder_lift_lower_limit + safety_pos_margin}"
+            soft_upper_limit="${shoulder_lift_upper_limit - safety_pos_margin}"
+            k_position="${safety_k_position}" k_velocity="0.0" />
         </xacro:if>
       </xacro:if>
@@ -188,11 +211,16 @@
         <limit lower="${-pi}" upper="${pi}" effort="150.0" velocity="3.14" />
         <xacro:if value="${safety_limits}">
-          <safety_controller soft_lower_limit="${-2.0 * pi + safety_pos_margin}" soft_upper_limit="${2.0 * pi - safety_pos_margin}" k_position="${safety_k_position}" k_velocity="0.0" />
+          <safety_controller soft_lower_limit="${-2.0 * pi + safety_pos_margin}"
+            soft_upper_limit="${2.0 * pi - safety_pos_margin}" k_position="${safety_k_position}"
+            k_velocity="0.0" />
         </xacro:if>
       </xacro:unless>
       <xacro:if value="${joint_limited}">
-        <limit lower="${elbow_joint_lower_limit}" upper="${elbow_joint_upper_limit}" effort="150.0" velocity="3.14" />
-        <xacro:if value="${safety_limits}">
-          <safety_controller soft_lower_limit="${elbow_joint_lower_limit + safety_pos_margin}" soft_upper_limit="${elbow_joint_upper_limit - safety_pos_margin}" k_position="${safety_k_position}" k_velocity="0.0" />
+        <limit lower="${elbow_joint_lower_limit}" upper="${elbow_joint_upper_limit}" effort="150.0"
+          velocity="3.14" />
+        <xacro:if value="${safety_limits}">
+          <safety_controller soft_lower_limit="${elbow_joint_lower_limit + safety_pos_margin}"
+            soft_upper_limit="${elbow_joint_upper_limit - safety_pos_margin}"
+            k_position="${safety_k_position}" k_velocity="0.0" />
         </xacro:if>
       </xacro:if>
@@ -225,11 +253,16 @@
         <limit lower="${-2.0 * pi}" upper="${2.0 * pi}" effort="28.0" velocity="6.28" />
         <xacro:if value="${safety_limits}">
-          <safety_controller soft_lower_limit="${-2.0 * pi + safety_pos_margin}" soft_upper_limit="${2.0 * pi - safety_pos_margin}" k_position="${safety_k_position}" k_velocity="0.0" />
+          <safety_controller soft_lower_limit="${-2.0 * pi + safety_pos_margin}"
+            soft_upper_limit="${2.0 * pi - safety_pos_margin}" k_position="${safety_k_position}"
+            k_velocity="0.0" />
         </xacro:if>
       </xacro:unless>
       <xacro:if value="${joint_limited}">
-        <limit lower="${wrist_1_lower_limit}" upper="${wrist_1_upper_limit}" effort="28.0" velocity="6.28" />
-        <xacro:if value="${safety_limits}">
-          <safety_controller soft_lower_limit="${wrist_1_lower_limit + safety_pos_margin}" soft_upper_limit="${wrist_1_upper_limit - safety_pos_margin}" k_position="${safety_k_position}" k_velocity="0.0" />
+        <limit lower="${wrist_1_lower_limit}" upper="${wrist_1_upper_limit}" effort="28.0"
+          velocity="6.28" />
+        <xacro:if value="${safety_limits}">
+          <safety_controller soft_lower_limit="${wrist_1_lower_limit + safety_pos_margin}"
+            soft_upper_limit="${wrist_1_upper_limit - safety_pos_margin}"
+            k_position="${safety_k_position}" k_velocity="0.0" />
         </xacro:if>
       </xacro:if>
@@ -262,11 +295,16 @@
         <limit lower="${-2.0 * pi}" upper="${2.0 * pi}" effort="28.0" velocity="6.28" />
         <xacro:if value="${safety_limits}">
-          <safety_controller soft_lower_limit="${-2.0 * pi + safety_pos_margin}" soft_upper_limit="${2.0 * pi - safety_pos_margin}" k_position="${safety_k_position}" k_velocity="0.0" />
+          <safety_controller soft_lower_limit="${-2.0 * pi + safety_pos_margin}"
+            soft_upper_limit="${2.0 * pi - safety_pos_margin}" k_position="${safety_k_position}"
+            k_velocity="0.0" />
         </xacro:if>
       </xacro:unless>
       <xacro:if value="${joint_limited}">
-        <limit lower="${wrist_2_lower_limit}" upper="${wrist_2_upper_limit}" effort="28.0" velocity="6.28" />
-        <xacro:if value="${safety_limits}">
-          <safety_controller soft_lower_limit="${wrist_2_lower_limit + safety_pos_margin}" soft_upper_limit="${wrist_2_upper_limit - safety_pos_margin}" k_position="${safety_k_position}" k_velocity="0.0" />
+        <limit lower="${wrist_2_lower_limit}" upper="${wrist_2_upper_limit}" effort="28.0"
+          velocity="6.28" />
+        <xacro:if value="${safety_limits}">
+          <safety_controller soft_lower_limit="${wrist_2_lower_limit + safety_pos_margin}"
+            soft_upper_limit="${wrist_2_upper_limit - safety_pos_margin}"
+            k_position="${safety_k_position}" k_velocity="0.0" />
         </xacro:if>
       </xacro:if>
@@ -299,11 +337,16 @@
         <limit lower="${-2.0 * pi}" upper="${2.0 * pi}" effort="28.0" velocity="6.28" />
         <xacro:if value="${safety_limits}">
-          <safety_controller soft_lower_limit="${-2.0 * pi + safety_pos_margin}" soft_upper_limit="${2.0 * pi - safety_pos_margin}" k_position="${safety_k_position}" k_velocity="0.0" />
+          <safety_controller soft_lower_limit="${-2.0 * pi + safety_pos_margin}"
+            soft_upper_limit="${2.0 * pi - safety_pos_margin}" k_position="${safety_k_position}"
+            k_velocity="0.0" />
         </xacro:if>
       </xacro:unless>
       <xacro:if value="${joint_limited}">
-        <limit lower="${wrist_3_lower_limit}" upper="${wrist_3_upper_limit}" effort="28.0" velocity="6.28" />
-        <xacro:if value="${safety_limits}">
-          <safety_controller soft_lower_limit="${wrist_3_lower_limit + safety_pos_margin}" soft_upper_limit="${wrist_3_upper_limit - safety_pos_margin}" k_position="${safety_k_position}" k_velocity="0.0" />
+        <limit lower="${wrist_3_lower_limit}" upper="${wrist_3_upper_limit}" effort="28.0"
+          velocity="6.28" />
+        <xacro:if value="${safety_limits}">
+          <safety_controller soft_lower_limit="${wrist_3_lower_limit + safety_pos_margin}"
+            soft_upper_limit="${wrist_3_upper_limit - safety_pos_margin}"
+            k_position="${safety_k_position}" k_velocity="0.0" />
         </xacro:if>
       </xacro:if>
@@ -341,6 +384,12 @@
       </collision>
     </link>
-    <!-- add gripper part -->
-    <!-- <link name="${prefix}gripper_link">
+    <!-- add gripper part start
+    ###################################################################-->
+    <!-- FOR THE GRIPPER (toogle gripper parts in):
+    ur_e_description/urdf/ur.transmission.xacro
+    ur_e_description/urdf/ur5e.urdf.xacro
+    ur_e_gazebo/launch/ur5.launch
+    ur5_e_moveit_config/config/ur5e.srdf -->
+    <link name="${prefix}gripper_link">
       <visual>
         <geometry>
@@ -430,6 +479,16 @@
       <parent link="${prefix}gripper_link" />
       <child link="${prefix}right_finger_link" />
-    </joint> -->
-    <!-- add gripper part -->
+    </joint>
+    <!-- add gripper part end ###################################################################-->
+    <!-- SENSOR CAMERA ON END EFFECTOR -->
+    <!-- Files to add sensor camera on end-effector:
+    ur.gazebo.xacro
+    ur5e.urdf.xacro -->
+    <xacro:include filename="$(find ur_e_description)/urdf/astra.urdf.xacro" />
+    <xacro:sensor_astra parent="ee_link" prefix="camera">
+      <origin xyz="0.06 -0.05 0.05"
+        rpy="${-pi} -0.0 0.0" />
+    </xacro:sensor_astra>
+    <!-- SENSOR CAMERA ON END EFFECTOR -->
     <xacro:ur_arm_transmission prefix="${prefix}" />
     <xacro:ur_arm_gazebo prefix="${prefix}" />

Commit message: update path to mesh

File: UR5/ur_e_description/urdf/astra.urdf.xacro (robot description, xacro)
@@ -56,5 +56,5 @@
         <origin xyz="0.0 0.0 -0.03" rpy="${pi/2} 0 0" />
         <geometry>
-          <mesh filename="package://t2rgb_description/meshes/sensors/astra2.dae" scale="1 1 1" />
+          <mesh filename="package://ur_e_description/meshes/sensors/astra2.dae" scale="1 1 1" />
         </geometry>
       </visual>
@@ -77,5 +77,5 @@
           <geometry> -->
             <!-- Use a slightly smaller scale than 1, so that when both models overlap its the rgb that appears.-->
-            <!-- <mesh filename="package://t2rgb_description/meshes/sensors/astra2.dae" scale="0.98 0.98 0.98" />
+            <!-- <mesh filename="package://ur_e_description/meshes/sensors/astra2.dae" scale="0.98 0.98 0.98" />
           </geometry>
         </visual> -->
