Commit message: add a velodine VLP 16 to the AGV

File: UR5/ur_e_description/urdf/moving_base_odom.urdf.xacro (robot description, xacro)
@@ -7,5 +7,5 @@
     <!-- VLP-16 -->
     <!-- velodyne -->
-    <!-- <xacro:arg name="gpu" default="false" />
+    <xacro:arg name="gpu" default="false" />
     <xacro:property name="gpu" value="$(arg gpu)" />
     <xacro:arg name="organize_cloud" default="false" />
@@ -14,6 +14,6 @@
     <xacro:VLP-16 parent="base_link_mb" name="velodyne" topic="/velodyne_points"
     organize_cloud="${organize_cloud}" hz="10" samples="440" gpu="${gpu}">
-        <origin xyz="-0.350 -0.250 0.850" rpy="0 0 0" />
-    </xacro:VLP-16> -->
+        <origin xyz="-0.350 0.050 0.850" rpy="0 0 0" />
+    </xacro:VLP-16>
     <!-- velodyne -->
     <!-- testing adding a sensor camera -->

Commit message: add intel realsense rgb-d D435  to the AGV

File: UR5/ur_e_description/urdf/moving_base_odom.urdf.xacro (robot description, xacro)
@@ -13,5 +13,5 @@
     <xacro:include filename="$(find velodyne_description)/urdf/VLP-16.urdf.xacro" />
     <xacro:VLP-16 parent="base_link_mb" name="velodyne" topic="/velodyne_points"
-    organize_cloud="${organize_cloud}" hz="10" samples="440" gpu="${gpu}">
+        organize_cloud="${organize_cloud}" hz="10" samples="440" gpu="${gpu}">
         <origin xyz="-0.350 0.050 0.850" rpy="0 0 0" />
     </xacro:VLP-16>
@@ -23,4 +23,27 @@
             rpy="0 0 3.14" />
     </xacro:sensor_astra>
+    <!-- testing adding a sensor camera -->
+    <!-- add intel realsense camera sensor -->
+    <xacro:arg name="realsense_enabled" default="$(optenv REALSENSE_ENABLED 1)" />
+    <xacro:arg name="realsense_topic" default="$(optenv REALSENSE_TOPIC realsense)" />
+    <xacro:arg name="realsense_prefix" default="$(optenv REALSENSE_PREFIX camera_realsense)" />
+    <xacro:arg name="realsense_parent" default="$(optenv REALSENSE_PARENT base_link_mb)" />
+    <xacro:arg name="realsense_xyz" default="$(optenv REALSENSE_XYZ 0.350 -0.180 0.850)" />
+    <xacro:arg name="realsense_rpy" default="$(optenv REALSENSE_RPY 0 0 0)" />
+    <material name="white">
+        <color rgba="1.0 1.0 1.0 1.0" />
+    </material>
+    <xacro:include filename="$(find ur_e_description)/urdf/realsense/intel_realsense.urdf.xacro" />
+    <xacro:if value="$(arg realsense_enabled)">
+        <link name="$(arg realsense_prefix)_realsense_mountpoint" />
+        <joint name="$(arg realsense_prefix)_realsense_mountpoint_joint" type="fixed">
+            <origin xyz="$(arg realsense_xyz)" rpy="$(arg realsense_rpy)" />
+            <parent link="$(arg realsense_parent)" />
+            <child link="$(arg realsense_prefix)_realsense_mountpoint" />
+        </joint>
+        <xacro:intel_realsense_mount prefix="$(arg realsense_prefix)" topic="$(arg realsense_topic)"
+            parent_link="$(arg realsense_prefix)_realsense_mountpoint" />
+    </xacro:if>
+    <!-- add intel realsense sensor -->
     <link name="base_footprint" />
     <joint name="base_joint" type="fixed">
@@ -86,5 +109,5 @@
             <origin xyz="0 0 0" />
             <mass value="2.637" />
-            <inertia  ixx="0.02467" ixy="0" ixz="0" iyy="0.04411" iyz="0" izz="0.02467" />
+            <inertia ixx="0.02467" ixy="0" ixz="0" iyy="0.04411" iyz="0" izz="0.02467" />
         </inertial>
     </link>
@@ -113,5 +136,5 @@
             <origin xyz="0 0 0" />
             <mass value="2.637" />
-            <inertia  ixx="0.02467" ixy="0" ixz="0" iyy="0.04411" iyz="0" izz="0.02467" />
+            <inertia ixx="0.02467" ixy="0" ixz="0" iyy="0.04411" iyz="0" izz="0.02467" />
         </inertial>
     </link>

Commit message: add realsense l515 with infra to the mobile manipulator

File: UR5/ur_e_description/urdf/moving_base_odom.urdf.xacro (robot description, xacro)
@@ -24,5 +24,5 @@
     </xacro:sensor_astra>
     <!-- testing adding a sensor camera -->
-    <!-- add intel realsense camera sensor -->
+    <!-- add intel realsense camera d415 sensor -->
     <xacro:arg name="realsense_enabled" default="$(optenv REALSENSE_ENABLED 1)" />
     <xacro:arg name="realsense_topic" default="$(optenv REALSENSE_TOPIC realsense)" />
@@ -45,5 +45,14 @@
             parent_link="$(arg realsense_prefix)_realsense_mountpoint" />
     </xacro:if>
-    <!-- add intel realsense sensor -->
+    <!-- add intel realsense d415 sensor -->
+    <!-- add intel realsense l515 camera -->
+    <xacro:arg name="use_nominal_extrinsics" default="false"/>
+    <xacro:arg name="add_plug" default="false" />
+    <xacro:arg name="use_mesh" default="true" />
+    <xacro:include filename="$(find ur_e_description)/urdf/realsense/_l515.urdf.xacro" />
+    <xacro:sensor_l515 parent="base_link_mb" use_nominal_extrinsics="$(arg use_nominal_extrinsics)" add_plug="$(arg add_plug)" use_mesh="$(arg use_mesh)">
+      <origin xyz="0.350 0.180 0.850" rpy="0 0 0"/>
+    </xacro:sensor_l515>
+    <!-- add intel realsense l515 camera -->
     <link name="base_footprint" />
     <joint name="base_joint" type="fixed">

Commit message: add intel realsense t265 to agv - odom didn't work properly, gazebo plugin connect to world frame and not to odom

File: UR5/ur_e_description/urdf/moving_base_odom.urdf.xacro (robot description, xacro)
@@ -47,12 +47,19 @@
     <!-- add intel realsense d415 sensor -->
     <!-- add intel realsense l515 camera -->
-    <xacro:arg name="use_nominal_extrinsics" default="false"/>
+    <xacro:arg name="use_nominal_extrinsics" default="false" />
     <xacro:arg name="add_plug" default="false" />
     <xacro:arg name="use_mesh" default="true" />
     <xacro:include filename="$(find ur_e_description)/urdf/realsense/_l515.urdf.xacro" />
-    <xacro:sensor_l515 parent="base_link_mb" use_nominal_extrinsics="$(arg use_nominal_extrinsics)" add_plug="$(arg add_plug)" use_mesh="$(arg use_mesh)">
-      <origin xyz="0.350 0.180 0.850" rpy="0 0 0"/>
+    <xacro:sensor_l515 parent="base_link_mb" use_nominal_extrinsics="$(arg use_nominal_extrinsics)"
+        add_plug="$(arg add_plug)" use_mesh="$(arg use_mesh)">
+        <origin xyz="0.350 0.180 0.850" rpy="0 0 0" />
     </xacro:sensor_l515>
     <!-- add intel realsense l515 camera -->
+    <!-- add intel realsense t265 -->
+    <xacro:include filename="$(find realsense_ros_gazebo)/xacro/tracker.xacro" />
+    <xacro:realsense_T265 sensor_name="camera_t265" parent_link="base_link_mb" rate="30.0">
+        <origin rpy="0 0 0" xyz="0.350 0.060 0.860" />
+    </xacro:realsense_T265>
+    <!-- add intel realsense t265 -->
     <link name="base_footprint" />
     <joint name="base_joint" type="fixed">

Commit message: positioning the manipulator, dimensions estimated with a measuring tape

File: UR5/ur_e_description/urdf/moving_base_odom.urdf.xacro (robot description, xacro)
@@ -11,23 +11,23 @@
     </xacro:sensor_astra> -->
     <!-- add intel realsense camera d415 sensor -->
-    <xacro:arg name="realsense_enabled" default="$(optenv REALSENSE_ENABLED 1)" />
-    <xacro:arg name="realsense_topic" default="$(optenv REALSENSE_TOPIC realsense)" />
-    <xacro:arg name="realsense_prefix" default="$(optenv REALSENSE_PREFIX camera_realsense)" />
-    <xacro:arg name="realsense_parent" default="$(optenv REALSENSE_PARENT base_link_mb)" />
-    <xacro:arg name="realsense_xyz" default="$(optenv REALSENSE_XYZ -0.350 0.180 0.870)" />
-    <xacro:arg name="realsense_rpy" default="$(optenv REALSENSE_RPY 0 0 3.14)" />
+    <xacro:arg name="realsense_AGV_enabled" default="$(optenv REALSENSE_AGV_ENABLED 1)" />
+    <xacro:arg name="realsense_AGV_topic" default="$(optenv REALSENSE_AGV_TOPIC AGV_realsense)" />
+    <xacro:arg name="realsense_AGV_prefix" default="$(optenv REALSENSE_AGV_PREFIX AGV_camera_realsense)" />
+    <xacro:arg name="realsense_AGV_parent" default="$(optenv REALSENSE_AGV_PARENT base_link_mb)" />
+    <xacro:arg name="realsense_AGV_xyz" default="$(optenv REALSENSE_AGV_XYZ -0.380 0.250 0.80)" />
+    <xacro:arg name="realsense_AGV_rpy" default="$(optenv REALSENSE_AGV_RPY 0 0 3.14)" />
     <material name="white">
         <color rgba="1.0 1.0 1.0 1.0" />
     </material>
     <xacro:include filename="$(find ur_e_description)/urdf/realsense/intel_realsense.urdf.xacro" />
-    <xacro:if value="$(arg realsense_enabled)">
-        <link name="$(arg realsense_prefix)_realsense_mountpoint" />
-        <joint name="$(arg realsense_prefix)_realsense_mountpoint_joint" type="fixed">
-            <origin xyz="$(arg realsense_xyz)" rpy="$(arg realsense_rpy)" />
-            <parent link="$(arg realsense_parent)" />
-            <child link="$(arg realsense_prefix)_realsense_mountpoint" />
+    <xacro:if value="$(arg realsense_AGV_enabled)">
+        <link name="$(arg realsense_AGV_prefix)_realsense_mountpoint" />
+        <joint name="$(arg realsense_AGV_prefix)_realsense_mountpoint_joint" type="fixed">
+            <origin xyz="$(arg realsense_AGV_xyz)" rpy="$(arg realsense_AGV_rpy)" />
+            <parent link="$(arg realsense_AGV_parent)" />
+            <child link="$(arg realsense_AGV_prefix)_realsense_mountpoint" />
         </joint>
-        <xacro:intel_realsense_mount prefix="$(arg realsense_prefix)" topic="$(arg realsense_topic)"
-            parent_link="$(arg realsense_prefix)_realsense_mountpoint" />
+        <xacro:intel_realsense_mount prefix="$(arg realsense_AGV_prefix)" topic="$(arg realsense_AGV_topic)"
+            parent_link="$(arg realsense_AGV_prefix)_realsense_mountpoint" />
     </xacro:if>
     <!-- add intel realsense d415 sensor -->
@@ -40,17 +40,18 @@
     <link name="base_link_mb">
         <visual>
-            <origin xyz="-0.43 -0.33 0.03" rpy="1.57 0 1.57" />
+            <origin xyz="-0.0 -0.0 0.47" rpy="0 0 0" />
             <geometry>
                 <!-- <box size="0.900 0.600 0.770" /> -->
                 <!-- <box size="0.900 0.650 0.770" /> -->
-                <mesh filename="package://ur_e_description/meshes/moving_base/moving_base.STL"
-                    scale="0.001 0.001 0.001" />
+                <box size="0.920 0.670 0.630" />
+                <!-- <mesh filename="package://ur_e_description/meshes/moving_base/moving_base.STL"
+                    scale="0.001 0.001 0.001" /> -->
             </geometry>
             <material name="light_black" />
         </visual>
         <collision>
-            <origin xyz="0 0 0.459" rpy="0 0 0" />
-            <geometry>
-                <box size="0.900 0.600 0.770" />
+            <origin xyz="0 0 0.46" rpy="0 0 0" />
+            <geometry>
+                <box size="0.920 0.670 0.780" />
             </geometry>
         </collision>

Commit message: update realsense camera visuals

File: UR5/ur_e_description/urdf/moving_base_odom.urdf.xacro (robot description, xacro)
@@ -4,10 +4,4 @@
     <xacro:include filename="$(find ur_e_description)/urdf/moving_base_odom.gazebo.xacro" />
     <xacro:property name="M_PI" value="3.1415926535897931" />
-    <!-- testing adding a sensor camera -->
-    <!-- <xacro:include filename="$(find ur_e_description)/urdf/astra.urdf.xacro" />
-    <xacro:sensor_astra parent="base_link_mb" prefix="camera_mb">
-        <origin xyz="-0.350 0.180 0.870"
-            rpy="0 0 3.14" />
-    </xacro:sensor_astra> -->
     <!-- add intel realsense camera d415 sensor -->
     <xacro:arg name="realsense_AGV_enabled" default="$(optenv REALSENSE_AGV_ENABLED 1)" />

File: UR5/ur_e_description/urdf/realsense/intel_realsense.urdf.xacro (robot description, xacro)
@@ -80,5 +80,5 @@
           <mesh filename="package://realsense2_description/meshes/d415.stl" />
         </geometry>
-        <material name="white" />
+        <material name="light_black" />
       </visual>
     </link>

File: UR5/ur_e_description/urdf/ur5e.urdf.xacro (robot description, xacro)
@@ -483,13 +483,4 @@
     </joint>
     <!-- add gripper part end ###################################################################-->
-    <!-- SENSOR CAMERA ON END EFFECTOR -->
-    <!-- Files to add sensor camera on end-effector:
-    ur.gazebo.xacro
-    ur5e.urdf.xacro -->
-    <!-- <xacro:include filename="$(find ur_e_description)/urdf/astra.urdf.xacro" />
-    <xacro:sensor_astra parent="ee_link" prefix="camera">
-      <origin xyz="0.06 -0.05 0.05"
-        rpy="${-pi} -0.0 0.0" />
-    </xacro:sensor_astra> -->
     <!-- add intel realsense camera d415 sensor -->
     <xacro:arg name="realsense_EE_enabled" default="$(optenv REALSENSE_EE_ENABLED 1)" />
@@ -499,7 +490,4 @@
     <xacro:arg name="realsense_EE_xyz" default="$(optenv REALSENSE_EE_XYZ 0.095 0.000 -0.075)" />
     <xacro:arg name="realsense_EE_rpy" default="$(optenv REALSENSE_EE_RPY -3.14 0.0 1.57)" />
-    <!-- <material name="white">
-      <color rgba="1.0 1.0 1.0 1.0" />
-    </material> -->
     <xacro:include filename="$(find ur_e_description)/urdf/realsense/intel_realsense.urdf.xacro" />
     <xacro:if value="$(arg realsense_EE_enabled)">

Commit message: remove gripper and modify the AGV

File: UR5/ur_e_description/urdf/moving_base_odom.urdf.xacro (robot description, xacro)
@@ -9,5 +9,5 @@
     <xacro:arg name="realsense_AGV_prefix" default="$(optenv REALSENSE_AGV_PREFIX AGV_camera_realsense)" />
     <xacro:arg name="realsense_AGV_parent" default="$(optenv REALSENSE_AGV_PARENT base_link_mb)" />
-    <xacro:arg name="realsense_AGV_xyz" default="$(optenv REALSENSE_AGV_XYZ -0.380 0.250 0.80)" />
+    <xacro:arg name="realsense_AGV_xyz" default="$(optenv REALSENSE_AGV_XYZ -0.380 0.250 0.79)" />
     <xacro:arg name="realsense_AGV_rpy" default="$(optenv REALSENSE_AGV_RPY 0 0 3.14)" />
     <material name="white">
@@ -34,18 +34,15 @@
     <link name="base_link_mb">
         <visual>
-            <origin xyz="-0.0 -0.0 0.47" rpy="0 0 0" />
-            <geometry>
-                <!-- <box size="0.900 0.600 0.770" /> -->
-                <!-- <box size="0.900 0.650 0.770" /> -->
+            <origin xyz="-0.46 0.335 0.06" rpy="1.57 0 0" />
+            <geometry>
+                <!-- <box size="0.920 0.670 0.630" /> -->
+                <mesh filename="package://ur_e_description/meshes/moving_base/AGV.STL" scale="0.01 0.01 0.01" />
+            </geometry>
+            <material name="light_black" />
+        </visual>
+        <collision>
+            <origin xyz="0 0 0.47" rpy="0 0 0" />
+            <geometry>
                 <box size="0.920 0.670 0.630" />
-                <!-- <mesh filename="package://ur_e_description/meshes/moving_base/moving_base.STL"
-                    scale="0.001 0.001 0.001" /> -->
-            </geometry>
-            <material name="light_black" />
-        </visual>
-        <collision>
-            <origin xyz="0 0 0.46" rpy="0 0 0" />
-            <geometry>
-                <box size="0.920 0.670 0.780" />
             </geometry>
         </collision>
@@ -246,5 +243,5 @@
     </joint>
     <link name="imu_link" />
-    <!-- ROMEVED FOR NOW - JORGE FEB 2023 -->
+    <!-- ROMEVED FOR NOW - JORGE FEB 2023 need check real position in the robot -->
     <!-- lidar sensor front -->
     <!-- <joint name="scan_joint_front" type="fixed">

File: UR5/ur_e_description/urdf/ur.transmission.xacro (robot description, xacro)
@@ -63,5 +63,5 @@
     ur5_e_moveit_config/config/ur5e.srdf
     -->
-    <transmission name="${prefix}left_finger_trans">
+    <!-- <transmission name="${prefix}left_finger_trans">
       <type>transmission_interface/SimpleTransmission</type>
       <joint name="${prefix}left_finger_joint">
@@ -82,5 +82,5 @@
         <mechanicalReduction>1</mechanicalReduction>
       </actuator>
-    </transmission>
+    </transmission> -->
     <!-- add gripper part end -->
   </xacro:macro>

File: UR5/ur_e_description/urdf/ur5e.urdf.xacro (robot description, xacro)
@@ -393,5 +393,5 @@
     ur_e_gazebo/launch/ur5.launch
     ur5_e_moveit_config/config/ur5e.srdf -->
-    <link name="${prefix}gripper_link">
+    <!-- <link name="${prefix}gripper_link">
       <visual>
         <geometry>
@@ -481,10 +481,44 @@
       <parent link="${prefix}gripper_link" />
       <child link="${prefix}right_finger_link" />
-    </joint>
+    </joint> -->
     <!-- add gripper part end ###################################################################-->
+    <!-- add camera support -->
+    <link name="${prefix}ee_camera_support_link">
+      <visual>
+        <geometry>
+          <box size="0.185 0.03 0.03" />
+        </geometry>
+        <material name="LightGrey">
+          <color rgba="0.7 0.7 0.7 1.0" />
+        </material>
+        <origin xyz="0 0 0" rpy="0 0 0" />
+      </visual>
+    </link>
+    <joint name="${prefix}ee_camera_support_joint" type="fixed">
+      <origin xyz="0.095 0 0" rpy="0 0 0" />
+      <parent link="${prefix}ee_link" />
+      <child link="${prefix}ee_camera_support_link" />
+    </joint>
+    <link name="${prefix}ee_camera_support_small_link">
+      <visual>
+        <geometry>
+          <box size="0.02 0.02 0.065" />
+        </geometry>
+        <material name="LightGrey">
+          <color rgba="0.7 0.7 0.7 1.0" />
+        </material>
+        <origin xyz="0 0 0" rpy="0 0 0" />
+      </visual>
+    </link>
+    <joint name="${prefix}ee_camera_support_small_joint" type="fixed">
+      <origin xyz="0 0 -0.04" rpy="0 0 0" />
+      <parent link="${prefix}ee_camera_support_link" />
+      <child link="${prefix}ee_camera_support_small_link" />
+    </joint>
     <!-- add intel realsense camera d415 sensor -->
     <xacro:arg name="realsense_EE_enabled" default="$(optenv REALSENSE_EE_ENABLED 1)" />
     <xacro:arg name="realsense_EE_topic" default="$(optenv REALSENSE_EE_TOPIC EE_realsense)" />
-    <xacro:arg name="realsense_EE_prefix" default="$(optenv REALSENSE_EE_PREFIX EE_camera_realsense)" />
+    <xacro:arg name="realsense_EE_prefix"
+      default="$(optenv REALSENSE_EE_PREFIX EE_camera_realsense)" />
     <xacro:arg name="realsense_EE_parent" default="$(optenv REALSENSE_EE_PARENT ee_link)" />
     <xacro:arg name="realsense_EE_xyz" default="$(optenv REALSENSE_EE_XYZ 0.095 0.000 -0.075)" />
@@ -498,5 +532,6 @@
         <child link="$(arg realsense_EE_prefix)_realsense_mountpoint" />
       </joint>
-      <xacro:intel_realsense_mount prefix="$(arg realsense_EE_prefix)" topic="$(arg realsense_EE_topic)"
+      <xacro:intel_realsense_mount prefix="$(arg realsense_EE_prefix)"
+        topic="$(arg realsense_EE_topic)"
         parent_link="$(arg realsense_EE_prefix)_realsense_mountpoint" />
     </xacro:if>

Commit message: update cam

File: UR5/ur_e_description/urdf/moving_base_odom.urdf.xacro (robot description, xacro)
@@ -9,8 +9,8 @@
     <xacro:arg name="realsense_AGV_prefix" default="$(optenv REALSENSE_AGV_PREFIX AGV_camera_realsense)" />
     <xacro:arg name="realsense_AGV_parent" default="$(optenv REALSENSE_AGV_PARENT base_link_mb)" />
-    <xacro:arg name="realsense_AGV_xyz" default="$(optenv REALSENSE_AGV_XYZ -0.380 0.250 0.79)" />
-    <xacro:arg name="realsense_AGV_rpy" default="$(optenv REALSENSE_AGV_RPY 0 0 3.14)" />
-    <material name="white">
-        <color rgba="1.0 1.0 1.0 1.0" />
+    <xacro:arg name="realsense_AGV_xyz" default="$(optenv REALSENSE_AGV_XYZ 0.400 -0.250 0.79)" />
+    <xacro:arg name="realsense_AGV_rpy" default="$(optenv REALSENSE_AGV_RPY 0 -0.2 0)" />
+    <material name="realsense_color">
+        <color rgba="0.1 0.1 1.0 1.0" />
     </material>
     <xacro:include filename="$(find ur_e_description)/urdf/realsense/intel_realsense.urdf.xacro" />

File: UR5/ur_e_description/urdf/realsense/intel_realsense.urdf.xacro (robot description, xacro)
@@ -80,5 +80,5 @@
           <mesh filename="package://realsense2_description/meshes/d415.stl" />
         </geometry>
-        <material name="light_black" />
+        <material name="realsense_color" />
       </visual>
     </link>

Commit message: adapt xacro to match zau real robot

File: UR5/ur_e_description/urdf/moving_base_odom.urdf.xacro (robot description, xacro)
@@ -5,7 +5,14 @@
     <xacro:property name="M_PI" value="3.1415926535897931" />
     <!-- add intel realsense camera d415 sensor -->
+    <!-- <xacro:include
+        filename="$(find ur_e_description)/urdf/realsense/intel_realsense_inesctec.urdf.xacro" />
+    <xacro:sensor_d415 parent="base_link_mb" use_nominal_extrinsics="true" name="camera_mb">
+        <origin xyz="0.400 -0.250 0.79"
+            rpy="0.0 -0.2 0.0" />
+    </xacro:sensor_d415> -->
     <xacro:arg name="realsense_AGV_enabled" default="$(optenv REALSENSE_AGV_ENABLED 1)" />
     <xacro:arg name="realsense_AGV_topic" default="$(optenv REALSENSE_AGV_TOPIC AGV_realsense)" />
-    <xacro:arg name="realsense_AGV_prefix" default="$(optenv REALSENSE_AGV_PREFIX AGV_camera_realsense)" />
+    <xacro:arg name="realsense_AGV_prefix" default="$(optenv REALSENSE_AGV_PREFIX
+    AGV_camera_realsense)" />
     <xacro:arg name="realsense_AGV_parent" default="$(optenv REALSENSE_AGV_PARENT base_link_mb)" />
     <xacro:arg name="realsense_AGV_xyz" default="$(optenv REALSENSE_AGV_XYZ 0.400 -0.250 0.79)" />
@@ -22,5 +29,6 @@
             <child link="$(arg realsense_AGV_prefix)_realsense_mountpoint" />
         </joint>
-        <xacro:intel_realsense_mount prefix="$(arg realsense_AGV_prefix)" topic="$(arg realsense_AGV_topic)"
+        <xacro:intel_realsense_mount prefix="$(arg realsense_AGV_prefix)" topic="$(arg
+    realsense_AGV_topic)"
             parent_link="$(arg realsense_AGV_prefix)_realsense_mountpoint" />
     </xacro:if>
@@ -37,5 +45,6 @@
             <geometry>
                 <!-- <box size="0.920 0.670 0.630" /> -->
-                <mesh filename="package://ur_e_description/meshes/moving_base/AGV.STL" scale="0.01 0.01 0.01" />
+                <mesh filename="package://ur_e_description/meshes/moving_base/AGV.STL"
+                    scale="0.01 0.01 0.01" />
             </geometry>
             <material name="light_black" />

File: UR5/ur_e_description/urdf/ur5e.urdf.xacro (robot description, xacro)
@@ -517,5 +517,11 @@
     </joint>
     <!-- add intel realsense camera d415 sensor -->
-    <xacro:arg name="realsense_EE_enabled" default="$(optenv REALSENSE_EE_ENABLED 1)" />
+    <xacro:include
+      filename="$(find ur_e_description)/urdf/realsense/intel_realsense_inesctec.urdf.xacro" />
+    <xacro:sensor_d415 parent="ee_link" use_nominal_extrinsics="true">
+      <origin xyz="0.095 0.000 -0.075"
+        rpy="-3.14 0.0 1.57" />
+    </xacro:sensor_d415>
+    <!-- <xacro:arg name="realsense_EE_enabled" default="$(optenv REALSENSE_EE_ENABLED 1)" />
     <xacro:arg name="realsense_EE_topic" default="$(optenv REALSENSE_EE_TOPIC EE_realsense)" />
     <xacro:arg name="realsense_EE_prefix"
@@ -535,5 +541,5 @@
         topic="$(arg realsense_EE_topic)"
         parent_link="$(arg realsense_EE_prefix)_realsense_mountpoint" />
-    </xacro:if>
+    </xacro:if> -->
     <!-- add intel realsense d415 sensor -->
     <!-- SENSOR CAMERA ON END EFFECTOR -->
