Commit message: add functionalities to main launch

File: UR5/ur_e_description/urdf/ur5e.urdf.xacro (robot description, xacro)
@@ -12,5 +12,4 @@
     <parent link="base_link_mb" />
     <child link="base_link" />
-    <!-- <origin xyz="0.0 0.0 0.771" rpy="0.0 0.0 0.0" /> -->
     <origin xyz="-0.296 -0.1688 0.826" rpy="0.0 0.0 0.0" />
   </joint>

Commit message: remove unused links from UR5

File: UR5/ur_e_description/urdf/ur5e.urdf.xacro (robot description, xacro)
@@ -495,22 +495,23 @@
     <xacro:ur_arm_transmission prefix="${prefix}" />
     <xacro:ur_arm_gazebo prefix="${prefix}" />
+    <!-- This link is not needed i.m.o.- Jorge 17/03/2023 -->
     <!-- ROS base_link to UR 'Base' Coordinates transform -->
-    <link name="${prefix}base" />
-    <joint name="${prefix}base_link-base_fixed_joint" type="fixed">
+    <!-- <link name="${prefix}base" />
+    <joint name="${prefix}base_link-base_fixed_joint" type="fixed"> -->
       <!-- NOTE: this rotation is only needed as long as base_link itself is
                  not corrected wrt the real robot (ie: rotated over 180
                  degrees)
       -->
-      <origin xyz="0 0 0" rpy="0 0 ${-pi}" />
+      <!-- <origin xyz="0 0 0" rpy="0 0 ${-pi}" />
       <parent link="${prefix}base_link" />
       <child link="${prefix}base" />
-    </joint>
+    </joint> -->
     <!-- Frame coincident with all-zeros TCP on UR controller -->
-    <link name="${prefix}tool0" />
+    <!-- <link name="${prefix}tool0" />
     <joint name="${prefix}wrist_3_link-tool0_fixed_joint" type="fixed">
       <origin xyz="0 ${wrist_3_length} 0" rpy="${pi/-2.0} 0 0" />
       <parent link="${prefix}wrist_3_link" />
       <child link="${prefix}tool0" />
-    </joint>
+    </joint> -->
   </xacro:macro>
 </robot>

Commit message: remove unused links

File: UR5/ur_e_description/urdf/ur5e.urdf.xacro (robot description, xacro)
@@ -496,21 +496,21 @@
     <xacro:ur_arm_gazebo prefix="${prefix}" />
     <!-- ROS base_link to UR 'Base' Coordinates transform -->
-    <link name="${prefix}base" />
-    <joint name="${prefix}base_link-base_fixed_joint" type="fixed">
+    <!-- <link name="${prefix}base" />
+    <joint name="${prefix}base_link-base_fixed_joint" type="fixed"> -->
       <!-- NOTE: this rotation is only needed as long as base_link itself is
                  not corrected wrt the real robot (ie: rotated over 180
                  degrees)
       -->
-      <origin xyz="0 0 0" rpy="0 0 ${-pi}" />
+      <!-- <origin xyz="0 0 0" rpy="0 0 ${-pi}" />
       <parent link="${prefix}base_link" />
       <child link="${prefix}base" />
-    </joint>
+    </joint> -->
     <!-- Frame coincident with all-zeros TCP on UR controller -->
-    <link name="${prefix}tool0" />
+    <!-- <link name="${prefix}tool0" />
     <joint name="${prefix}wrist_3_link-tool0_fixed_joint" type="fixed">
       <origin xyz="0 ${wrist_3_length} 0" rpy="${pi/-2.0} 0 0" />
       <parent link="${prefix}wrist_3_link" />
       <child link="${prefix}tool0" />
-    </joint>
+    </joint> -->
   </xacro:macro>
 </robot>

Commit message: remove gripper tags

File: UR5/ur_e_description/urdf/ur5e.urdf.xacro (robot description, xacro)
@@ -387,101 +387,4 @@
       </collision>
     </link>
-    <!-- add gripper part start
-    ###################################################################-->
-    <!-- FOR THE GRIPPER (toogle gripper parts in):
-    ur_e_description/urdf/ur.transmission.xacro
-    ur_e_description/urdf/ur5e.urdf.xacro
-    ur_e_gazebo/launch/ur5.launch
-    ur5_e_moveit_config/config/ur5e.srdf -->
-    <!-- <link name="${prefix}gripper_link">
-      <visual>
-        <geometry>
-          <mesh filename="package://ur_e_description/meshes/ur5e/visual/weiss-mount.dae" />
-        </geometry>
-        <origin xyz="-0.071 0 0" rpy="${pi/-2.0} 0 ${pi/-2.0}" />
-      </visual>
-      <visual>
-        <geometry>
-          <mesh filename="package://ur_e_description/meshes/ur5e/visual/weiss-cg.dae" />
-        </geometry>
-        <origin xyz="-0.07 0 0" rpy="${pi/-2.0} 0 ${pi/-2.0}" />
-      </visual>
-      <collision>
-        <geometry>
-          <box size="0.071 0.105 0.06" />
-        </geometry>
-        <origin rpy="0 0 0" xyz="${-0.071*0.5} 0 0" />
-      </collision>
-      <inertial>
-        <origin xyz="0 0 0" rpy="0 0 0" />
-        <mass value="1.7" />
-        <inertia ixx="1.0" ixy="0.0" ixz="0.0" iyy="1.0" iyz="0.0" izz="1.0" />
-      </inertial>
-      <dynamics damping="0.0" friction="0.0" />
-    </link>
-    <joint name="${prefix}gripper_fixed_joint" type="fixed">
-      <origin xyz="0.071 0 0" rpy="0 0 0" />
-      <parent link="${prefix}ee_link" />
-      <child link="${prefix}gripper_link" />
-    </joint>
-    <joint name="${prefix}left_finger_joint" type="prismatic">
-      <origin xyz="0 0.02 0" rpy="0 0 0" />
-      <axis xyz="0 1 0" />
-      <limit lower="0" upper="0.03078" effort="100" velocity="0.05" />
-      <parent link="${prefix}gripper_link" />
-      <child link="${prefix}left_finger_link" />
-    </joint>
-    <link name="${prefix}left_finger_link">
-      <visual>
-        <geometry>
-          <box size="0.095 0.02 0.02" />
-        </geometry>
-        <material name="LightGrey">
-          <color rgba="0.7 0.7 0.7 1.0" />
-        </material>
-        <origin xyz="${0.095*0.5} 0 0" rpy="0 0 0" />
-      </visual>
-      <collision>
-        <geometry>
-          <box size="0.095 0.02 0.02" />
-        </geometry>
-        <origin xyz="${0.095*0.5} 0 0" rpy="0 0 0" />
-      </collision>
-      <inertial>
-        <origin xyz="0 0 0" rpy="0 0 0" />
-        <mass value="0.1" />
-        <inertia ixx="1.0" ixy="0.0" ixz="0.0" iyy="1.0" iyz="0.0" izz="1.0" />
-      </inertial>
-    </link>
-    <link name="${prefix}right_finger_link">
-      <visual>
-        <geometry>
-          <box size="0.095 0.02 0.02" />
-        </geometry>
-        <material name="LightGrey">
-          <color rgba="0.7 0.7 0.7 1.0" />
-        </material>
-        <origin xyz="${0.095*0.5} 0 0" rpy="0 0 0" />
-      </visual>
-      <collision>
-        <geometry>
-          <box size="0.095 0.02 0.02" />
-        </geometry>
-        <origin xyz="${0.095*0.5} 0 0" rpy="0 0 0" />
-      </collision>
-      <inertial>
-        <origin xyz="0 0 0" rpy="0 0 0" />
-        <mass value="0.1" />
-        <inertia ixx="1.0" ixy="0.0" ixz="0.0" iyy="1.0" iyz="0.0" izz="1.0" />
-      </inertial>
-    </link>
-    <joint name="${prefix}right_finger_joint" type="prismatic">
-      <origin xyz="0 -0.02 0" rpy="0 0 0" />
-      <axis xyz="0 -1 0" />
-      <limit lower="0" upper="0.03078" effort="100" velocity="0.05" />
-      <parent link="${prefix}gripper_link" />
-      <child link="${prefix}right_finger_link" />
-    </joint> -->
-    <!-- add gripper part end ###################################################################-->
     <!-- SENSOR CAMERA ON END EFFECTOR -->
     <!-- Files to add sensor camera on end-effector:
@@ -521,5 +424,5 @@
     </joint>
     <xacro:include filename="$(find ur_e_description)/urdf/realsense/intel_realsense.urdf.xacro" />
-    <xacro:sensor_d415 parent="ee_link" use_nominal_extrinsics="true">
+    <xacro:sensor_d415 parent="ee_link" use_nominal_extrinsics="true" gazebo_plugin="true">
       <origin xyz="0.095 0.000 -0.075"
         rpy="-3.14 0.0 1.57" />

File: UR5/ur_e_description/urdf/ur5e_joint_limited_robot.urdf.xacro (robot description, xacro)
@@ -15,47 +15,3 @@
     wrist_3_lower_limit="${-pi}" wrist_3_upper_limit="${pi}"
   />
-  <!-- THIS PART WAS MOVED TO UR5E.URDF.XACRO  -->
-  <!-- place robot on moving base -->
-  <!-- <xacro:include filename="$(find ur_e_description)/urdf/moving_base.urdf.xacro" />
-  <joint name="moving_base_to_ur5e" type="fixed">
-    <parent link="base_link_mb" />
-    <child link="base_link" />
-    <origin xyz="-0.296 -0.1688 0.826" rpy="0.0 0.0 0.0"/>
-  </joint> -->
-  <!-- THIS PART WAS MOVED TO UR5E.URDF.XACRO  -->
-  <!-- <link name="base_footprint" /> -->
-  <!-- initial robot pose on world - FROM ORIGINAL FILE -->
-  <!-- toogle this part to move the AGV in odom -->
-  <!-- <link name="world" />
-  <joint name="world_joint" type="fixed">
-    <parent link="world" />
-    <child link="base_link_mb" />
-    <origin xyz="0.0 0.0 0.0" rpy="0.0 0.0 0.0" />
-  </joint> -->
-  <!-- initial robot pose on world - FROM ORIGINAL FILE -->
-  <!-- THIS PART WAS FOR TEST ONLY - JORGE -->
-  <!-- put robot on table -->
-  <!-- <xacro:property name="M_PI" value="3.1415926535897931" /> -->
-  <!-- Tables properties-->
-  <!-- <xacro:property name="table_height" value="0.795" />
-  <xacro:property name="table_width" value=".9" />
-  <xacro:property name="table_lenght" value="0.9" />
-  <xacro:property name="table_tabletop_thickness" value="0.015" />
-  <xacro:property name="table_leg_radius" value="0.02" /> -->
-  <!-- Scene objets-->
-  <!-- <xacro:include filename="$(find ur_e_description)/urdf/properties.xacro" />
-  <xacro:include filename="$(find ur_e_description)/urdf/table.macro.xacro" /> -->
-  <!-- Place table 1 in the scene-->
-  <!-- <xacro:table_macro name="table" parent="world" width="${table_width}"
-    lenght="${table_lenght}" height="${table_height}"
-    tabletop_thickness="${table_tabletop_thickness}" leg_radius="${table_leg_radius}">
-    <origin xyz="-1 0 0" rpy="0 0 1.57" />
-  </xacro:table_macro> -->
-  <!--  Place robot on top of the table -->
-  <!-- <joint name="tabletop_table_to_ur5e" type="fixed">
-    <parent link="tabletop_table" />
-    <child link="base_link" />
-    <origin xyz="0.0 0.0 0.001" rpy="0.0 0.0 0.0" />
-  </joint> -->
-  <!-- THIS PART WAS FOR TEST ONLY - JORGE -->
 </robot>

Commit message: update camera position

File: UR5/ur_e_description/urdf/ur5e.urdf.xacro (robot description, xacro)
@@ -9,5 +9,5 @@
   <!-- <xacro:include filename="$(find ur_e_description)/urdf/moving_base_odom.urdf.xacro" />  -->
   <!-- *************THIS IS THE TRANSFORMATION TO BE CALIBRATED************* -->
-<!-- <link name="world"/> -->
+  <!-- <link name="world"/> -->
   <!-- <joint name="moving_base_to_ur5e" type="fixed">
     <parent link="world" />
@@ -403,5 +403,5 @@
     </link>
     <joint name="${prefix}ee_camera_support_joint" type="fixed">
-      <origin xyz="0.095 0 0" rpy="0 0 0" />
+      <origin xyz="0.095 0 0" rpy="${-pi/2+pi/4} 0 0" />
       <parent link="${prefix}ee_link" />
       <child link="${prefix}ee_camera_support_link" />
@@ -424,7 +424,7 @@
     </joint>
     <xacro:include filename="$(find ur_e_description)/urdf/realsense/intel_realsense.urdf.xacro" />
-    <xacro:sensor_d415 parent="ee_link" use_nominal_extrinsics="true" >
-      <origin xyz="0.095 0.000 -0.075"
-        rpy="-3.14 0.0 1.57" />
+    <xacro:sensor_d415 parent="${prefix}ee_link" use_nominal_extrinsics="true">
+      <origin xyz="0.095 -0.053 -0.053"
+        rpy="3.139 0.785 1.570" />
     </xacro:sensor_d415>
     <!-- SENSOR CAMERA ON END EFFECTOR -->
@@ -434,9 +434,9 @@
     <!-- <link name="${prefix}base" />
     <joint name="${prefix}base_link-base_fixed_joint" type="fixed"> -->
-      <!-- NOTE: this rotation is only needed as long as base_link itself is
+    <!-- NOTE: this rotation is only needed as long as base_link itself is
                  not corrected wrt the real robot (ie: rotated over 180
                  degrees)
       -->
-      <!-- <origin xyz="0 0 0" rpy="0 0 ${-pi}" />
+    <!-- <origin xyz="0 0 0" rpy="0 0 ${-pi}" />
       <parent link="${prefix}base_link" />
       <child link="${prefix}base" />

Commit message: Transforms missing

File: UR5/ur_e_description/urdf/ur5e.urdf.xacro (robot description, xacro)
@@ -1,4 +1,11 @@
 <?xml version="1.0"?>
 <robot xmlns:xacro="http://ros.org/wiki/xacro">
+  <!-- TRANSFORMATIONS MISSING ON REAL ZAU BOT
+  AGV TO ARM
+  <origin xyz="-0.295 0.0 0.780" rpy="0.0 0.0 0.0" />
+  CAMERA D414
+  <origin xyz="0.095 -0.053 -0.053" rpy="3.139 0.785 1.570" />
+  CAMERA L515
+  <origin xyz="0.340 -0.35 0.70" rpy="0 0 -1.57" /> -->
   <xacro:include filename="$(find ur_e_description)/urdf/ur.transmission.xacro" />
   <xacro:include filename="$(find ur_e_description)/urdf/ur.gazebo.xacro" />
