Commit message: e5 run calibration test

File: UR5/ur_e_description/urdf/optimized.urdf.xacro (robot description, xacro)
@@ -165,5 +165,5 @@
   </gazebo>
   <joint name="camera_mb_rgb_joint" type="fixed">
-    <origin xyz="0.0 -0.045 0.0" rpy="0.0 -0.0 0.0"/>
+    <origin xyz="-0.0025015140549755985 -0.024119564231781077 0.004173799232878207" rpy="0.00020131023426650055 0.00454660351523446 0.0032054536137352367"/>
     <parent link="camera_mb_link"/>
     <child link="camera_mb_rgb_frame"/>
@@ -423,5 +423,5 @@
   <link name="imu_link"/>
   <joint name="moving_base_to_ur5e" type="fixed">
-    <origin xyz="-0.296 -0.1688 0.826" rpy="0.0 -0.0 0.0"/>
+    <origin xyz="-0.296 -0.1688 0.826" rpy="0.0 0.0 0.0"/>
     <parent link="base_link_mb"/>
     <child link="base_link"/>
@@ -738,5 +738,5 @@
   </gazebo>
   <joint name="camera_rgb_joint" type="fixed">
-    <origin xyz="0.0 -0.045 0.0" rpy="0.0 -0.0 0.0"/>
+    <origin xyz="0.0005708999221550831 -0.04483417895998767 -0.014856254433937226" rpy="-0.0016201598511101118 -0.01284397397093856 0.020932728494081596"/>
     <parent link="camera_link"/>
     <child link="camera_rgb_frame"/>

Commit message: rerun calibration

File: UR5/ur_e_description/urdf/optimized.urdf.xacro (robot description, xacro)
@@ -218,5 +218,5 @@
   </link>
   <joint name="ee_camera_support_joint" type="fixed">
-    <origin xyz="0.095 0.0 0.0" rpy="0.0 0.0 0.0"/>
+    <origin xyz="0.095 0.0 0.0" rpy="-0.7853981633974483 0.0 0.0"/>
     <parent link="ee_link"/>
     <child link="ee_camera_support_link"/>
@@ -245,5 +245,5 @@
   </material>
   <joint name="camera_joint" type="fixed">
-    <origin xyz="0.095 0.0 -0.075" rpy="-3.14 0.0 1.57"/>
+    <origin xyz="0.095 -0.053 -0.053" rpy="3.139 0.785 1.57"/>
     <parent link="ee_link"/>
     <child link="camera_bottom_screw_frame"/>

File: UR5/ur_e_description/urdf/optimized/optimized_2023_05_01-02_34_55_PM.urdf.xacro (robot description, xacro)
@@ -294,5 +294,5 @@
   <link name="camera_color_frame"/>
   <joint name="camera_aligned_depth_to_color_frame_joint" type="fixed">
-    <origin xyz="0.0 0.0 0.0" rpy="0.0 -0.0 0.0"/>
+    <origin xyz="-0.05298173400346154 -0.0174023821816474 -0.04993786146093298" rpy="0.089805555457002 -1.0650113792975349 -0.058841870204059385"/>
     <parent link="camera_link"/>
     <child link="camera_aligned_depth_to_color_frame"/>

Commit message: add optimized urdf

File: UR5/ur_e_description/urdf/optimized.urdf.xacro (robot description, xacro)
@@ -294,5 +294,5 @@
   <link name="camera_color_frame"/>
   <joint name="camera_aligned_depth_to_color_frame_joint" type="fixed">
-    <origin xyz="-0.05298173400346154 -0.0174023821816474 -0.04993786146093298" rpy="0.089805555457002 -1.0650113792975349 -0.058841870204059385"/>
+    <origin xyz="-0.007084414652850824 -0.01451531594060645 -0.024115140013064067" rpy="0.050169235346926855 -0.28320603927167837 -0.03327284138624655"/>
     <parent link="camera_link"/>
     <child link="camera_aligned_depth_to_color_frame"/>

Commit message: Updates in several files.

File: UR5/ur_e_description/urdf/optimized.urdf.xacro (robot description, xacro)
@@ -144,5 +144,5 @@
   </gazebo>
   <joint name="cam_2_joint" type="fixed">
-    <origin xyz="0.34 -0.35 0.7" rpy="-0.03318539261743347 0.006678026885604881 -1.688657977914159"/>
+    <origin xyz="0.1530038774570458 -0.2841450931970692 0.7825282951310043" rpy="-0.13671031564148944 -0.04121685400062677 -1.4420036320148786"/>
     <parent link="zau/base_link"/>
     <child link="cam_2_link"/>
@@ -213,5 +213,5 @@
   </link>
   <joint name="moving_base_to_ur5e" type="fixed">
-    <origin xyz="-0.295 0.0 0.78" rpy="0.0 -0.0 0.0"/>
+    <origin xyz="-0.2979179738119831 -0.11465486950124598 0.6182400882946293" rpy="-0.1311170899972734 -0.14416229797522645 0.043683285513000825"/>
     <parent link="zau/base_link"/>
     <child link="base_link"/>
@@ -425,5 +425,5 @@
   </material>
   <joint name="cam_1_joint" type="fixed">
-    <origin xyz="0.0949999988079071 -0.05299999937415123 -0.05299999937415123" rpy="1.4705796373386142 1.5526547081704947 3.040323153814818"/>
+    <origin xyz="0.30851401464230965 -0.20902636369158029 -0.0170192376060322" rpy="-3.1381629570168874 0.9110892255756052 1.7940029716605277"/>
     <parent link="ee_link"/>
     <child link="cam_1_link"/>

File: UR5/ur_e_description/urdf/optimized/optimized_2023_05_26-02_09_29_PM.urdf.xacro (robot description, xacro)
@@ -144,5 +144,5 @@
   </gazebo>
   <joint name="cam_2_joint" type="fixed">
-    <origin xyz="0.34 -0.35 0.7" rpy="-0.03318539261743347 0.006678026885604881 -1.688657977914159"/>
+    <origin xyz="0.31150373950124965 -0.8043696491120605 -0.008281171640317437" rpy="1.1793734548466825 -0.8096229670698206 -1.6432492851909746"/>
     <parent link="zau/base_link"/>
     <child link="cam_2_link"/>
@@ -213,5 +213,5 @@
   </link>
   <joint name="moving_base_to_ur5e" type="fixed">
-    <origin xyz="-0.295 0.0 0.78" rpy="0.0 -0.0 0.0"/>
+    <origin xyz="-0.23099492280096728 -0.1867556446894586 0.7229437843798114" rpy="2.8246006183063455 1.2311145532392187 2.7137624172129424"/>
     <parent link="zau/base_link"/>
     <child link="base_link"/>
@@ -425,5 +425,5 @@
   </material>
   <joint name="cam_1_joint" type="fixed">
-    <origin xyz="0.0949999988079071 -0.05299999937415123 -0.05299999937415123" rpy="1.4705796373386142 1.5526547081704947 3.040323153814818"/>
+    <origin xyz="0.17082898217475778 0.5684020965540681 -0.16228456384334783" rpy="1.5901011400620986 0.8161435550726787 -2.9526791922734215"/>
     <parent link="ee_link"/>
     <child link="cam_1_link"/>

File: UR5/ur_e_description/urdf/optimized/optimized_2023_05_26-02_30_54_PM.urdf.xacro (robot description, xacro)
@@ -144,5 +144,5 @@
   </gazebo>
   <joint name="cam_2_joint" type="fixed">
-    <origin xyz="0.34 -0.35 0.7" rpy="-0.03318539261743347 0.006678026885604881 -1.688657977914159"/>
+    <origin xyz="0.34838070463192033 -0.8186420792628797 0.018510745012290292" rpy="1.2334394467043706 -0.818723803936033 -1.6812990989739722"/>
     <parent link="zau/base_link"/>
     <child link="cam_2_link"/>
@@ -213,5 +213,5 @@
   </link>
   <joint name="moving_base_to_ur5e" type="fixed">
-    <origin xyz="-0.295 0.0 0.78" rpy="0.0 -0.0 0.0"/>
+    <origin xyz="-0.23217632526907253 -0.1904560815060482 0.7307172143472246" rpy="2.797555067102324 1.2615478416654053 2.688835128316127"/>
     <parent link="zau/base_link"/>
     <child link="base_link"/>
@@ -425,5 +425,5 @@
   </material>
   <joint name="cam_1_joint" type="fixed">
-    <origin xyz="0.0949999988079071 -0.05299999937415123 -0.05299999937415123" rpy="1.4705796373386142 1.5526547081704947 3.040323153814818"/>
+    <origin xyz="0.1685438503450023 0.5561255596071937 -0.16659620123936061" rpy="1.5885385373163687 0.8101311318379685 -2.9566877572851817"/>
     <parent link="ee_link"/>
     <child link="cam_1_link"/>

File: UR5/ur_e_description/urdf/optimized/optimized_2023_05_26-02_34_25_PM.urdf.xacro (robot description, xacro)
@@ -144,5 +144,5 @@
   </gazebo>
   <joint name="cam_2_joint" type="fixed">
-    <origin xyz="0.34 -0.35 0.7" rpy="-0.03318539261743347 0.006678026885604881 -1.688657977914159"/>
+    <origin xyz="0.6104677442479142 -0.4199529484957182 0.9856988627186496" rpy="0.530153195015799 0.19934985222984206 -1.7005380417249443"/>
     <parent link="zau/base_link"/>
     <child link="cam_2_link"/>
@@ -213,5 +213,5 @@
   </link>
   <joint name="moving_base_to_ur5e" type="fixed">
-    <origin xyz="-0.295 0.0 0.78" rpy="0.0 -0.0 0.0"/>
+    <origin xyz="-0.4591791217901308 0.2970981639743416 0.6268823041724385" rpy="0.31886428233072667 -0.2950990175336813 -0.15646218171540455"/>
     <parent link="zau/base_link"/>
     <child link="base_link"/>
@@ -425,5 +425,5 @@
   </material>
   <joint name="cam_1_joint" type="fixed">
-    <origin xyz="0.0949999988079071 -0.05299999937415123 -0.05299999937415123" rpy="1.4705796373386142 1.5526547081704947 3.040323153814818"/>
+    <origin xyz="0.5986653946476126 -0.24056267961111275 -0.1954086048952822" rpy="-2.926318352492197 1.1232385755054164 1.4532874690819761"/>
     <parent link="ee_link"/>
     <child link="cam_1_link"/>

File: UR5/ur_e_description/urdf/ur5e.urdf.xacro (robot description, xacro)
@@ -528,5 +528,5 @@
     <xacro:sensor_d415 name="cam_1" parent="${prefix}ee_link" use_nominal_extrinsics="true">
       <origin xyz="0.095 -0.053 -0.053"
-        rpy="3.139 0.785 1.570" />
+              rpy="3.139 0.785 1.570" />
     </xacro:sensor_d415>
       <!-- <origin xyz="0.095 0.000 -0.075" -->

Commit message: Add optimization results.

File: UR5/ur_e_description/urdf/optimized.urdf.xacro (robot description, xacro)
@@ -144,5 +144,5 @@
   </gazebo>
   <joint name="cam_2_joint" type="fixed">
-    <origin xyz="0.1530038774570458 -0.2841450931970692 0.7825282951310043" rpy="-0.13671031564148944 -0.04121685400062677 -1.4420036320148786"/>
+    <origin xyz="0.15290404237629823 -0.2841245584238319 0.782611623493062" rpy="-0.13663778008446342 -0.04114220660927234 -1.4418924474387382"/>
     <parent link="zau/base_link"/>
     <child link="cam_2_link"/>
@@ -213,5 +213,5 @@
   </link>
   <joint name="moving_base_to_ur5e" type="fixed">
-    <origin xyz="-0.2979179738119831 -0.11465486950124598 0.6182400882946293" rpy="-0.1311170899972734 -0.14416229797522645 0.043683285513000825"/>
+    <origin xyz="-0.2979608358483814 -0.11472442040002608 0.6181986448159426" rpy="-0.1311052993810706 -0.1443570322955178 0.04368511806425719"/>
     <parent link="zau/base_link"/>
     <child link="base_link"/>
@@ -425,5 +425,5 @@
   </material>
   <joint name="cam_1_joint" type="fixed">
-    <origin xyz="0.30851401464230965 -0.20902636369158029 -0.0170192376060322" rpy="-3.1381629570168874 0.9110892255756052 1.7940029716605277"/>
+    <origin xyz="0.3087070120211423 -0.2090674234359881 -0.017002222824133648" rpy="-3.1382800935211925 0.9109924691532048 1.7940296688604156"/>
     <parent link="ee_link"/>
     <child link="cam_1_link"/>

File: UR5/ur_e_description/urdf/optimized/optimized_2023_05_26-05_20_56_PM.urdf.xacro (robot description, xacro)
@@ -144,5 +144,5 @@
   </gazebo>
   <joint name="cam_2_joint" type="fixed">
-    <origin xyz="0.6104677442479142 -0.4199529484957182 0.9856988627186496" rpy="0.530153195015799 0.19934985222984206 -1.7005380417249443"/>
+    <origin xyz="0.15290404237629823 -0.2841245584238319 0.782611623493062" rpy="-0.13663778008446342 -0.04114220660927234 -1.4418924474387382"/>
     <parent link="zau/base_link"/>
     <child link="cam_2_link"/>
@@ -213,5 +213,5 @@
   </link>
   <joint name="moving_base_to_ur5e" type="fixed">
-    <origin xyz="-0.4591791217901308 0.2970981639743416 0.6268823041724385" rpy="0.31886428233072667 -0.2950990175336813 -0.15646218171540455"/>
+    <origin xyz="-0.2979608358483814 -0.11472442040002608 0.6181986448159426" rpy="-0.1311052993810706 -0.1443570322955178 0.04368511806425719"/>
     <parent link="zau/base_link"/>
     <child link="base_link"/>
@@ -425,5 +425,5 @@
   </material>
   <joint name="cam_1_joint" type="fixed">
-    <origin xyz="0.5986653946476126 -0.24056267961111275 -0.1954086048952822" rpy="-2.926318352492197 1.1232385755054164 1.4532874690819761"/>
+    <origin xyz="0.3087070120211423 -0.2090674234359881 -0.017002222824133648" rpy="-3.1382800935211925 0.9109924691532048 1.7940296688604156"/>
     <parent link="ee_link"/>
     <child link="cam_1_link"/>
