Commit message: AGV odom

File: UR5/ur_e_description/urdf/moving_base_odom.gazebo.xacro (robot description, xacro)
@@ -42,6 +42,6 @@
     <!--  back caster -->
     <gazebo reference="caster_back_right_link">
-        <mu1>0.01</mu1>
-        <mu2>0.01</mu2>
+        <mu1>0.1</mu1>
+        <mu2>0.1</mu2>
         <kp>1000000.0</kp>
         <kd>100.0</kd>
@@ -51,6 +51,6 @@
     </gazebo>
     <gazebo reference="caster_back_left_link">
-        <mu1>0.01</mu1>
-        <mu2>0.01</mu2>
+        <mu1>0.1</mu1>
+        <mu2>0.1</mu2>
         <kp>1000000.0</kp>
         <kd>100.0</kd>
@@ -62,6 +62,6 @@
     <!--  front caster -->
     <gazebo reference="caster_front_right_link">
-        <mu1>0.01</mu1>
-        <mu2>0.01</mu2>
+        <mu1>0.1</mu1>
+        <mu2>0.1</mu2>
         <kp>1000000.0</kp>
         <kd>100.0</kd>
@@ -71,6 +71,6 @@
     </gazebo>
     <gazebo reference="caster_front_left_link">
-        <mu1>0.01</mu1>
-        <mu2>0.01</mu2>
+        <mu1>0.1</mu1>
+        <mu2>0.1</mu2>
         <kp>1000000.0</kp>
         <kd>100.0</kd>

File: UR5/ur_e_description/urdf/moving_base_odom.urdf.xacro (robot description, xacro)
@@ -50,5 +50,5 @@
     <link name="inertial_link">
         <inertial>
-            <mass value="100" />
+            <mass value="500" />
             <origin xyz="-0.00065 -0.085 0.062" />
             <inertia ixx="0.6022" ixy="-0.02364" ixz="-0.1197" iyy="1.7386" iyz="-0.001544"

File: UR5/ur_e_description/urdf/ur5e.urdf.xacro (robot description, xacro)
@@ -4,5 +4,8 @@
   <xacro:include filename="$(find ur_e_description)/urdf/ur.gazebo.xacro" />
   <!-- place robot on moving base -->
-  <xacro:include filename="$(find ur_e_description)/urdf/moving_base.urdf.xacro" />
+  <!-- fixed AGV -->
+  <!-- <xacro:include filename="$(find ur_e_description)/urdf/moving_base.urdf.xacro" /> -->
+  <!-- moving AGV -->
+  <xacro:include filename="$(find ur_e_description)/urdf/moving_base_odom.urdf.xacro" />
   <!-- *************THIS IS THE TRANSFORMATION TO BE CALIBRATED************* -->
   <joint name="moving_base_to_ur5e" type="fixed">

File: UR5/ur_e_description/urdf/ur5e_joint_limited_robot.urdf.xacro (robot description, xacro)
@@ -27,10 +27,10 @@
   <!-- initial robot pose on world - FROM ORIGINAL FILE -->
   <!-- toogle this part to move the AGV in odom -->
-  <link name="world" />
+  <!-- <link name="world" />
   <joint name="world_joint" type="fixed">
     <parent link="world" />
     <child link="base_link_mb" />
     <origin xyz="0.0 0.0 0.0" rpy="0.0 0.0 0.0" />
-  </joint>
+  </joint> -->
   <!-- initial robot pose on world - FROM ORIGINAL FILE -->
   <!-- THIS PART WAS FOR TEST ONLY - JORGE -->

Commit message: add 2D lidars to the AGV

File: UR5/ur_e_description/urdf/moving_base_odom.gazebo.xacro (robot description, xacro)
@@ -184,5 +184,5 @@
     <!-- add sensor camera part -->
     <!-- lidar sensor front -->
-    <!-- <gazebo reference="base_scan_front">
+    <gazebo reference="base_scan_front">
         <material>Gazebo/DarkGrey</material>
         <sensor type="ray" name="lds_lfcd_sensor_front">
@@ -215,8 +215,8 @@
             </plugin>
         </sensor>
-    </gazebo> -->
+    </gazebo>
     <!-- lidar sensor front -->
     <!-- lidar sensor back -->
-    <!-- <gazebo reference="base_scan_back">
+    <gazebo reference="base_scan_back">
         <material>Gazebo/DarkGrey</material>
         <sensor type="ray" name="lds_lfcd_sensor_back">
@@ -249,5 +249,5 @@
             </plugin>
         </sensor>
-    </gazebo> -->
+    </gazebo>
     <!-- lidar sensor back -->
 </robot>

File: UR5/ur_e_description/urdf/moving_base_odom.urdf.xacro (robot description, xacro)
@@ -242,10 +242,9 @@
     </joint>
     <link name="imu_link" />
-<!-- ROMEVED FOR NOW - JORGE FEB 2023 -->
     <!-- lidar sensor front -->
-    <!-- <joint name="scan_joint_front" type="fixed">
+    <joint name="scan_joint_front" type="fixed">
         <parent link="base_link_mb" />
         <child link="base_scan_front" />
-        <origin xyz="-0.700 0 0.180" rpy="0 0 ${M_PI/4}" />
+        <origin xyz="-0.450 0.3 0.180" rpy="0 0 0" />
     </joint>
     <link name="base_scan_front">
@@ -261,11 +260,11 @@
             <inertia ixx="0.001" ixy="0.0" ixz="0.0" iyy="0.001" iyz="0.0" izz="0.001" />
         </inertial>
-    </link> -->
+    </link>
     <!-- lidar sensor front -->
     <!-- lidar sensor back -->
-    <!-- <joint name="scan_joint_back" type="fixed">
+    <joint name="scan_joint_back" type="fixed">
         <parent link="base_link_mb" />
         <child link="base_scan_back" />
-        <origin xyz="0.700 0 0.180" rpy="0 0 -${3*M_PI/4}" />
+        <origin xyz="0.500 -0.3 0.180" rpy="0 0 -3.14" />
     </joint>
     <link name="base_scan_back">
@@ -281,6 +280,5 @@
             <inertia ixx="0.001" ixy="0.0" ixz="0.0" iyy="0.001" iyz="0.0" izz="0.001" />
         </inertial>
-    </link> -->
+    </link>
     <!-- lidar sensor back -->
-    <!-- ROMEVED FOR NOW - JORGE FEB 2023 -->
 </robot>

Commit message: add intel realsense

File: UR5/ur_e_description/urdf/moving_base_odom.gazebo.xacro (robot description, xacro)
@@ -144,5 +144,5 @@
     </gazebo>
     <!-- add sensor camera part -->
-    <xacro:macro name="sim_3dsensor" params="prefix">
+    <!-- <xacro:macro name="sim_3dsensor" params="prefix">
         <gazebo reference="${prefix}_depth_frame">
             <sensor type="depth" name="camera">
@@ -181,5 +181,5 @@
             </sensor>
         </gazebo>
-    </xacro:macro>
+    </xacro:macro> -->
     <!-- add sensor camera part -->
     <!-- lidar sensor front -->

File: UR5/ur_e_description/urdf/moving_base_odom.urdf.xacro (robot description, xacro)
@@ -4,23 +4,32 @@
     <xacro:include filename="$(find ur_e_description)/urdf/moving_base_odom.gazebo.xacro" />
     <xacro:property name="M_PI" value="3.1415926535897931" />
-    <!-- testing adding a velodyne laser  -->
-    <!-- VLP-16 -->
-    <!-- velodyne -->
-    <!-- <xacro:arg name="gpu" default="false" />
-    <xacro:property name="gpu" value="$(arg gpu)" />
-    <xacro:arg name="organize_cloud" default="false" />
-    <xacro:property name="organize_cloud" value="$(arg organize_cloud)" />
-    <xacro:include filename="$(find velodyne_description)/urdf/VLP-16.urdf.xacro" />
-    <xacro:VLP-16 parent="base_link_mb" name="velodyne" topic="/velodyne_points"
-    organize_cloud="${organize_cloud}" hz="10" samples="440" gpu="${gpu}">
-        <origin xyz="-0.350 0.050 0.850" rpy="0 0 0" />
-    </xacro:VLP-16> -->
-    <!-- velodyne -->
     <!-- testing adding a sensor camera -->
-    <xacro:include filename="$(find ur_e_description)/urdf/astra.urdf.xacro" />
+    <!-- <xacro:include filename="$(find ur_e_description)/urdf/astra.urdf.xacro" />
     <xacro:sensor_astra parent="base_link_mb" prefix="camera_mb">
         <origin xyz="-0.350 0.180 0.870"
             rpy="0 0 3.14" />
-    </xacro:sensor_astra>
+    </xacro:sensor_astra> -->
+    <!-- add intel realsense camera d415 sensor -->
+    <xacro:arg name="realsense_enabled" default="$(optenv REALSENSE_ENABLED 1)" />
+    <xacro:arg name="realsense_topic" default="$(optenv REALSENSE_TOPIC realsense)" />
+    <xacro:arg name="realsense_prefix" default="$(optenv REALSENSE_PREFIX camera_realsense)" />
+    <xacro:arg name="realsense_parent" default="$(optenv REALSENSE_PARENT base_link_mb)" />
+    <xacro:arg name="realsense_xyz" default="$(optenv REALSENSE_XYZ -0.350 0.180 0.870)" />
+    <xacro:arg name="realsense_rpy" default="$(optenv REALSENSE_RPY 0 0 3.14)" />
+    <material name="white">
+        <color rgba="1.0 1.0 1.0 1.0" />
+    </material>
+    <xacro:include filename="$(find ur_e_description)/urdf/realsense/intel_realsense.urdf.xacro" />
+    <xacro:if value="$(arg realsense_enabled)">
+        <link name="$(arg realsense_prefix)_realsense_mountpoint" />
+        <joint name="$(arg realsense_prefix)_realsense_mountpoint_joint" type="fixed">
+            <origin xyz="$(arg realsense_xyz)" rpy="$(arg realsense_rpy)" />
+            <parent link="$(arg realsense_parent)" />
+            <child link="$(arg realsense_prefix)_realsense_mountpoint" />
+        </joint>
+        <xacro:intel_realsense_mount prefix="$(arg realsense_prefix)" topic="$(arg realsense_topic)"
+            parent_link="$(arg realsense_prefix)_realsense_mountpoint" />
+    </xacro:if>
+    <!-- add intel realsense d415 sensor -->
     <link name="base_footprint" />
     <joint name="base_joint" type="fixed">
@@ -86,5 +95,5 @@
             <origin xyz="0 0 0" />
             <mass value="2.637" />
-            <inertia  ixx="0.02467" ixy="0" ixz="0" iyy="0.04411" iyz="0" izz="0.02467" />
+            <inertia ixx="0.02467" ixy="0" ixz="0" iyy="0.04411" iyz="0" izz="0.02467" />
         </inertial>
     </link>
@@ -113,5 +122,5 @@
             <origin xyz="0 0 0" />
             <mass value="2.637" />
-            <inertia  ixx="0.02467" ixy="0" ixz="0" iyy="0.04411" iyz="0" izz="0.02467" />
+            <inertia ixx="0.02467" ixy="0" ixz="0" iyy="0.04411" iyz="0" izz="0.02467" />
         </inertial>
     </link>
@@ -242,5 +251,5 @@
     </joint>
     <link name="imu_link" />
-<!-- ROMEVED FOR NOW - JORGE FEB 2023 -->
+    <!-- ROMEVED FOR NOW - JORGE FEB 2023 -->
     <!-- lidar sensor front -->
     <!-- <joint name="scan_joint_front" type="fixed">

Commit message: add calibration files

File: UR5/ur_e_description/urdf/moving_base_odom.gazebo.xacro (robot description, xacro)
@@ -96,6 +96,6 @@
         <plugin name="moving_base_controller" filename="libgazebo_ros_diff_drive.so">
             <commandTopic>cmd_vel</commandTopic>
-            <odometryTopic>odom</odometryTopic>
-            <odometryFrame>odom</odometryFrame>
+            <odometryTopic>zau/odom</odometryTopic>
+            <odometryFrame>zau/odom</odometryFrame>
             <odometrySource>world</odometrySource>
             <publishOdomTF>true</publishOdomTF>

File: UR5/ur_e_description/urdf/moving_base_odom.urdf.xacro (robot description, xacro)
@@ -4,16 +4,26 @@
     <xacro:include filename="$(find ur_e_description)/urdf/moving_base_odom.gazebo.xacro" />
     <xacro:property name="M_PI" value="3.1415926535897931" />
+    <!-- add intel realsense l515 camera -->
+    <xacro:arg name="use_nominal_extrinsics" default="true" />
+    <xacro:arg name="add_plug" default="false" />
+    <xacro:arg name="use_mesh" default="true" />
+    <xacro:include filename="$(find ur_e_description)/urdf/realsense/_l515.urdf.xacro" />
+    <xacro:sensor_l515 name="cam_2" parent="zau/base_link" use_nominal_extrinsics="$(arg use_nominal_extrinsics)"
+        add_plug="$(arg add_plug)" use_mesh="$(arg use_mesh)">
+        <origin xyz="0.340 -0.35 0.70" rpy="0 0 -1.57" />
+    </xacro:sensor_l515>
+    <!-- add intel realsense l515 camera -->
     <!-- add intel realsense camera d415 sensor -->
     <!-- <xacro:include
         filename="$(find ur_e_description)/urdf/realsense/intel_realsense_inesctec.urdf.xacro" />
-    <xacro:sensor_d415 parent="base_link_mb" use_nominal_extrinsics="true" name="camera_mb">
+    <xacro:sensor_d415 parent="zau/base_link" use_nominal_extrinsics="true" name="camera_mb">
         <origin xyz="0.400 -0.250 0.79"
             rpy="0.0 -0.2 0.0" />
     </xacro:sensor_d415> -->
-    <xacro:arg name="realsense_AGV_enabled" default="$(optenv REALSENSE_AGV_ENABLED 1)" />
+    <!-- <xacro:arg name="realsense_AGV_enabled" default="$(optenv REALSENSE_AGV_ENABLED 1)" />
     <xacro:arg name="realsense_AGV_topic" default="$(optenv REALSENSE_AGV_TOPIC AGV_realsense)" />
     <xacro:arg name="realsense_AGV_prefix" default="$(optenv REALSENSE_AGV_PREFIX
     AGV_camera_realsense)" />
-    <xacro:arg name="realsense_AGV_parent" default="$(optenv REALSENSE_AGV_PARENT base_link_mb)" />
+    <xacro:arg name="realsense_AGV_parent" default="$(optenv REALSENSE_AGV_PARENT zau/base_link)" />
     <xacro:arg name="realsense_AGV_xyz" default="$(optenv REALSENSE_AGV_XYZ 0.400 -0.250 0.79)" />
     <xacro:arg name="realsense_AGV_rpy" default="$(optenv REALSENSE_AGV_RPY 0 -0.2 0)" />
@@ -32,13 +42,13 @@
     realsense_AGV_topic)"
             parent_link="$(arg realsense_AGV_prefix)_realsense_mountpoint" />
-    </xacro:if>
+    </xacro:if> -->
     <!-- add intel realsense d415 sensor -->
-    <link name="base_footprint" />
+    <link name="zau/base_footprint" />
     <joint name="base_joint" type="fixed">
-        <parent link="base_footprint" />
-        <child link="base_link_mb" />
+        <parent link="zau/base_footprint" />
+        <child link="zau/base_link" />
         <origin xyz="0 0 0.010" rpy="0 0 0" />
     </joint>
-    <link name="base_link_mb">
+    <link name="zau/base_link">
         <visual>
             <origin xyz="-0.46 0.335 0.06" rpy="1.57 0 0" />
@@ -58,5 +68,5 @@
     </link>
     <!-- Inertial link stores the robot's inertial information -->
-    <link name="inertial_link">
+    <!-- <link name="inertial_link">
         <inertial>
             <mass value="500" />
@@ -65,13 +75,13 @@
                 izz="2.0296" />
         </inertial>
-    </link>
-    <joint name="inertial_joint" type="fixed">
+    </link> -->
+    <!-- <joint name="inertial_joint" type="fixed">
         <origin xyz="0 0 0" rpy="0 0 0" />
-        <parent link="base_link_mb" />
+        <parent link="zau/base_link" />
         <child link="inertial_link" />
-    </joint>
+    </joint> -->
     <!-- #################### wheels #################### -->
-    <joint name="wheel_left_joint" type="continuous">
-        <parent link="base_link_mb" />
+    <!-- <joint name="wheel_left_joint" type="continuous">
+        <parent link="zau/base_link" />
         <child link="wheel_left_link" />
         <origin xyz="0.0 0.325 0.074" rpy="-1.57 0 0" />
@@ -100,5 +110,5 @@
     </link>
     <joint name="wheel_right_joint" type="continuous">
-        <parent link="base_link_mb" />
+        <parent link="zau/base_link" />
         <child link="wheel_right_link" />
         <origin xyz="0.0 -0.325 0.074" rpy="-1.57 0 0" />
@@ -125,12 +135,12 @@
             <inertia ixx="0.02467" ixy="0" ixz="0" iyy="0.04411" iyz="0" izz="0.02467" />
         </inertial>
-    </link>
+    </link> -->
     <!-- back caster -->
-    <joint name="caster_back_right_joint" type="fixed">
-        <parent link="base_link_mb" />
+    <!-- <joint name="caster_back_right_joint" type="fixed">
+        <parent link="zau/base_link" />
         <child link="caster_back_right_link" />
         <origin xyz="-0.345 -0.190 -0.004" rpy="-1.57 0 0" />
-    </joint>
-    <link name="caster_back_right_link">
+    </joint> -->
+    <!-- <link name="caster_back_right_link">
         <visual>
             <origin xyz="0.027 -0.06 0" rpy="1.57 0 0" />
@@ -138,5 +148,4 @@
                 <mesh filename="package://ur_e_description/meshes/wheels/left_tire.stl"
                     scale="0.0020 0.0020 0.0020" />
-                <!-- <cylinder length="0.024" radius="0.084" /> -->
             </geometry>
             <material name="dark" />
@@ -155,11 +164,11 @@
                 izz="0.001" />
         </inertial>
-    </link>
-    <joint name="caster_back_left_joint" type="fixed">
-        <parent link="base_link_mb" />
+    </link> -->
+    <!-- <joint name="caster_back_left_joint" type="fixed">
+        <parent link="zau/base_link" />
         <child link="caster_back_left_link" />
         <origin xyz="-0.345 0.190 -0.004" rpy="-1.57 0 0" />
-    </joint>
-    <link name="caster_back_left_link">
+    </joint> -->
+    <!-- <link name="caster_back_left_link">
         <visual>
             <origin xyz="0.027 -0.06 0" rpy="-1.57 0 0" />
@@ -167,5 +176,4 @@
                 <mesh filename="package://ur_e_description/meshes/wheels/left_tire.stl"
                     scale="0.0020 0.0020 0.0020" />
-                <!-- <cylinder length="0.024" radius="0.084" /> -->
             </geometry>
             <material name="dark" />
@@ -184,9 +192,9 @@
                 izz="0.001" />
         </inertial>
-    </link>
+    </link> -->
     <!-- back caster -->
     <!-- front caster -->
-    <joint name="caster_front_right_joint" type="fixed">
-        <parent link="base_link_mb" />
+    <!-- <joint name="caster_front_right_joint" type="fixed">
+        <parent link="zau/base_link" />
         <child link="caster_front_right_link" />
         <origin xyz="0.345 -0.190 -0.004" rpy="-1.57 0 0" />
@@ -198,5 +206,4 @@
                 <mesh filename="package://ur_e_description/meshes/wheels/left_tire.stl"
                     scale="0.0020 0.0020 0.0020" />
-                <!-- <cylinder length="0.024" radius="0.084" /> -->
             </geometry>
             <material name="dark" />
@@ -215,11 +222,11 @@
                 izz="0.001" />
         </inertial>
-    </link>
-    <joint name="caster_front_left_joint" type="fixed">
-        <parent link="base_link_mb" />
+    </link> -->
+    <!-- <joint name="caster_front_left_joint" type="fixed">
+        <parent link="zau/base_link" />
         <child link="caster_front_left_link" />
         <origin xyz="0.345 0.190 -0.004" rpy="-1.57 0 0" />
-    </joint>
-    <link name="caster_front_left_link">
+    </joint> -->
+    <!-- <link name="caster_front_left_link">
         <visual>
             <origin xyz="0 -0.06 0" rpy="-1.57 0 0" />
@@ -227,5 +234,4 @@
                 <mesh filename="package://ur_e_description/meshes/wheels/left_tire.stl"
                     scale="0.0020 0.0020 0.0020" />
-                <!-- <cylinder length="0.024" radius="0.084" /> -->
             </geometry>
             <material name="dark" />
@@ -244,16 +250,16 @@
                 izz="0.001" />
         </inertial>
-    </link>
+    </link> -->
     <!-- front caster -->
-    <joint name="imu_joint" type="fixed">
-        <parent link="base_link_mb" />
+    <!-- <joint name="imu_joint" type="fixed">
+        <parent link="zau/base_link" />
         <child link="imu_link" />
         <origin xyz="0.0 0 0.068" rpy="0 0 0" />
     </joint>
-    <link name="imu_link" />
+    <link name="imu_link" /> -->
     <!-- ROMEVED FOR NOW - JORGE FEB 2023 need check real position in the robot -->
     <!-- lidar sensor front -->
     <!-- <joint name="scan_joint_front" type="fixed">
-        <parent link="base_link_mb" />
+        <parent link="zau/base_link" />
         <child link="base_scan_front" />
         <origin xyz="-0.700 0 0.180" rpy="0 0 ${M_PI/4}" />
@@ -275,5 +281,5 @@
     <!-- lidar sensor back -->
     <!-- <joint name="scan_joint_back" type="fixed">
-        <parent link="base_link_mb" />
+        <parent link="zau/base_link" />
         <child link="base_scan_back" />
         <origin xyz="0.700 0 0.180" rpy="0 0 -${3*M_PI/4}" />

File: UR5/ur_e_description/urdf/realsense/intel_realsense_inesctec.urdf.xacro (robot description, xacro)
@@ -34,12 +34,12 @@
       <xacro:insert_block name="origin" />
       <parent link="${parent}"/>
-      <child link="${name}_bottom_screw_frame" />
+      <child link="${name}_link" />
     </joint>
-    <link name="${name}_bottom_screw_frame"/>
+    <!-- <link name="${name}_bottom_screw_frame"/>
     <joint name="${name}_link_joint" type="fixed">
       <origin xyz="0 ${d415_cam_depth_py} ${d415_cam_depth_pz}" rpy="0 0 0"/>
       <parent link="${name}_bottom_screw_frame"/>
       <child link="${name}_link" />
-    </joint>
+    </joint> -->
     <link name="${name}_link">
       <visual>
@@ -115,10 +115,10 @@
       <link name="${name}_infra2_optical_frame" /> -->
       <!-- camera color joints and links -->
-      <joint name="${name}_color_joint" type="fixed">
+      <!-- <joint name="${name}_color_joint" type="fixed">
         <origin xyz="0 ${d415_cam_depth_to_color_offset} 0" rpy="0 0 0" />
         <parent link="${name}_link" />
         <child link="${name}_color_frame" />
       </joint>
-      <link name="${name}_color_frame" />
+      <link name="${name}_color_frame" /> -->
       <!-- <joint name="${name}_color_optical_joint" type="fixed">
         <origin xyz="0 0 0" rpy="${-M_PI/2} 0 ${-M_PI/2}" />
@@ -130,10 +130,10 @@
         <origin xyz="0 0 0" rpy="0 0 0" />
         <parent link="${name}_link" />
-        <child link="${name}_aligned_depth_to_color_frame" />
+        <child link="${name}_color_frame" />
       </joint>
-      <link name="${name}_aligned_depth_to_color_frame" />
+      <link name="${name}_color_frame" />
       <joint name="${name}_color_optical_joint" type="fixed">
         <origin xyz="0 0 0" rpy="${-M_PI/2} 0 ${-M_PI/2}" />
-        <parent link="${name}_aligned_depth_to_color_frame" />
+        <parent link="${name}_color_frame" />
         <child link="${name}_color_optical_frame" />
       </joint>

File: UR5/ur_e_description/urdf/ur5e.urdf.xacro (robot description, xacro)
@@ -10,5 +10,5 @@
   <!-- *************THIS IS THE TRANSFORMATION TO BE CALIBRATED************* -->
   <joint name="moving_base_to_ur5e" type="fixed">
-    <parent link="base_link_mb" />
+    <parent link="zau/base_link" />
     <child link="base_link" />
     <origin xyz="-0.295 0.0 0.780" rpy="0.0 0.0 0.0" />
@@ -484,5 +484,5 @@
     <!-- add gripper part end ###################################################################-->
     <!-- add camera support -->
-    <link name="${prefix}ee_camera_support_link">
+    <!-- <link name="${prefix}ee_camera_support_link">
       <visual>
         <geometry>
@@ -515,12 +515,13 @@
       <parent link="${prefix}ee_camera_support_link" />
       <child link="${prefix}ee_camera_support_small_link" />
-    </joint>
+    </joint> -->
     <!-- add intel realsense camera d415 sensor -->
     <xacro:include
       filename="$(find ur_e_description)/urdf/realsense/intel_realsense_inesctec.urdf.xacro" />
-    <xacro:sensor_d415 parent="ee_link" use_nominal_extrinsics="true">
-      <origin xyz="0.095 0.000 -0.075"
-        rpy="-3.14 0.0 1.57" />
+    <xacro:sensor_d415 name="cam_1" parent="${prefix}ee_link" use_nominal_extrinsics="true">
+      <origin xyz="0.095 -0.053 -0.053"
+        rpy="3.139 0.785 1.570" />
     </xacro:sensor_d415>
+      <!-- <origin xyz="0.095 0.000 -0.075" -->
     <!-- <xacro:arg name="realsense_EE_enabled" default="$(optenv REALSENSE_EE_ENABLED 1)" />
     <xacro:arg name="realsense_EE_topic" default="$(optenv REALSENSE_EE_TOPIC EE_realsense)" />
