Commit message: Add camera support and remove IMU link used for gazebo simulation.

File: UR5/ur_e_description/urdf/moving_base_odom.gazebo.xacro (robot description, xacro)
@@ -115,5 +115,5 @@
         </plugin>
     </gazebo>
-    <gazebo>
+    <!-- <gazebo>
         <plugin name="imu_plugin" filename="libgazebo_ros_imu.so">
             <alwaysOn>true</alwaysOn>
@@ -142,5 +142,5 @@
             </imu>
         </plugin>
-    </gazebo>
+    </gazebo> -->
     <!-- add sensor camera part -->
     <!-- <xacro:macro name="sim_3dsensor" params="prefix">

File: UR5/ur_e_description/urdf/ur5e.urdf.xacro (robot description, xacro)
@@ -491,8 +491,8 @@
     <!-- add gripper part end ###################################################################-->
     <!-- add camera support -->
-    <!-- <link name="${prefix}ee_camera_support_link">
-      <visual>
-        <geometry>
-          <box size="0.185 0.03 0.03" />
+    <link name="${prefix}ee_camera_support_link">
+      <visual>
+        <geometry>
+          <box size="0.15 0.03 0.03" />
         </geometry>
         <material name="LightGrey">
@@ -503,5 +503,5 @@
     </link>
     <joint name="${prefix}ee_camera_support_joint" type="fixed">
-      <origin xyz="0.095 0 0" rpy="0 0 0" />
+      <origin xyz="0.075 0 0" rpy="-0.785 0 0" />
       <parent link="${prefix}ee_link" />
       <child link="${prefix}ee_camera_support_link" />
@@ -522,5 +522,5 @@
       <parent link="${prefix}ee_camera_support_link" />
       <child link="${prefix}ee_camera_support_small_link" />
-    </joint> -->
+    </joint>
     <!-- add intel realsense camera d415 sensor -->
     <xacro:include
