Commit message: update e5

File: e5_DualRGB_arm2agv/e5_dualrgb_arm2agv_optimized/optimized/nig_0_0_optimized_dualrgb_arm2agv.urdf.xacro (robot description, xacro)
@@ -165,5 +165,5 @@
   </gazebo>
   <joint name="camera_mb_rgb_joint" type="fixed">
-    <origin xyz="-0.0005323809894553315 -0.01905332711317387 -0.007426163734254366" rpy="-1.6577534800718458e-05 -0.00039720245443191916 -0.001784354851982843"/>
+    <origin xyz="-0.0005468304863673578 -0.01978960480022218 -0.0016769780370784074" rpy="-0.00011729742680485002 0.00035540253112038145 -0.0014571668767702785"/>
     <parent link="camera_mb_link"/>
     <child link="camera_mb_rgb_frame"/>
@@ -423,6 +423,5 @@
   <link name="imu_link"/>
   <joint name="moving_base_to_ur5e" type="fixed">
-    <origin xyz="-0.29453838375094427 -0.16750697765626305 0.8203502127898897" rpy="0.0004717161498466556 -0.0007159745850205707 0.001072048560706622"/>
-    <!-- <origin xyz="-0.29466405085302455 -0.16821715652259384 0.83670476943398" rpy="0.0004903019915529824 1.0848955144563524e-05 0.000890764102930763"/> -->
+    <origin xyz="-0.29406503816446494 -0.16648855569170692 0.8262450094522876" rpy="0.0004507227081607748 -0.0015447953627994375 0.0016074847496047706"/>
     <parent link="base_link_mb"/>
     <child link="base_link"/>
@@ -739,5 +738,5 @@
   </gazebo>
   <joint name="camera_rgb_joint" type="fixed">
-    <origin xyz="0.0007852945275768551 -0.021544849161948758 -0.00040653966792914405" rpy="0.00040251243900585787 0.00043231794437063187 0.0005938325632927141"/>
+    <origin xyz="0.0008344938317361108 -0.021203213155327093 -5.080613760048783e-05" rpy="0.0003620045628476182 0.000745553208859285 0.00021687503586853156"/>
     <parent link="camera_link"/>
     <child link="camera_rgb_frame"/>
