Commit message: add e2 calibration

File: e2_arm2agv_rgb2ee/optimized/optimized_2023_03_04-09_12_00_AM.urdf.xacro (robot description, xacro)
@@ -329,5 +329,5 @@
   <link name="imu_link"/>
   <joint name="moving_base_to_ur5e" type="fixed">
-    <origin xyz="-0.296 -0.1688 0.826" rpy="0.0 -0.0 0.0"/>
+    <origin xyz="-0.20208207407196427 -0.20495120420482743 0.8405196945274782" rpy="-0.0573444165774149 0.017883775618432705 0.09047014867115873"/>
     <parent link="base_link_mb"/>
     <child link="base_link"/>
@@ -623,5 +623,5 @@
   </joint>
   <joint name="camera_joint" type="fixed">
-    <origin xyz="0.0600758568472458 -0.07451415139078899 0.04999473796135022" rpy="-3.141483156142495 -0.0009436775284828712 0.000545084455893016"/>
+    <origin xyz="0.05999529448690997 -0.07534268179850052 0.04961939102275036" rpy="3.141508334871305 -0.0012780257928761533 0.001219051288723527"/>
     <parent link="ee_link"/>
     <child link="camera_link"/>
@@ -644,5 +644,5 @@
   </gazebo>
   <joint name="camera_rgb_joint" type="fixed">
-    <origin xyz="0.0 -0.045 0.0" rpy="0.0 -0.0 0.0"/>
+    <origin xyz="0.0 -0.045 0.0" rpy="0.0 0.0 0.0"/>
     <parent link="camera_link"/>
     <child link="camera_rgb_frame"/>

File: e2_arm2agv_rgb2ee/optimized/optimized_2023_03_04-09_14_36_AM.urdf.xacro (robot description, xacro)
@@ -329,5 +329,5 @@
   <link name="imu_link"/>
   <joint name="moving_base_to_ur5e" type="fixed">
-    <origin xyz="-0.296 -0.1688 0.826" rpy="0.0 -0.0 0.0"/>
+    <origin xyz="-0.1731355558989543 -0.31155040851299554 0.8247675114172166" rpy="-0.165897034960856 -0.21376191920587986 0.17225340918871368"/>
     <parent link="base_link_mb"/>
     <child link="base_link"/>
@@ -623,5 +623,5 @@
   </joint>
   <joint name="camera_joint" type="fixed">
-    <origin xyz="0.0600758568472458 -0.07451415139078899 0.04999473796135022" rpy="-3.141483156142495 -0.0009436775284828712 0.000545084455893016"/>
+    <origin xyz="0.059374899777039615 -0.07534990687778702 0.05061996075516738" rpy="3.1415786050286174 -0.0003715034486972256 0.0012817209657054228"/>
     <parent link="ee_link"/>
     <child link="camera_link"/>
@@ -644,5 +644,5 @@
   </gazebo>
   <joint name="camera_rgb_joint" type="fixed">
-    <origin xyz="0.0 -0.045 0.0" rpy="0.0 -0.0 0.0"/>
+    <origin xyz="0.0 -0.045 0.0" rpy="0.0 0.0 0.0"/>
     <parent link="camera_link"/>
     <child link="camera_rgb_frame"/>
