Commit message: e0 update calibration

File: e0_rgb2ee/e0_rgb2ee_calibration/urdf/initial_estimate.urdf.xacro (robot description, xacro)
@@ -1,61 +1,823 @@
-<?xml version="1.0"?>
-<robot xmlns:xacro="http://ros.org/wiki/xacro"
-  name="ur5e">
-  <!-- common stuff -->
-  <xacro:include filename="$(find ur_e_description)/urdf/common.gazebo.xacro" />
-  <!-- ur5e -->
-  <xacro:include filename="$(find ur_e_description)/urdf/ur5e.urdf.xacro" />
-  <!-- arm -->
-  <xacro:ur5e_robot prefix="" joint_limited="true"
-    shoulder_pan_lower_limit="${-pi}" shoulder_pan_upper_limit="${pi}"
-    shoulder_lift_lower_limit="${-pi}" shoulder_lift_upper_limit="${pi}"
-    elbow_joint_lower_limit="${-pi}" elbow_joint_upper_limit="${pi}"
-    wrist_1_lower_limit="${-pi}" wrist_1_upper_limit="${pi}"
-    wrist_2_lower_limit="${-pi}" wrist_2_upper_limit="${pi}"
-    wrist_3_lower_limit="${-pi}" wrist_3_upper_limit="${pi}"
-  />
-  <!-- THIS PART WAS MOVED TO UR5E.URDF.XACRO  -->
-  <!-- place robot on moving base -->
-  <!-- <xacro:include filename="$(find ur_e_description)/urdf/moving_base.urdf.xacro" />
+<?xml version="1.0" ?>
+<robot name="ur5e" version="1.0">
+  <gazebo>
+    <plugin filename="libgazebo_ros_control.so" name="ros_control">
+    </plugin>
+  </gazebo>
+  <material name="grey">
+    <color rgba="0.7 0.7 0.7 1.0"/>
+  </material>
+  <material name="dark">
+    <color rgba="0.3 0.3 0.3 1.0"/>
+  </material>
+  <material name="light_black">
+    <color rgba="0.4 0.4 0.4 1.0"/>
+  </material>
+  <gazebo reference="base_link_mb">
+    <sensor name="base_link_mb" type="contact">
+      <update_rate>1000.0</update_rate>
+      <always_on>true</always_on>
+      <contact>
+        <collision>base_footprint_fixed_joint_lump__base_link_collision</collision>
+      </contact>
+      <plugin filename="libgazebo_ros_bumper.so" name="base_link_contact_sensor_plugin">
+        <bumperTopicName>contact</bumperTopicName>
+        <frameName>world</frameName>
+      </plugin>
+    </sensor>
+  </gazebo>
+  <gazebo reference="base_link_mb">
+    <material>Gazebo/DarkGrey</material>
+  </gazebo>
+  <gazebo reference="wheel_left_link">
+    <mu1>100.0</mu1>
+    <mu2>50.0</mu2>
+    <kp>500000.0</kp>
+    <kd>10.0</kd>
+    <minDepth>0.001</minDepth>
+    <maxVel>0.1</maxVel>
+    <fdir1>1 0 0</fdir1>
+    <material>Gazebo/FlatBlack</material>
+  </gazebo>
+  <gazebo reference="wheel_right_link">
+    <mu1>100.0</mu1>
+    <mu2>50.0</mu2>
+    <kp>500000.0</kp>
+    <kd>10.0</kd>
+    <minDepth>0.001</minDepth>
+    <maxVel>0.1</maxVel>
+    <fdir1>1 0 0</fdir1>
+    <material>Gazebo/FlatBlack</material>
+  </gazebo>
+  <gazebo reference="caster_back_right_link">
+    <mu1>0.01</mu1>
+    <mu2>0.01</mu2>
+    <kp>1000000.0</kp>
+    <kd>100.0</kd>
+    <minDepth>0.001</minDepth>
+    <maxVel>1.0</maxVel>
+    <material>Gazebo/FlatBlack</material>
+  </gazebo>
+  <gazebo reference="caster_back_left_link">
+    <mu1>0.01</mu1>
+    <mu2>0.01</mu2>
+    <kp>1000000.0</kp>
+    <kd>100.0</kd>
+    <minDepth>0.001</minDepth>
+    <maxVel>1.0</maxVel>
+    <material>Gazebo/FlatBlack</material>
+  </gazebo>
+  <gazebo reference="caster_front_right_link">
+    <mu1>0.01</mu1>
+    <mu2>0.01</mu2>
+    <kp>1000000.0</kp>
+    <kd>100.0</kd>
+    <minDepth>0.001</minDepth>
+    <maxVel>1.0</maxVel>
+    <material>Gazebo/FlatBlack</material>
+  </gazebo>
+  <gazebo reference="caster_front_left_link">
+    <mu1>0.01</mu1>
+    <mu2>0.01</mu2>
+    <kp>1000000.0</kp>
+    <kd>100.0</kd>
+    <minDepth>0.001</minDepth>
+    <maxVel>1.0</maxVel>
+    <material>Gazebo/FlatBlack</material>
+  </gazebo>
+  <gazebo reference="imu_link">
+    <sensor name="imu" type="imu">
+      <always_on>true</always_on>
+      <visualize>false</visualize>
+    </sensor>
+    <material>Gazebo/Grey</material>
+  </gazebo>
+  <gazebo>
+    <plugin filename="libgazebo_ros_diff_drive.so" name="moving_base_controller">
+      <commandTopic>cmd_vel</commandTopic>
+      <odometryTopic>odom</odometryTopic>
+      <odometryFrame>odom</odometryFrame>
+      <odometrySource>world</odometrySource>
+      <publishOdomTF>true</publishOdomTF>
+      <robotBaseFrame>world</robotBaseFrame>
+      <publishWheelTF>false</publishWheelTF>
+      <publishTf>true</publishTf>
+      <publishWheelJointState>true</publishWheelJointState>
+      <legacyMode>false</legacyMode>
+      <updateRate>30</updateRate>
+      <leftJoint>wheel_left_joint</leftJoint>
+      <rightJoint>wheel_right_joint</rightJoint>
+      <wheelSeparation>0.650</wheelSeparation>
+      <wheelDiameter>0.168</wheelDiameter>
+      <wheelAcceleration>1</wheelAcceleration>
+      <wheelTorque>50</wheelTorque>
+      <rosDebugLevel>na</rosDebugLevel>
+    </plugin>
+  </gazebo>
+  <gazebo>
+    <plugin filename="libgazebo_ros_imu.so" name="imu_plugin">
+      <alwaysOn>true</alwaysOn>
+      <bodyName>imu_link</bodyName>
+      <frameName>imu_link</frameName>
+      <topicName>imu</topicName>
+      <serviceName>imu_service</serviceName>
+      <gaussianNoise>0.0</gaussianNoise>
+      <updateRate>0</updateRate>
+      <imu>
+        <noise>
+          <type>gaussian</type>
+          <rate>
+            <mean>0.0</mean>
+            <stddev>2e-4</stddev>
+            <bias_mean>0.0000075</bias_mean>
+            <bias_stddev>0.0000008</bias_stddev>
+          </rate>
+          <accel>
+            <mean>0.0</mean>
+            <stddev>1.7e-2</stddev>
+            <bias_mean>0.1</bias_mean>
+            <bias_stddev>0.001</bias_stddev>
+          </accel>
+        </noise>
+      </imu>
+    </plugin>
+  </gazebo>
+  <link name="base_link_mb">
+    <visual>
+      <origin xyz="-0.43 -0.33 0.03" rpy="1.5707963267948966 0.0 1.5707963267948966"/>
+      <geometry>
+        <mesh filename="package://ur_e_description/meshes/moving_base/moving_base.STL" scale="0.001 0.001 0.001"/>
+      </geometry>
+      <material name="light_black"/>
+    </visual>
+    <collision>
+      <origin xyz="0.0 0.0 0.459" rpy="0.0 0.0 0.0"/>
+      <geometry>
+        <box size="0.9 0.6 0.77"/>
+      </geometry>
+    </collision>
+  </link>
+  <link name="inertial_link">
+    <inertial>
+      <origin xyz="-0.00065 -0.085 0.062" rpy="0.0 0.0 0.0"/>
+      <mass value="46.034"/>
+      <inertia ixx="0.6022" ixy="-0.02364" ixz="-0.1197" iyy="1.7386" iyz="-0.001544" izz="2.0296"/>
+    </inertial>
+  </link>
+  <joint name="inertial_joint" type="fixed">
+    <origin xyz="0.0 0.0 0.0" rpy="0.0 0.0 0.0"/>
+    <parent link="base_link_mb"/>
+    <child link="inertial_link"/>
+  </joint>
+  <joint name="wheel_left_joint" type="continuous">
+    <origin xyz="0.0 0.325 0.074" rpy="-1.57 0.0 0.0"/>
+    <axis xyz="0.0 0.0 1.0"/>
+    <parent link="base_link_mb"/>
+    <child link="wheel_left_link"/>
+  </joint>
+  <link name="wheel_left_link">
+    <inertial>
+      <origin xyz="0.0 0.0 0.0" rpy="0.0 0.0 0.0"/>
+      <mass value="0.02849894"/>
+      <inertia ixx="1.117558e-05" ixy="-4.2369783e-11" ixz="-5.9381719e-09" iyy="1.1192413e-05" iyz="-1.4400107e-11" izz="2.0712558e-05"/>
+    </inertial>
+    <visual>
+      <origin xyz="0.0 0.0 -0.055" rpy="-1.57 0.0 0.0"/>
+      <geometry>
+        <mesh filename="package://ur_e_description/meshes/wheels/left_tire.stl" scale="0.0025 0.0025 0.0025"/>
+      </geometry>
+      <material name="dark"/>
+    </visual>
+    <collision>
+      <origin xyz="0.0 0.0 0.0" rpy="0.0 0.0 0.0"/>
+      <geometry>
+        <cylinder radius="0.084" length="0.044"/>
+      </geometry>
+    </collision>
+  </link>
+  <joint name="wheel_right_joint" type="continuous">
+    <origin xyz="0.0 -0.325 0.074" rpy="-1.57 0.0 0.0"/>
+    <axis xyz="0.0 0.0 1.0"/>
+    <parent link="base_link_mb"/>
+    <child link="wheel_right_link"/>
+  </joint>
+  <link name="wheel_right_link">
+    <inertial>
+      <origin xyz="0.0 0.0 0.0" rpy="0.0 0.0 0.0"/>
+      <mass value="0.02849894"/>
+      <inertia ixx="1.117558e-05" ixy="-4.2369783e-11" ixz="-5.9381719e-09" iyy="1.1192413e-05" iyz="-1.4400107e-11" izz="2.0712558e-05"/>
+    </inertial>
+    <visual>
+      <origin xyz="0.0 0.0 0.055" rpy="1.57 0.0 0.0"/>
+      <geometry>
+        <mesh filename="package://ur_e_description/meshes/wheels/left_tire.stl" scale="0.0025 0.0025 0.0025"/>
+      </geometry>
+      <material name="dark"/>
+    </visual>
+    <collision>
+      <origin xyz="0.0 0.0 0.0" rpy="0.0 0.0 0.0"/>
+      <geometry>
+        <cylinder radius="0.084" length="0.044"/>
+      </geometry>
+    </collision>
+  </link>
+  <joint name="caster_back_right_joint" type="fixed">
+    <origin xyz="-0.345 -0.19 -0.004" rpy="-1.57 0.0 0.0"/>
+    <parent link="base_link_mb"/>
+    <child link="caster_back_right_link"/>
+  </joint>
+  <link name="caster_back_right_link">
+    <inertial>
+      <origin xyz="0.0 0.0 0.0" rpy="0.0 0.0 0.0"/>
+      <mass value="0.005"/>
+      <inertia ixx="0.001" ixy="0.0" ixz="0.0" iyy="0.001" iyz="0.0" izz="0.001"/>
+    </inertial>
+    <visual>
+      <origin xyz="0.027 -0.06 0.0" rpy="1.57 0.0 0.0"/>
+      <geometry>
+        <mesh filename="package://ur_e_description/meshes/wheels/left_tire.stl" scale="0.002 0.002 0.002"/>
+      </geometry>
+      <material name="dark"/>
+    </visual>
+    <collision>
+      <origin xyz="0.0 0.001 0.0" rpy="0.0 0.0 0.0"/>
+      <geometry>
+        <box size="0.03 0.009 0.078"/>
+      </geometry>
+    </collision>
+  </link>
+  <joint name="caster_back_left_joint" type="fixed">
+    <origin xyz="-0.345 0.19 -0.004" rpy="-1.57 0.0 0.0"/>
+    <parent link="base_link_mb"/>
+    <child link="caster_back_left_link"/>
+  </joint>
+  <link name="caster_back_left_link">
+    <inertial>
+      <origin xyz="0.0 0.0 0.0" rpy="0.0 0.0 0.0"/>
+      <mass value="0.005"/>
+      <inertia ixx="0.001" ixy="0.0" ixz="0.0" iyy="0.001" iyz="0.0" izz="0.001"/>
+    </inertial>
+    <visual>
+      <origin xyz="0.027 -0.06 0.0" rpy="-1.57 0.0 0.0"/>
+      <geometry>
+        <mesh filename="package://ur_e_description/meshes/wheels/left_tire.stl" scale="0.002 0.002 0.002"/>
+      </geometry>
+      <material name="dark"/>
+    </visual>
+    <collision>
+      <origin xyz="0.0 0.001 0.0" rpy="0.0 0.0 0.0"/>
+      <geometry>
+        <box size="0.03 0.009 0.078"/>
+      </geometry>
+    </collision>
+  </link>
+  <joint name="caster_front_right_joint" type="fixed">
+    <origin xyz="0.345 -0.19 -0.004" rpy="-1.57 0.0 0.0"/>
+    <parent link="base_link_mb"/>
+    <child link="caster_front_right_link"/>
+  </joint>
+  <link name="caster_front_right_link">
+    <inertial>
+      <origin xyz="0.0 0.0 0.0" rpy="0.0 0.0 0.0"/>
+      <mass value="0.005"/>
+      <inertia ixx="0.001" ixy="0.0" ixz="0.0" iyy="0.001" iyz="0.0" izz="0.001"/>
+    </inertial>
+    <visual>
+      <origin xyz="0.0 -0.06 0.0" rpy="1.57 0.0 0.0"/>
+      <geometry>
+        <mesh filename="package://ur_e_description/meshes/wheels/left_tire.stl" scale="0.002 0.002 0.002"/>
+      </geometry>
+      <material name="dark"/>
+    </visual>
+    <collision>
+      <origin xyz="0.0 0.001 0.0" rpy="0.0 0.0 0.0"/>
+      <geometry>
+        <box size="0.03 0.009 0.078"/>
+      </geometry>
+    </collision>
+  </link>
+  <joint name="caster_front_left_joint" type="fixed">
+    <origin xyz="0.345 0.19 -0.004" rpy="-1.57 0.0 0.0"/>
+    <parent link="base_link_mb"/>
+    <child link="caster_front_left_link"/>
+  </joint>
+  <link name="caster_front_left_link">
+    <inertial>
+      <origin xyz="0.0 0.0 0.0" rpy="0.0 0.0 0.0"/>
+      <mass value="0.005"/>
+      <inertia ixx="0.001" ixy="0.0" ixz="0.0" iyy="0.001" iyz="0.0" izz="0.001"/>
+    </inertial>
+    <visual>
+      <origin xyz="0.0 -0.06 0.0" rpy="-1.57 0.0 0.0"/>
+      <geometry>
+        <mesh filename="package://ur_e_description/meshes/wheels/left_tire.stl" scale="0.002 0.002 0.002"/>
+      </geometry>
+      <material name="dark"/>
+    </visual>
+    <collision>
+      <origin xyz="0.0 0.001 0.0" rpy="0.0 0.0 0.0"/>
+      <geometry>
+        <box size="0.03 0.009 0.078"/>
+      </geometry>
+    </collision>
+  </link>
+  <joint name="imu_joint" type="fixed">
+    <origin xyz="0.0 0.0 0.068" rpy="0.0 0.0 0.0"/>
+    <parent link="base_link_mb"/>
+    <child link="imu_link"/>
+  </joint>
+  <link name="imu_link"/>
   <joint name="moving_base_to_ur5e" type="fixed">
-    <parent link="base_link_mb" />
-    <child link="base_link" />
     <origin xyz="-0.296 -0.1688 0.826" rpy="0.0 0.0 0.0"/>
-  </joint> -->
-  <!-- THIS PART WAS MOVED TO UR5E.URDF.XACRO  -->
-  <!-- <link name="base_footprint" /> -->
-  <!-- initial robot pose on world - FROM ORIGINAL FILE -->
-  <!-- toogle this part to move the AGV in odom -->
-  <link name="world" />
+    <parent link="base_link_mb"/>
+    <child link="base_link"/>
+  </joint>
+  <link name="base_link">
+    <inertial>
+      <origin xyz="0.0 0.0 0.0" rpy="0.0 0.0 0.0"/>
+      <mass value="4.0"/>
+      <inertia ixx="0.00443333156" ixy="0.0" ixz="0.0" iyy="0.00443333156" iyz="0.0" izz="0.0072"/>
+    </inertial>
+    <visual>
+      <geometry>
+        <mesh filename="package://ur_e_description/meshes/ur5e/visual/base.dae"/>
+      </geometry>
+      <material name="LightGrey">
+        <color rgba="0.7 0.7 0.7 1.0"/>
+      </material>
+    </visual>
+    <collision>
+      <geometry>
+        <mesh filename="package://ur_e_description/meshes/ur5e/collision/base.stl"/>
+      </geometry>
+    </collision>
+  </link>
+  <joint name="shoulder_pan_joint" type="revolute">
+    <origin xyz="0.0 0.0 0.163" rpy="0.0 0.0 0.0"/>
+    <axis xyz="0.0 0.0 1.0"/>
+    <parent link="base_link"/>
+    <child link="shoulder_link"/>
+    <limit effort="150.0" lower="-3.141592653589793" upper="3.141592653589793" velocity="3.14"/>
+    <dynamics damping="0.0" friction="0.0"/>
+  </joint>
+  <link name="shoulder_link">
+    <inertial>
+      <origin xyz="0.0 0.0 0.0" rpy="0.0 0.0 0.0"/>
+      <mass value="3.7"/>
+      <inertia ixx="0.010267495893" ixy="0.0" ixz="0.0" iyy="0.010267495893" iyz="0.0" izz="0.00666"/>
+    </inertial>
+    <visual>
+      <geometry>
+        <mesh filename="package://ur_e_description/meshes/ur5e/visual/shoulder.dae"/>
+      </geometry>
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
Commit message: zau v1

File: e0_rgb2ee/e0_rgb2ee_calibration/urdf/initial_estimate.urdf.xacro (robot description, xacro)
@@ -160,5 +160,5 @@
   <link name="inertial_link">
     <inertial>
-      <origin xyz="-0.00065 -0.085 0.062" rpy="0.0 0.0 0.0"/>
+      <origin xyz="-0.00065 -0.085 0.062" rpy="0 0 0"/>
       <mass value="46.034"/>
       <inertia ixx="0.6022" ixy="-0.02364" ixz="-0.1197" iyy="1.7386" iyz="-0.001544" izz="2.0296"/>
@@ -178,5 +178,5 @@
   <link name="wheel_left_link">
     <inertial>
-      <origin xyz="0.0 0.0 0.0" rpy="0.0 0.0 0.0"/>
+      <origin xyz="0.0 0.0 0.0" rpy="0 0 0"/>
       <mass value="0.02849894"/>
       <inertia ixx="1.117558e-05" ixy="-4.2369783e-11" ixz="-5.9381719e-09" iyy="1.1192413e-05" iyz="-1.4400107e-11" izz="2.0712558e-05"/>
@@ -204,5 +204,5 @@
   <link name="wheel_right_link">
     <inertial>
-      <origin xyz="0.0 0.0 0.0" rpy="0.0 0.0 0.0"/>
+      <origin xyz="0.0 0.0 0.0" rpy="0 0 0"/>
       <mass value="0.02849894"/>
       <inertia ixx="1.117558e-05" ixy="-4.2369783e-11" ixz="-5.9381719e-09" iyy="1.1192413e-05" iyz="-1.4400107e-11" izz="2.0712558e-05"/>
@@ -229,5 +229,5 @@
   <link name="caster_back_right_link">
     <inertial>
-      <origin xyz="0.0 0.0 0.0" rpy="0.0 0.0 0.0"/>
+      <origin xyz="0.0 0.0 0.0" rpy="0 0 0"/>
       <mass value="0.005"/>
       <inertia ixx="0.001" ixy="0.0" ixz="0.0" iyy="0.001" iyz="0.0" izz="0.001"/>
@@ -254,5 +254,5 @@
   <link name="caster_back_left_link">
     <inertial>
-      <origin xyz="0.0 0.0 0.0" rpy="0.0 0.0 0.0"/>
+      <origin xyz="0.0 0.0 0.0" rpy="0 0 0"/>
       <mass value="0.005"/>
       <inertia ixx="0.001" ixy="0.0" ixz="0.0" iyy="0.001" iyz="0.0" izz="0.001"/>
@@ -279,5 +279,5 @@
   <link name="caster_front_right_link">
     <inertial>
-      <origin xyz="0.0 0.0 0.0" rpy="0.0 0.0 0.0"/>
+      <origin xyz="0.0 0.0 0.0" rpy="0 0 0"/>
       <mass value="0.005"/>
       <inertia ixx="0.001" ixy="0.0" ixz="0.0" iyy="0.001" iyz="0.0" izz="0.001"/>
@@ -304,5 +304,5 @@
   <link name="caster_front_left_link">
     <inertial>
-      <origin xyz="0.0 0.0 0.0" rpy="0.0 0.0 0.0"/>
+      <origin xyz="0.0 0.0 0.0" rpy="0 0 0"/>
       <mass value="0.005"/>
       <inertia ixx="0.001" ixy="0.0" ixz="0.0" iyy="0.001" iyz="0.0" izz="0.001"/>
@@ -623,5 +623,5 @@
   </joint>
   <joint name="camera_joint" type="fixed">
-    <origin xyz="0.0600758568472458 -0.07451415139078899 0.04999473796135022" rpy="-3.141483156142495 -0.0009436775284828712 0.0005450844558930153"/>
+    <origin xyz="0.0600758568472458 -0.07451415139078899 0.04999473796135022" rpy="-3.141483156142495 -0.0009436775284828712 0.000545084455893016"/>
     <parent link="ee_link"/>
     <child link="camera_link"/>
@@ -629,5 +629,5 @@
   <link name="camera_link">
     <inertial>
-      <origin xyz="0.0 0.0 0.0" rpy="0.0 0.0 0.0"/>
+      <origin xyz="0.0 0.0 0.0" rpy="0 0 0"/>
       <mass value="0.564"/>
       <inertia ixx="0.003881243" ixy="0.0" ixz="0.0" iyy="0.00049894" iyz="0.0" izz="0.003879257"/>
