Commit message: run configure calibration

File: Zau_INESCTEC/zau_eye_on_hand_calibration/urdf/initial_estimate.urdf.xacro (robot description, xacro)
@@ -1,400 +1,61 @@
-<?xml version="1.0" ?>
-<robot name="ur5e" version="1.0">
-  <gazebo>
-    <plugin filename="libgazebo_ros_control.so" name="ros_control">
-    </plugin>
-  </gazebo>
-  <link name="base_link">
-    <inertial>
-      <origin xyz="0.0 0.0 0.0" rpy="0.0 0.0 0.0"/>
-      <mass value="4.0"/>
-      <inertia ixx="0.00443333156" ixy="0.0" ixz="0.0" iyy="0.00443333156" iyz="0.0" izz="0.0072"/>
-    </inertial>
-    <visual>
-      <geometry>
-        <mesh filename="package://ur_e_description/meshes/ur5e/visual/base.dae"/>
-      </geometry>
-      <material name="LightGrey">
-        <color rgba="0.7 0.7 0.7 1.0"/>
-      </material>
-    </visual>
-    <collision>
-      <geometry>
-        <mesh filename="package://ur_e_description/meshes/ur5e/collision/base.stl"/>
-      </geometry>
-    </collision>
-  </link>
-  <joint name="shoulder_pan_joint" type="revolute">
-    <origin xyz="0.0 0.0 0.163" rpy="0.0 0.0 0.0"/>
-    <axis xyz="0.0 0.0 1.0"/>
-    <parent link="base_link"/>
-    <child link="shoulder_link"/>
-    <limit effort="150.0" lower="-3.141592653589793" upper="3.141592653589793" velocity="3.14"/>
-    <dynamics damping="0.0" friction="0.0"/>
-  </joint>
-  <link name="shoulder_link">
-    <inertial>
-      <origin xyz="0.0 0.0 0.0" rpy="0.0 0.0 0.0"/>
-      <mass value="3.7"/>
-      <inertia ixx="0.010267495893" ixy="0.0" ixz="0.0" iyy="0.010267495893" iyz="0.0" izz="0.00666"/>
-    </inertial>
-    <visual>
-      <geometry>
-        <mesh filename="package://ur_e_description/meshes/ur5e/visual/shoulder.dae"/>
-      </geometry>
-      <material name="LightGrey">
-        <color rgba="0.7 0.7 0.7 1.0"/>
-      </material>
-    </visual>
-    <collision>
-      <geometry>
-        <mesh filename="package://ur_e_description/meshes/ur5e/collision/shoulder.stl"/>
-      </geometry>
-    </collision>
-  </link>
-  <joint name="shoulder_lift_joint" type="revolute">
-    <origin xyz="0.0 0.138 0.0" rpy="0.0 1.5707963267948966 0.0"/>
-    <axis xyz="0.0 1.0 0.0"/>
-    <parent link="shoulder_link"/>
-    <child link="upper_arm_link"/>
-    <limit effort="150.0" lower="-3.141592653589793" upper="3.141592653589793" velocity="3.14"/>
-    <dynamics damping="0.0" friction="0.0"/>
-  </joint>
-  <link name="upper_arm_link">
-    <inertial>
-      <origin xyz="0.0 0.0 0.2125" rpy="0.0 0.0 0.0"/>
-      <mass value="8.393"/>
-      <inertia ixx="0.1338857818623325" ixy="0.0" ixz="0.0" iyy="0.1338857818623325" iyz="0.0" izz="0.0151074"/>
-    </inertial>
-    <visual>
-      <geometry>
-        <mesh filename="package://ur_e_description/meshes/ur5e/visual/upperarm.dae"/>
-      </geometry>
-      <material name="LightGrey">
-        <color rgba="0.7 0.7 0.7 1.0"/>
-      </material>
-    </visual>
-    <collision>
-      <geometry>
-        <mesh filename="package://ur_e_description/meshes/ur5e/collision/upperarm.stl"/>
-      </geometry>
-    </collision>
-  </link>
-  <joint name="elbow_joint" type="revolute">
-    <origin xyz="0.0 -0.131 0.425" rpy="0.0 0.0 0.0"/>
-    <axis xyz="0.0 1.0 0.0"/>
-    <parent link="upper_arm_link"/>
-    <child link="forearm_link"/>
-    <limit effort="150.0" lower="-3.141592653589793" upper="3.141592653589793" velocity="3.14"/>
-    <dynamics damping="0.0" friction="0.0"/>
-  </joint>
-  <link name="forearm_link">
-    <inertial>
-      <origin xyz="0.0 0.0 0.196" rpy="0.0 0.0 0.0"/>
-      <mass value="2.275"/>
-      <inertia ixx="0.031179620861480004" ixy="0.0" ixz="0.0" iyy="0.031179620861480004" iyz="0.0" izz="0.004095"/>
-    </inertial>
-    <visual>
-      <geometry>
-        <mesh filename="package://ur_e_description/meshes/ur5e/visual/forearm.dae"/>
-      </geometry>
-      <material name="LightGrey">
-        <color rgba="0.7 0.7 0.7 1.0"/>
-      </material>
-    </visual>
-    <collision>
-      <geometry>
-        <mesh filename="package://ur_e_description/meshes/ur5e/collision/forearm.stl"/>
-      </geometry>
-    </collision>
-  </link>
-  <joint name="wrist_1_joint" type="revolute">
-    <origin xyz="0.0 0.0 0.392" rpy="0.0 1.5707963267948966 0.0"/>
-    <axis xyz="0.0 1.0 0.0"/>
-    <parent link="forearm_link"/>
-    <child link="wrist_1_link"/>
-    <limit effort="28.0" lower="-3.141592653589793" upper="3.141592653589793" velocity="6.28"/>
-    <dynamics damping="0.0" friction="0.0"/>
-  </joint>
-  <link name="wrist_1_link">
-    <inertial>
-      <origin xyz="0.0 0.127 0.0" rpy="0.0 0.0 0.0"/>
-      <mass value="1.219"/>
-      <inertia ixx="0.0025598989760400002" ixy="0.0" ixz="0.0" iyy="0.0025598989760400002" iyz="0.0" izz="0.0021942"/>
-    </inertial>
-    <visual>
-      <geometry>
-        <mesh filename="package://ur_e_description/meshes/ur5e/visual/wrist1.dae"/>
-      </geometry>
-      <material name="LightGrey">
-        <color rgba="0.7 0.7 0.7 1.0"/>
-      </material>
-    </visual>
-    <collision>
-      <geometry>
-        <mesh filename="package://ur_e_description/meshes/ur5e/collision/wrist1.stl"/>
-      </geometry>
-    </collision>
-  </link>
-  <joint name="wrist_2_joint" type="revolute">
-    <origin xyz="0.0 0.127 0.0" rpy="0.0 0.0 0.0"/>
-    <axis xyz="0.0 0.0 1.0"/>
-    <parent link="wrist_1_link"/>
-    <child link="wrist_2_link"/>
-    <limit effort="28.0" lower="-3.141592653589793" upper="3.141592653589793" velocity="6.28"/>
-    <dynamics damping="0.0" friction="0.0"/>
-  </joint>
-  <link name="wrist_2_link">
-    <inertial>
-      <origin xyz="0.0 0.0 0.1" rpy="0.0 0.0 0.0"/>
-      <mass value="1.219"/>
-      <inertia ixx="0.0025598989760400002" ixy="0.0" ixz="0.0" iyy="0.0025598989760400002" iyz="0.0" izz="0.0021942"/>
-    </inertial>
-    <visual>
-      <geometry>
-        <mesh filename="package://ur_e_description/meshes/ur5e/visual/wrist2.dae"/>
-      </geometry>
-      <material name="LightGrey">
-        <color rgba="0.7 0.7 0.7 1.0"/>
-      </material>
-    </visual>
-    <collision>
-      <geometry>
-        <mesh filename="package://ur_e_description/meshes/ur5e/collision/wrist2.stl"/>
-      </geometry>
-    </collision>
-  </link>
-  <joint name="wrist_3_joint" type="revolute">
-    <origin xyz="0.0 0.0 0.1" rpy="0.0 0.0 0.0"/>
-    <axis xyz="0.0 1.0 0.0"/>
-    <parent link="wrist_2_link"/>
-    <child link="wrist_3_link"/>
-    <limit effort="28.0" lower="-3.141592653589793" upper="3.141592653589793" velocity="6.28"/>
-    <dynamics damping="0.0" friction="0.0"/>
-  </joint>
-  <link name="wrist_3_link">
-    <inertial>
-      <origin xyz="0.0 0.0771 0.0" rpy="1.5707963267948966 0.0 0.0"/>
-      <mass value="0.1879"/>
-      <inertia ixx="9.890410052167731e-05" ixy="0.0" ixz="0.0" iyy="9.890410052167731e-05" iyz="0.0" izz="0.0001321171875"/>
-    </inertial>
-    <visual>
-      <geometry>
-        <mesh filename="package://ur_e_description/meshes/ur5e/visual/wrist3.dae"/>
-      </geometry>
-      <material name="LightGrey">
-        <color rgba="0.7 0.7 0.7 1.0"/>
-      </material>
-    </visual>
-    <collision>
-      <geometry>
-        <mesh filename="package://ur_e_description/meshes/ur5e/collision/wrist3.stl"/>
-      </geometry>
-    </collision>
-  </link>
-  <joint name="ee_fixed_joint" type="fixed">
-    <origin xyz="0.0 0.1 0.0" rpy="0.0 0.0 1.5707963267948966"/>
-    <parent link="wrist_3_link"/>
-    <child link="ee_link"/>
-  </joint>
-  <link name="ee_link">
-    <collision>
-      <origin xyz="-0.01 0.0 0.0" rpy="0.0 0.0 0.0"/>
-      <geometry>
-        <box size="0.01 0.01 0.01"/>
-      </geometry>
-    </collision>
-  </link>
-  <link name="ee_camera_support_link">
-    <visual>
-      <origin xyz="0.0 0.0 0.0" rpy="0.0 0.0 0.0"/>
-      <geometry>
-        <box size="0.185 0.03 0.03"/>
-      </geometry>
-      <material name="LightGrey">
-        <color rgba="0.7 0.7 0.7 1.0"/>
-      </material>
-    </visual>
-  </link>
-  <joint name="ee_camera_support_joint" type="fixed">
-    <origin xyz="0.095 0.0 0.0" rpy="0.0 0.0 0.0"/>
-    <parent link="ee_link"/>
-    <child link="ee_camera_support_link"/>
-  </joint>
-  <link name="ee_camera_support_small_link">
-    <visual>
-      <origin xyz="0.0 0.0 0.0" rpy="0.0 0.0 0.0"/>
-      <geometry>
-        <box size="0.02 0.02 0.065"/>
-      </geometry>
-      <material name="LightGrey">
-        <color rgba="0.7 0.7 0.7 1.0"/>
-      </material>
-    </visual>
-  </link>
-  <joint name="ee_camera_support_small_joint" type="fixed">
-    <origin xyz="0.0 0.0 -0.04" rpy="0.0 0.0 0.0"/>
-    <parent link="ee_camera_support_link"/>
-    <child link="ee_camera_support_small_link"/>
-  </joint>
-  <material name="aluminum">
-    <color rgba="0.5 0.5 0.5 1.0"/>
-  </material>
-  <material name="plastic">
-    <color rgba="0.1 0.1 0.1 1.0"/>
-  </material>
-  <joint name="camera_joint" type="fixed">
-    <origin xyz="0.095 0.0 -0.075" rpy="-3.14 0.0 1.57"/>
-    <parent link="ee_link"/>
-    <child link="camera_bottom_screw_frame"/>
-  </joint>
-  <link name="camera_bottom_screw_frame"/>
-  <joint name="camera_link_joint" type="fixed">
-    <origin xyz="0.0 0.02 0.0115" rpy="0.0 0.0 0.0"/>
-    <parent link="camera_bottom_screw_frame"/>
-    <child link="camera_link"/>
-  </joint>
-  <link name="camera_link">
-    <inertial>
-      <origin xyz="0.0 0.0 0.0" rpy="0 0 0"/>
-      <mass value="0.072"/>
-      <inertia ixx="0.003881243" ixy="0.0" ixz="0.0" iyy="0.00049894" iyz="0.0" izz="0.003879257"/>
-    </inertial>
-    <visual>
-      <origin xyz="0.00987 -0.02 0.0" rpy="1.5707963267948966 0.0 1.5707963267948966"/>
-      <geometry>
-        <mesh filename="package://realsense2_description/meshes/d415.stl"/>
-      </geometry>
-      <material name="aluminum"/>
-    </visual>
-    <collision>
-      <origin xyz="0.0 -0.02 0.0" rpy="0.0 0.0 0.0"/>
-      <geometry>
-        <box size="0.02005 0.099 0.023"/>
-      </geometry>
-    </collision>
-  </link>
-  <joint name="camera_depth_joint" type="fixed">
-    <origin xyz="0.0 0.0 0.0" rpy="0.0 0.0 0.0"/>
-    <parent link="camera_link"/>
-    <child link="camera_depth_frame"/>
-  </joint>
-  <link name="camera_depth_frame"/>
-  <joint name="camera_depth_optical_joint" type="fixed">
-    <origin xyz="0.0 0.0 0.0" rpy="-1.5707963267948966 0.0 -1.5707963267948966"/>
-    <parent link="camera_depth_frame"/>
-    <child link="camera_depth_optical_frame"/>
-  </joint>
-  <link name="camera_depth_optical_frame"/>
-  <joint name="camera_infra1_joint" type="fixed">
-    <origin xyz="0.0 0.0 0.0" rpy="0.0 0.0 0.0"/>
-    <parent link="camera_link"/>
-    <child link="camera_infra1_frame"/>
-  </joint>
-  <link name="camera_infra1_frame"/>
-  <joint name="camera_infra1_optical_joint" type="fixed">
-    <origin xyz="0.0 0.0 0.0" rpy="-1.5707963267948966 0.0 -1.5707963267948966"/>
-    <parent link="camera_infra1_frame"/>
-    <child link="camera_infra1_optical_frame"/>
-  </joint>
-  <link name="camera_infra1_optical_frame"/>
-  <joint name="camera_infra2_joint" type="fixed">
-    <origin xyz="0.0 -0.055 0.0" rpy="0.0 0.0 0.0"/>
-    <parent link="camera_link"/>
-    <child link="camera_infra2_frame"/>
-  </joint>
-  <link name="camera_infra2_frame"/>
-  <joint name="camera_infra2_optical_joint" type="fixed">
-    <origin xyz="0.0 0.0 0.0" rpy="-1.5707963267948966 0.0 -1.5707963267948966"/>
-    <parent link="camera_infra2_frame"/>
-    <child link="camera_infra2_optical_frame"/>
-  </joint>
-  <link name="camera_infra2_optical_frame"/>
-  <joint name="camera_color_joint" type="fixed">
-    <origin xyz="0.0 0.015 0.0" rpy="0.0 -0.0 0.0"/>
-    <parent link="camera_link"/>
-    <child link="camera_color_frame"/>
-  </joint>
-  <link name="camera_color_frame"/>
-  <joint name="camera_color_optical_joint" type="fixed">
-    <origin xyz="0.0 0.0 0.0" rpy="-1.5707963267948966 0.0 -1.5707963267948966"/>
-    <parent link="camera_color_frame"/>
-    <child link="camera_color_optical_frame"/>
-  </joint>
-  <link name="camera_color_optical_frame"/>
-  <transmission name="shoulder_pan_trans">
-    <type>transmission_interface/SimpleTransmission</type>
-    <joint name="shoulder_pan_joint">
-      <hardwareInterface>hardware_interface/PositionJointInterface</hardwareInterface>
-    </joint>
-    <actuator name="shoulder_pan_motor">
-      <mechanicalReduction>1.0</mechanicalReduction>
-    </actuator>
-  </transmission>
-  <transmission name="shoulder_lift_trans">
-    <type>transmission_interface/SimpleTransmission</type>
-    <joint name="shoulder_lift_joint">
-      <hardwareInterface>hardware_interface/PositionJointInterface</hardwareInterface>
-    </joint>
-    <actuator name="shoulder_lift_motor">
-      <mechanicalReduction>1.0</mechanicalReduction>
-    </actuator>
-  </transmission>
-  <transmission name="elbow_trans">
-    <type>transmission_interface/SimpleTransmission</type>
-    <joint name="elbow_joint">
-      <hardwareInterface>hardware_interface/PositionJointInterface</hardwareInterface>
-    </joint>
-    <actuator name="elbow_motor">
-      <mechanicalReduction>1.0</mechanicalReduction>
-    </actuator>
-  </transmission>
-  <transmission name="wrist_1_trans">
-    <type>transmission_interface/SimpleTransmission</type>
-    <joint name="wrist_1_joint">
-      <hardwareInterface>hardware_interface/PositionJointInterface</hardwareInterface>
-    </joint>
-    <actuator name="wrist_1_motor">
-      <mechanicalReduction>1.0</mechanicalReduction>
-    </actuator>
-  </transmission>
-  <transmission name="wrist_2_trans">
-    <type>transmission_interface/SimpleTransmission</type>
-    <joint name="wrist_2_joint">
-      <hardwareInterface>hardware_interface/PositionJointInterface</hardwareInterface>
-    </joint>
-    <actuator name="wrist_2_motor">
-      <mechanicalReduction>1.0</mechanicalReduction>
-    </actuator>
-  </transmission>
-  <transmission name="wrist_3_trans">
-    <type>transmission_interface/SimpleTransmission</type>
-    <joint name="wrist_3_joint">
-      <hardwareInterface>hardware_interface/PositionJointInterface</hardwareInterface>
-    </joint>
-    <actuator name="wrist_3_motor">
-      <mechanicalReduction>1.0</mechanicalReduction>
-    </actuator>
-  </transmission>
-  <gazebo reference="shoulder_link">
-    <selfCollide>true</selfCollide>
-  </gazebo>
-  <gazebo reference="upper_arm_link">
-    <selfCollide>true</selfCollide>
-  </gazebo>
-  <gazebo reference="forearm_link">
-    <selfCollide>true</selfCollide>
-  </gazebo>
-  <gazebo reference="wrist_1_link">
-    <selfCollide>true</selfCollide>
-  </gazebo>
-  <gazebo reference="wrist_3_link">
-    <selfCollide>true</selfCollide>
-  </gazebo>
-  <gazebo reference="wrist_2_link">
-    <selfCollide>true</selfCollide>
-  </gazebo>
-  <gazebo reference="ee_link">
-    <selfCollide>true</selfCollide>
-  </gazebo>
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