Commit message: add modifications to the system to perform eye on hand calibration

File: UR5/ur_e_description/urdf/realsense/intel_realsense.urdf.xacro (robot description, xacro)
@@ -1,97 +1,133 @@
 <?xml version="1.0"?>
-<robot xmlns:xacro="http://ros.org/wiki/xacro">
-  <xacro:macro name="intel_realsense_mount" params="prefix topic parent_link">
-    <xacro:macro name="intel_realsense" params="
-               frame:=realsense          topic:=realsense
-               h_fov:=1.5184351666666667 v_fov:=1.0122901111111111
-               min_range:=0.105          max_range:=8.0
-               width:=640                height:=480
-               update_rate:=30
-               robot_namespace:=/">
-      <!-- this link is the origin for the camera's data -->
-      <link name="${frame}" />
-      <!--
-        The gazebo plugin aligns the depth data with the Z axis, with X=left and Y=up
-        ROS expects the depth data along the X axis, with Y=left and Z=up
-        This link only exists to give the gazebo plugin the correctly-oriented frame
-      -->
-      <link name="${frame}_gazebo" />
-      <joint name="${frame}_gazebo_joint" type="fixed">
-        <parent link="${frame}"/>
-        <child link="${frame}_gazebo"/>
-        <origin xyz="0.0 0 0" rpy="-1.5707963267948966 0 -1.5707963267948966"/>
+<!--
+License: Apache 2.0. See LICENSE file in root directory.
+Copyright(c) 2017 Intel Corporation. All Rights Reserved
+This is the URDF model for the Intel RealSense 415 camera, in its
+aluminum peripherial evaluation case.
+-->
+<robot name="sensor_d415" xmlns:xacro="http://ros.org/wiki/xacro">
+  <!-- Includes -->
+  <xacro:include filename="$(find realsense2_description)/urdf/_materials.urdf.xacro" />
+  <xacro:include filename="$(find realsense2_description)/urdf/_usb_plug.urdf.xacro" />
+  <xacro:macro name="sensor_d415" params="parent *origin  name:=camera  use_nominal_extrinsics:=false add_plug:=false use_mesh:=true">
+    <xacro:property name="M_PI" value="3.1415926535897931" />
+    <!-- The following values are approximate, and the camera node
+     publishing TF values with actual calibrated camera extrinsic values -->
+    <xacro:property name="d415_cam_depth_to_infra1_offset" value="0.0"/>
+    <xacro:property name="d415_cam_depth_to_infra2_offset" value="-0.055"/>
+    <xacro:property name="d415_cam_depth_to_color_offset" value="0.015"/>
+    <!-- The following values model the aluminum peripherial case for the
+  	d415 camera, with the camera joint represented by the actual
+  	peripherial camera tripod mount -->
+    <xacro:property name="d415_cam_width" value="0.099"/>
+    <xacro:property name="d415_cam_height" value="0.023"/>
+    <xacro:property name="d415_cam_depth" value="0.02005"/>
+    <xacro:property name="d415_cam_mount_from_center_offset" value="0.00987"/>
+    <!-- The following offset is relative the the physical d415 camera peripherial
+  	camera tripod mount -->
+    <xacro:property name="d415_cam_depth_px" value="${d415_cam_mount_from_center_offset}"/>
+    <xacro:property name="d415_cam_depth_py" value="0.020"/>
+    <xacro:property name="d415_cam_depth_pz" value="${d415_cam_height/2}"/>
+    <!-- camera body, with origin at bottom screw mount -->
+    <joint name="${name}_joint" type="fixed">
+      <xacro:insert_block name="origin" />
+      <parent link="${parent}"/>
+      <child link="${name}_bottom_screw_frame" />
+    </joint>
+    <link name="${name}_bottom_screw_frame"/>
+    <joint name="${name}_link_joint" type="fixed">
+      <origin xyz="0 ${d415_cam_depth_py} ${d415_cam_depth_pz}" rpy="0 0 0"/>
+      <parent link="${name}_bottom_screw_frame"/>
+      <child link="${name}_link" />
+    </joint>
+    <link name="${name}_link">
+      <visual>
+        <xacro:if value="${use_mesh}">
+          <origin xyz="${d415_cam_mount_from_center_offset} ${-d415_cam_depth_py} 0" rpy="${M_PI/2} 0 ${M_PI/2}"/>
+          <geometry>
+            <mesh filename="package://realsense2_description/meshes/d415.stl" />
+          </geometry>
+          <material name="aluminum"/>
+        </xacro:if>
+        <xacro:unless value="${use_mesh}">
+          <origin xyz="0 ${-d415_cam_depth_py} 0" rpy="0 0 0"/>
+          <geometry>
+            <box size="${d415_cam_depth} ${d415_cam_width} ${d415_cam_height}"/>
+          </geometry>
+        </xacro:unless>
+      </visual>
+      <collision>
+        <origin xyz="0 ${-d415_cam_depth_py} 0" rpy="0 0 0"/>
+        <geometry>
+        <box size="${d415_cam_depth} ${d415_cam_width} ${d415_cam_height}"/>
+        </geometry>
+      </collision>
+      <inertial>
+        <mass value="0.072" />
+        <!-- The following are not reliable values, and should not be used for modeling -->
+        <origin xyz="0 0 0" />
+        <inertia ixx="0.003881243" ixy="0.0" ixz="0.0" iyy="0.000498940" iyz="0.0" izz="0.003879257" />
+      </inertial>
+    </link>
+    <!-- Use the nominal extrinsics between camera frames if the calibrated extrinsics aren't being published. e.g. running the device in simulation  -->
+    <xacro:if value="${use_nominal_extrinsics}">
+      <!-- camera depth joints and links -->
+      <joint name="${name}_depth_joint" type="fixed">
+        <origin xyz="0 0 0" rpy="0 0 0"/>
+        <parent link="${name}_link"/>
+        <child link="${name}_depth_frame" />
       </joint>
-      <gazebo reference="${frame}">
-        <turnGravityOff>true</turnGravityOff>
-        <sensor type="depth" name="${prefix}_realsense_depth">
-          <update_rate>${update_rate}</update_rate>
-          <camera>
-            <!-- 75x65 degree FOV for the depth sensor -->
-            <horizontal_fov>${h_fov}</horizontal_fov>
-            <vertical_fov>${v_fov}</vertical_fov>
-            <image>
-              <width>${width}</width>
-              <height>${height}</height>
-              <!-- TODO: check what format the Realsense hardware delivers and set this to match! -->
-              <format>RGB_INT8</format>
-            </image>
-            <clip>
-              <!-- give the color sensor a maximum range of 50m so that the simulation renders nicely -->
-              <near>0.01</near>
-              <far>50.0</far>
-            </clip>
-          </camera>
-          <plugin name="kinect_controller" filename="libgazebo_ros_openni_kinect.so">
-            <baseline>0.2</baseline>
-            <alwaysOn>true</alwaysOn>
-            <updateRate>${update_rate}</updateRate>
-            <cameraName>${topic}</cameraName>
-            <imageTopicName>color/image_raw</imageTopicName>
-            <cameraInfoTopicName>color/camera_info</cameraInfoTopicName>
-            <depthImageTopicName>depth/image_rect_raw</depthImageTopicName>
-            <depthImageInfoTopicName>depth/camera_info</depthImageInfoTopicName>
-            <pointCloudTopicName>depth/color/points</pointCloudTopicName>
-            <frameName>${frame}_gazebo</frameName>
-            <pointCloudCutoff>${min_range}</pointCloudCutoff>
-            <pointCloudCutoffMax>${max_range}</pointCloudCutoffMax>
-            <distortionK1>0.00000001</distortionK1>
-            <distortionK2>0.00000001</distortionK2>
-            <distortionK3>0.00000001</distortionK3>
-            <distortionT1>0.00000001</distortionT1>
-            <distortionT2>0.00000001</distortionT2>
-            <CxPrime>0</CxPrime>
-            <Cx>0</Cx>
-            <Cy>0</Cy>
-            <focalLength>0</focalLength>
-            <hackBaseline>0</hackBaseline>
-          </plugin>
-        </sensor>
-      </gazebo>
-    </xacro:macro>
-    <link name="${prefix}_realsense_lens">
-      <visual>
-        <!--
-          the model's origin is in the middle & it's rotated to lie in
-          the optical standard with X left, Y up, and Z forward
-        -->
-        <origin xyz="0.0115 0 0.0100" rpy="1.570796 0 1.570796" />
-        <geometry>
-          <!-- Origin of this mesh is the base of the bracket. -->
-          <mesh filename="package://realsense2_description/meshes/d415.stl" />
-        </geometry>
-        <material name="realsense_color" />
-      </visual>
-    </link>
-    <joint type="fixed" name="${prefix}_realsense_lens_joint">
-      <origin xyz="0 0 0" rpy="0 0 0" />
-      <parent link="${parent_link}" />
-      <child link="${prefix}_realsense_lens" />
-    </joint>
-    <joint type="fixed" name="${prefix}_realsense_joint">
-      <origin xyz="0.025 0 0" rpy="0 0 0" />
-      <parent link="${prefix}_realsense_lens" />
-      <child link="${prefix}_realsense" />
-    </joint>
-    <xacro:intel_realsense frame="${prefix}_realsense" topic="${topic}"/>
+      <link name="${name}_depth_frame"/>
+      <joint name="${name}_depth_optical_joint" type="fixed">
+        <origin xyz="0 0 0" rpy="${-M_PI/2} 0 ${-M_PI/2}" />
+        <parent link="${name}_depth_frame" />
+        <child link="${name}_depth_optical_frame" />
+      </joint>
+      <link name="${name}_depth_optical_frame"/>
+      <!-- camera left IR joints and links -->
+      <joint name="${name}_infra1_joint" type="fixed">
+        <origin xyz="0 ${d415_cam_depth_to_infra1_offset} 0" rpy="0 0 0" />
+        <parent link="${name}_link" />
+        <child link="${name}_infra1_frame" />
+      </joint>
+      <link name="${name}_infra1_frame"/>
+      <joint name="${name}_infra1_optical_joint" type="fixed">
+        <origin xyz="0 0 0" rpy="${-M_PI/2} 0 ${-M_PI/2}" />
+        <parent link="${name}_infra1_frame" />
+        <child link="${name}_infra1_optical_frame" />
+      </joint>
+      <link name="${name}_infra1_optical_frame"/>
+      <!-- camera right IR joints and links -->
+      <joint name="${name}_infra2_joint" type="fixed">
+        <origin xyz="0 ${d415_cam_depth_to_infra2_offset} 0" rpy="0 0 0" />
+        <parent link="${name}_link" />
+        <child link="${name}_infra2_frame" />
+      </joint>
+      <link name="${name}_infra2_frame"/>
+      <joint name="${name}_infra2_optical_joint" type="fixed">
+        <origin xyz="0 0 0" rpy="${-M_PI/2} 0 ${-M_PI/2}" />
+        <parent link="${name}_infra2_frame" />
+        <child link="${name}_infra2_optical_frame" />
+      </joint>
+      <link name="${name}_infra2_optical_frame"/>
+      <!-- camera color joints and links -->
+      <joint name="${name}_color_joint" type="fixed">
+        <origin xyz="0 ${d415_cam_depth_to_color_offset} 0" rpy="0 0 0" />
+        <parent link="${name}_link" />
+        <child link="${name}_color_frame" />
+      </joint>
+      <link name="${name}_color_frame"/>
+      <joint name="${name}_color_optical_joint" type="fixed">
+        <origin xyz="0 0 0" rpy="${-M_PI/2} 0 ${-M_PI/2}" />
+        <parent link="${name}_color_frame" />
+        <child link="${name}_color_optical_frame" />
+      </joint>
+      <link name="${name}_color_optical_frame"/>
+    </xacro:if>
+    <xacro:if value="${add_plug}">
+      <xacro:usb_plug parent="${name}_link" name="${name}_usb_plug">
+        <origin xyz="${d415_cam_mount_from_center_offset - 0.01587} ${-d415_cam_depth_py - 0.0358} 0" rpy="0 0 0"/>
+      </xacro:usb_plug>
+    </xacro:if>
   </xacro:macro>
 </robot>

File: UR5/ur_e_description/urdf/ur5e.urdf.xacro (robot description, xacro)
@@ -7,11 +7,12 @@
   <!-- <xacro:include filename="$(find ur_e_description)/urdf/moving_base.urdf.xacro" /> -->
   <!-- moving AGV -->
-  <xacro:include filename="$(find ur_e_description)/urdf/moving_base_odom.urdf.xacro" />
+  <!-- <xacro:include filename="$(find ur_e_description)/urdf/moving_base_odom.urdf.xacro" />  -->
   <!-- *************THIS IS THE TRANSFORMATION TO BE CALIBRATED************* -->
-  <joint name="moving_base_to_ur5e" type="fixed">
-    <parent link="base_link_mb" />
+<!-- <link name="world"/> -->
+  <!-- <joint name="moving_base_to_ur5e" type="fixed">
+    <parent link="world" />
     <child link="base_link" />
-    <origin xyz="-0.295 0.0 0.780" rpy="0.0 0.0 0.0" />
-  </joint>
+    <origin xyz="-0.0 -0.0 0.0" rpy="0.0 0.0 0.0" />
+  </joint> -->
   <!-- place robot on moving base -->
   <xacro:macro name="cylinder_inertial" params="radius length mass *origin">
@@ -483,5 +484,8 @@
     </joint> -->
     <!-- add gripper part end ###################################################################-->
-    <!-- add camera support -->
+    <!-- SENSOR CAMERA ON END EFFECTOR -->
+    <!-- Files to add sensor camera on end-effector:
+    ur.gazebo.xacro
+    ur5e.urdf.xacro -->
     <link name="${prefix}ee_camera_support_link">
       <visual>
@@ -516,25 +520,9 @@
       <child link="${prefix}ee_camera_support_small_link" />
     </joint>
-    <!-- add intel realsense camera d415 sensor -->
-    <xacro:arg name="realsense_EE_enabled" default="$(optenv REALSENSE_EE_ENABLED 1)" />
-    <xacro:arg name="realsense_EE_topic" default="$(optenv REALSENSE_EE_TOPIC EE_realsense)" />
-    <xacro:arg name="realsense_EE_prefix"
-      default="$(optenv REALSENSE_EE_PREFIX EE_camera_realsense)" />
-    <xacro:arg name="realsense_EE_parent" default="$(optenv REALSENSE_EE_PARENT ee_link)" />
-    <xacro:arg name="realsense_EE_xyz" default="$(optenv REALSENSE_EE_XYZ 0.095 0.000 -0.075)" />
-    <xacro:arg name="realsense_EE_rpy" default="$(optenv REALSENSE_EE_RPY -3.14 0.0 1.57)" />
     <xacro:include filename="$(find ur_e_description)/urdf/realsense/intel_realsense.urdf.xacro" />
-    <xacro:if value="$(arg realsense_EE_enabled)">
-      <link name="$(arg realsense_EE_prefix)_realsense_mountpoint" />
-      <joint name="$(arg realsense_EE_prefix)_realsense_mountpoint_joint" type="fixed">
-        <origin xyz="$(arg realsense_EE_xyz)" rpy="$(arg realsense_EE_rpy)" />
-        <parent link="$(arg realsense_EE_parent)" />
-        <child link="$(arg realsense_EE_prefix)_realsense_mountpoint" />
-      </joint>
-      <xacro:intel_realsense_mount prefix="$(arg realsense_EE_prefix)"
-        topic="$(arg realsense_EE_topic)"
-        parent_link="$(arg realsense_EE_prefix)_realsense_mountpoint" />
-    </xacro:if>
-    <!-- add intel realsense d415 sensor -->
+    <xacro:sensor_d415 parent="ee_link" use_nominal_extrinsics="true">
+      <origin xyz="0.095 0.000 -0.075"
+        rpy="-3.14 0.0 1.57" />
+    </xacro:sensor_d415>
     <!-- SENSOR CAMERA ON END EFFECTOR -->
     <xacro:ur_arm_transmission prefix="${prefix}" />
@@ -543,9 +531,9 @@
     <!-- <link name="${prefix}base" />
     <joint name="${prefix}base_link-base_fixed_joint" type="fixed"> -->
-    <!-- NOTE: this rotation is only needed as long as base_link itself is
+      <!-- NOTE: this rotation is only needed as long as base_link itself is
                  not corrected wrt the real robot (ie: rotated over 180
                  degrees)
       -->
-    <!-- <origin xyz="0 0 0" rpy="0 0 ${-pi}" />
+      <!-- <origin xyz="0 0 0" rpy="0 0 ${-pi}" />
       <parent link="${prefix}base_link" />
       <child link="${prefix}base" />
