Commit message: update xacro file to match real zau robot

File: UR5/ur_e_description/urdf/realsense/intel_realsense.urdf.xacro (robot description, xacro)
@@ -10,23 +10,24 @@
   <xacro:include filename="$(find realsense2_description)/urdf/_materials.urdf.xacro" />
   <xacro:include filename="$(find realsense2_description)/urdf/_usb_plug.urdf.xacro" />
-  <xacro:macro name="sensor_d415" params="parent *origin  name:=camera  use_nominal_extrinsics:=false add_plug:=false use_mesh:=true">
+  <xacro:macro name="sensor_d415"
+    params="parent *origin  name:=camera  use_nominal_extrinsics:=false add_plug:=false use_mesh:=true">
     <xacro:property name="M_PI" value="3.1415926535897931" />
     <!-- The following values are approximate, and the camera node
      publishing TF values with actual calibrated camera extrinsic values -->
-    <xacro:property name="d415_cam_depth_to_infra1_offset" value="0.0"/>
-    <xacro:property name="d415_cam_depth_to_infra2_offset" value="-0.055"/>
-    <xacro:property name="d415_cam_depth_to_color_offset" value="0.015"/>
+    <xacro:property name="d415_cam_depth_to_infra1_offset" value="0.0" />
+    <xacro:property name="d415_cam_depth_to_infra2_offset" value="-0.055" />
+    <xacro:property name="d415_cam_depth_to_color_offset" value="0.015" />
     <!-- The following values model the aluminum peripherial case for the
   	d415 camera, with the camera joint represented by the actual
   	peripherial camera tripod mount -->
-    <xacro:property name="d415_cam_width" value="0.099"/>
-    <xacro:property name="d415_cam_height" value="0.023"/>
-    <xacro:property name="d415_cam_depth" value="0.02005"/>
-    <xacro:property name="d415_cam_mount_from_center_offset" value="0.00987"/>
+    <xacro:property name="d415_cam_width" value="0.099" />
+    <xacro:property name="d415_cam_height" value="0.023" />
+    <xacro:property name="d415_cam_depth" value="0.02005" />
+    <xacro:property name="d415_cam_mount_from_center_offset" value="0.00987" />
     <!-- The following offset is relative the the physical d415 camera peripherial
   	camera tripod mount -->
-    <xacro:property name="d415_cam_depth_px" value="${d415_cam_mount_from_center_offset}"/>
-    <xacro:property name="d415_cam_depth_py" value="0.020"/>
-    <xacro:property name="d415_cam_depth_pz" value="${d415_cam_height/2}"/>
+    <xacro:property name="d415_cam_depth_px" value="${d415_cam_mount_from_center_offset}" />
+    <xacro:property name="d415_cam_depth_py" value="0.020" />
+    <xacro:property name="d415_cam_depth_pz" value="${d415_cam_height/2}" />
     <!-- camera body, with origin at bottom screw mount -->
     <joint name="${name}_joint" type="fixed">
@@ -44,21 +45,22 @@
       <visual>
         <xacro:if value="${use_mesh}">
-          <origin xyz="${d415_cam_mount_from_center_offset} ${-d415_cam_depth_py} 0" rpy="${M_PI/2} 0 ${M_PI/2}"/>
+          <origin xyz="${d415_cam_mount_from_center_offset} ${-d415_cam_depth_py} 0"
+            rpy="${M_PI/2} 0 ${M_PI/2}" />
           <geometry>
             <mesh filename="package://realsense2_description/meshes/d415.stl" />
           </geometry>
-          <material name="aluminum"/>
+          <material name="aluminum" />
         </xacro:if>
         <xacro:unless value="${use_mesh}">
-          <origin xyz="0 ${-d415_cam_depth_py} 0" rpy="0 0 0"/>
+          <origin xyz="0 ${-d415_cam_depth_py} 0" rpy="0 0 0" />
           <geometry>
-            <box size="${d415_cam_depth} ${d415_cam_width} ${d415_cam_height}"/>
+            <box size="${d415_cam_depth} ${d415_cam_width} ${d415_cam_height}" />
           </geometry>
         </xacro:unless>
       </visual>
       <collision>
-        <origin xyz="0 ${-d415_cam_depth_py} 0" rpy="0 0 0"/>
+        <origin xyz="0 ${-d415_cam_depth_py} 0" rpy="0 0 0" />
         <geometry>
-        <box size="${d415_cam_depth} ${d415_cam_width} ${d415_cam_height}"/>
+          <box size="${d415_cam_depth} ${d415_cam_width} ${d415_cam_height}" />
         </geometry>
       </collision>
@@ -70,13 +72,14 @@
       </inertial>
     </link>
-    <!-- Use the nominal extrinsics between camera frames if the calibrated extrinsics aren't being published. e.g. running the device in simulation  -->
+    <!-- Use the nominal extrinsics between camera frames if the calibrated extrinsics aren't being
+    published. e.g. running the device in simulation  -->
     <xacro:if value="${use_nominal_extrinsics}">
       <!-- camera depth joints and links -->
       <joint name="${name}_depth_joint" type="fixed">
-        <origin xyz="0 0 0" rpy="0 0 0"/>
-        <parent link="${name}_link"/>
+        <origin xyz="0 0 0" rpy="0 0 0" />
+        <parent link="${name}_link" />
         <child link="${name}_depth_frame" />
       </joint>
-      <link name="${name}_depth_frame"/>
+      <link name="${name}_depth_frame" />
       <joint name="${name}_depth_optical_joint" type="fixed">
         <origin xyz="0 0 0" rpy="${-M_PI/2} 0 ${-M_PI/2}" />
@@ -84,25 +87,25 @@
         <child link="${name}_depth_optical_frame" />
       </joint>
-      <link name="${name}_depth_optical_frame"/>
+      <link name="${name}_depth_optical_frame" />
       <!-- camera left IR joints and links -->
-      <joint name="${name}_infra1_joint" type="fixed">
+      <!-- <joint name="${name}_infra1_joint" type="fixed">
         <origin xyz="0 ${d415_cam_depth_to_infra1_offset} 0" rpy="0 0 0" />
         <parent link="${name}_link" />
         <child link="${name}_infra1_frame" />
       </joint>
-      <link name="${name}_infra1_frame"/>
-      <joint name="${name}_infra1_optical_joint" type="fixed">
+      <link name="${name}_infra1_frame" /> -->
+      <!-- <joint name="${name}_infra1_optical_joint" type="fixed">
         <origin xyz="0 0 0" rpy="${-M_PI/2} 0 ${-M_PI/2}" />
         <parent link="${name}_infra1_frame" />
         <child link="${name}_infra1_optical_frame" />
       </joint>
-      <link name="${name}_infra1_optical_frame"/>
+      <link name="${name}_infra1_optical_frame" /> -->
       <!-- camera right IR joints and links -->
-      <joint name="${name}_infra2_joint" type="fixed">
+      <!-- <joint name="${name}_infra2_joint" type="fixed">
         <origin xyz="0 ${d415_cam_depth_to_infra2_offset} 0" rpy="0 0 0" />
         <parent link="${name}_link" />
         <child link="${name}_infra2_frame" />
       </joint>
-      <link name="${name}_infra2_frame"/>
+      <link name="${name}_infra2_frame" />
       <joint name="${name}_infra2_optical_joint" type="fixed">
         <origin xyz="0 0 0" rpy="${-M_PI/2} 0 ${-M_PI/2}" />
@@ -110,5 +113,5 @@
         <child link="${name}_infra2_optical_frame" />
       </joint>
-      <link name="${name}_infra2_optical_frame"/>
+      <link name="${name}_infra2_optical_frame" /> -->
       <!-- camera color joints and links -->
       <joint name="${name}_color_joint" type="fixed">
@@ -117,15 +120,29 @@
         <child link="${name}_color_frame" />
       </joint>
-      <link name="${name}_color_frame"/>
-      <joint name="${name}_color_optical_joint" type="fixed">
+      <link name="${name}_color_frame" />
+      <!-- <joint name="${name}_color_optical_joint" type="fixed">
         <origin xyz="0 0 0" rpy="${-M_PI/2} 0 ${-M_PI/2}" />
         <parent link="${name}_color_frame" />
         <child link="${name}_color_optical_frame" />
       </joint>
-      <link name="${name}_color_optical_frame"/>
+      <link name="${name}_color_optical_frame" /> -->
+      <joint name="${name}_aligned_depth_to_color_frame_joint" type="fixed">
+        <origin xyz="0 0 0" rpy="${-M_PI/2} 0 ${-M_PI/2}" />
+        <parent link="${name}_link" />
+        <child link="${name}_aligned_depth_to_color_frame" />
+      </joint>
+      <link name="${name}_aligned_depth_to_color_frame" />
+      <joint name="${name}_color_optical_joint" type="fixed">
+        <origin xyz="0 0 0" rpy="${-M_PI/2} 0 ${-M_PI/2}" />
+        <parent link="${name}_aligned_depth_to_color_frame" />
+        <child link="${name}_color_optical_frame" />
+      </joint>
+      <link name="${name}_color_optical_frame" />
     </xacro:if>
     <xacro:if value="${add_plug}">
       <xacro:usb_plug parent="${name}_link" name="${name}_usb_plug">
-        <origin xyz="${d415_cam_mount_from_center_offset - 0.01587} ${-d415_cam_depth_py - 0.0358} 0" rpy="0 0 0"/>
+        <origin
+          xyz="${d415_cam_mount_from_center_offset - 0.01587} ${-d415_cam_depth_py - 0.0358} 0"
+          rpy="0 0 0" />
       </xacro:usb_plug>
     </xacro:if>

Commit message: update summary

File: UR5/ur_e_description/urdf/realsense/intel_realsense.urdf.xacro (robot description, xacro)
@@ -128,5 +128,5 @@
       <link name="${name}_color_optical_frame" /> -->
       <joint name="${name}_aligned_depth_to_color_frame_joint" type="fixed">
-        <origin xyz="0 0 0" rpy="${-M_PI/2} 0 ${-M_PI/2}" />
+        <origin xyz="0 0 0" rpy="0 0 0" />
         <parent link="${name}_link" />
         <child link="${name}_aligned_depth_to_color_frame" />
